Commit message: Revert head_2 CoM because Gazebo shows it in wrong place.

File: reem_description/urdf/head/head.urdf.xacro (robot description, xacro)
@@ -44,5 +44,5 @@
     <joint name="${name}_joint" type="revolute">
       <parent link="${parent}"/>
-        <child link="${name}_link"/>
+      <child link="${name}_link"/>
       <origin xyz="-0.024 -0.412 0" rpy="${90.0 * deg_to_rad} 0 0" />
       <axis xyz="0 0 1" />
@@ -60,5 +60,6 @@
     <link name="${name}_link">
       <inertial>
-        <origin xyz="-0.04431 -0.13008 0.00011" rpy="0 0 0" />
+<!--         <origin xyz="-0.04431 -0.13008 0.00011" rpy="0 0 0" /> --> <!--TODO: Figure out why CoM is not properly displayed in Gazebo!-->
+        <origin xyz="0 0 0" rpy="0 0 0" />
         <mass value="1.20862" />
         <!-- NOTE: Assuming box with d=0.28433, w=0.20302, h=0.26741 -->
