Commit message: Add better center of mass estimates (no inertia).
Signed-off-by: Adolfo Rodriguez Tsouroukdissian <adolfo.rodriguez@pal-robotics.com>

File: reem_description/urdf/arm/arm.urdf.xacro (robot description, xacro)
@@ -33,6 +33,6 @@
     <link name="arm_${side}_1_link">
       <inertial>
-        <origin xyz="0.00013 -0.01746 -0.10788" rpy="0 0 0"/>
-        <mass value="1.775" />
+        <origin xyz="${reflect*0.000816} -0.00041 ${reflect*0.17187}" rpy="0 0 0"/>
+        <mass value="1.08342" />
         <inertia ixx="0"  ixy="0"  ixz="0" iyy="0" iyz="0" izz="0" />
       </inertial>
@@ -53,6 +53,6 @@
    <link name="arm_${side}_2_link">
       <inertial>
-        <origin xyz="0.0181 -0.10023 -0.0053" rpy="0 0 0"/>
-        <mass value="1.575" />
+        <origin xyz="0.00454 -0.01220 -0.00823" rpy="0 0 0"/>
+        <mass value="1.65272" />
         <inertia ixx="0"  ixy="0"  ixz="0" iyy="0" iyz="0" izz="0" />
       </inertial>
@@ -73,6 +73,6 @@
     <link name="arm_${side}_3_link">
       <inertial>
-        <origin xyz="0.00172 ${reflect * 0.01644} ${reflect * 0.10561}" rpy="0 0 0"/>
-        <mass value="1.645" />
+        <origin xyz="0.00506 ${reflect * -0.00198} ${reflect * -0.00231}" rpy="0 0 0"/>
+        <mass value="1.60923" />
         <inertia ixx="0"  ixy="0"  ixz="0" iyy="0" iyz="0" izz="0" />
       </inertial>
@@ -93,6 +93,6 @@
     <link name="arm_${side}_4_link">
       <inertial>
-        <origin xyz="-0.05593 ${-reflect * 0.01466} ${-reflect * 0.01020}" rpy="0 0 0"/>
-        <mass value="0.775" />
+        <origin xyz="-0.01128 ${-reflect * 0.00406} ${-reflect * 0.00837}" rpy="0 0 0"/>
+        <mass value="1.61314" />
         <inertia ixx="0"  ixy="0"  ixz="0" iyy="0" iyz="0" izz="0" />
       </inertial>
@@ -113,6 +113,6 @@
     <link name="arm_${side}_5_link">
       <inertial>
-        <origin xyz="-0.00232 0 ${reflect * 0.05825}" rpy="0 0 0"/>
-        <mass value="1.440" />
+        <origin xyz="-0.00051 -0.00003 ${reflect * -0.06628}" rpy="0 0 0"/>
+        <mass value="2.26358" />
         <inertia ixx="0"  ixy="0"  ixz="0" iyy="0" iyz="0" izz="0" />
       </inertial>
@@ -133,6 +133,6 @@
     <link name="arm_${side}_6_link">
       <inertial>
-        <origin xyz="0 -0.00656 0" rpy="0 0 0"/>
-        <mass value="0.250" />
+        <origin xyz="-0.00005 -0.01216 0.0" rpy="0 0 0"/>
+        <mass value="0.35648" />
         <inertia ixx="0"  ixy="0"  ixz="0" iyy="0" iyz="0" izz="0" />
       </inertial>
@@ -153,6 +153,6 @@
     <link name="arm_${side}_7_link">
       <inertial>
-        <origin xyz="0 0 0" rpy="0 0 0"/>
-        <mass value="0.001" /> <!-- NOTE: Dummy mass -->
+        <origin xyz="0.001880317  -0.005168045 -0.109404509" rpy="0 0 0"/>
+        <mass value="0.152461831" /> <!-- NOTE: Dummy mass -->
         <inertia ixx="0"  ixy="0"  ixz="0" iyy="0" iyz="0" izz="0" />
       </inertial>

File: reem_description/urdf/base/base.urdf.xacro (robot description, xacro)
@@ -151,6 +151,6 @@
     <link name="${name}_link">
       <inertial>
-        <origin xyz="-0.3 0 0.2" rpy="0 0 0" /> <!-- assuming d=0.6, w=0.5, h=0.4 -->
-        <mass value="90.0" />
+        <origin xyz="-0.14527 -0.00003 0.24721" rpy="0 0 0" /> <!-- assuming d=0.6, w=0.5, h=0.4 -->
+        <mass value="63.58850" />
         <inertia ixx="3.42"  ixy="0"  ixz="0" iyy="4.33" iyz="0" izz="5.08" /> <!-- assuming d=0.6, w=0.5, h=0.4 -->
       </inertial>

File: reem_description/urdf/head/head.urdf.xacro (robot description, xacro)
@@ -23,6 +23,6 @@
     <link name="${name}_link">
       <inertial>
-        <origin />
-        <mass value="1.0" />
+        <origin xyz="0.01741 0.00466 -0.00434" rpy="0 0 0" />
+        <mass value="0.98547" />
         <inertia ixx="1"  ixy="0"  ixz="0" iyy="1" iyz="0" izz="1" />
       </inertial>
@@ -59,6 +59,6 @@
     <link name="${name}_link">
       <inertial>
-        <origin />
-        <mass value="1.0" />
+        <origin xyz="-0.04431 -0.13008 0.000011" rpy="0 0 0" />
+        <mass value="1.20862" />
         <inertia ixx="1"  ixy="0"  ixz="0" iyy="1" iyz="0" izz="1" />
       </inertial>

File: reem_description/urdf/torso/torso.urdf.xacro (robot description, xacro)
@@ -23,6 +23,6 @@
     <link name="${name}_1_link">
       <inertial>
-        <origin xyz="0 0 0" rpy="0 0 0" />
-        <mass value="1.0" />
+        <origin xyz="-0.00299 0.00501 -0.07336" rpy="0 0 0" />
+        <mass value="6.653" />
         <inertia ixx="1"  ixy="0"  ixz="0" iyy="1" iyz="0" izz="1" />
       </inertial>
@@ -58,6 +58,6 @@
     <link name="${name}_2_link">
       <inertial>
-        <origin />
-        <mass value="1.0" />
+        <origin xyz="-0.01241 -0.16263 0.00011" rpy="0 0 0"/>
+        <mass value="11.717" />
         <inertia ixx="1"  ixy="0"  ixz="0" iyy="1" iyz="0" izz="1" />
       </inertial>

Commit message: Removed stale comment about dummy mass.

File: reem_description/urdf/arm/arm.urdf.xacro (robot description, xacro)
@@ -154,5 +154,5 @@
       <inertial>
         <origin xyz="0.001880317  -0.005168045 -0.109404509" rpy="0 0 0"/>
-        <mass value="0.152461831" /> <!-- NOTE: Dummy mass -->
+        <mass value="0.152461831" />
         <inertia ixx="0"  ixy="0"  ixz="0" iyy="0" iyz="0" izz="0" />
       </inertial>

Commit message: Fill gap between arm_2 and arm_3 with a dummy cylindrical link.

File: reem_description/urdf/arm/arm.urdf.xacro (robot description, xacro)
@@ -117,4 +117,25 @@
       <dynamics friction="${arm_friction}" damping="${arm_damping}"/>
     </joint>
+    <!-- Dummy visualization-only link -->
+    <link name="arm_${side}_3_internal_link">
+      <visual>
+        <origin xyz="0 0 0" rpy="0 0 0" />
+        <geometry>
+          <cylinder radius="0.045" length="0.01"/>
+        </geometry>
+        <material name="DarkGrey" />
+      </visual>
+      <collision>
+        <origin xyz="0 0 0" rpy="0 0 0" />
+        <geometry>
+          <cylinder radius="0.045" length="0.01"/>
+        </geometry>
+      </collision>
+    </link>
+    <joint name="arm_${side}_3_internal_joint" type="fixed">
+      <parent link="arm_${side}_3_link" />
+      <child link="arm_${side}_3_internal_link" />
+      <origin xyz="0 0 ${-reflect * 0.025}" rpy="0 0 0" />
+    </joint>
     <!--************************-->
     <!--        ELBOW           -->

Commit message: Fix wrong translation for arm_1 axis.

File: reem_description/urdf/arm/arm.urdf.xacro (robot description, xacro)
@@ -56,5 +56,5 @@
       <parent link="torso_2_link" />
       <child link="arm_${side}_1_link" />
-      <origin xyz="-0.01 -0.273 0" rpy="${(-165.0 * reflect) * deg_to_rad} 0 0" />
+      <origin xyz="-0.015 -0.273 0" rpy="${(-165.0 * reflect) * deg_to_rad} 0 0" />
       <axis xyz="0 0 1" />
       <limit lower="${-45.0 * deg_to_rad}" upper="${180.0 * deg_to_rad}" effort="0.0" velocity="${arm_max_vel}" />

Commit message: Add Gazebo color spec to arm_3_internal_link.

File: reem_description/urdf/arm/arm.urdf.xacro (robot description, xacro)
@@ -133,4 +133,7 @@
       </collision>
     </link>
+    <gazebo reference="arm_${side}_3_internal_link">
+      <material>reem/DarkGrey</material>
+    </gazebo>
     <joint name="arm_${side}_3_internal_joint" type="fixed">
       <parent link="arm_${side}_3_link" />

Commit message: Fix typo in arm_*_3_joint upper joint limit.

File: reem_description/urdf/arm/arm.urdf.xacro (robot description, xacro)
@@ -114,5 +114,5 @@
       <origin xyz="0.02 -0.142 0" rpy="${90.0 * reflect * deg_to_rad} 0 0" />
       <axis xyz="0 0 1" />
-      <limit lower="${-135.0 * deg_to_rad}" upper="${157.5.0 * deg_to_rad}" effort="0.0" velocity="${arm_max_vel}" />
+      <limit lower="${-135.0 * deg_to_rad}" upper="${157.5 * deg_to_rad}" effort="0.0" velocity="${arm_max_vel}" />
       <dynamics friction="${arm_friction}" damping="${arm_damping}"/>
     </joint>

Commit message: Update inertial properties.
- Fix some wrongly placed inertial origins.

- Tune joint dynamic parameters to improve dynamic simulation stability.

File: reem_description/urdf/arm/arm.urdf.xacro (robot description, xacro)
@@ -15,8 +15,8 @@
   <xacro:property name="arm_reduction_low"  value= "80.0" />
   <xacro:property name="wrist_reduction"    value="336.0" />
-  <xacro:property name="arm_friction"    value="1.0" /> <!--TODO: Tune-->
-  <xacro:property name="wrist_friction"  value="1.0" /> <!--TODO: Tune-->
-  <xacro:property name="arm_damping"     value="1.0" /> <!--TODO: Tune-->
-  <xacro:property name="wrist_damping"   value="1.0" /> <!--TODO: Tune-->
+  <xacro:property name="arm_friction"    value="5.0" />
+  <xacro:property name="wrist_friction"  value="5.0" />
+  <xacro:property name="arm_damping"     value="2.0" />
+  <xacro:property name="wrist_damping"   value="0.1" />
  <xacro:property name="arm_max_vel"      value="1.0" />
  <xacro:property name="wrist_max_vel"    value="1.0" />
@@ -33,9 +33,8 @@
     <link name="arm_${side}_1_link">
       <inertial>
-        <origin xyz="${reflect*0.0006} -0.0005 ${reflect*0.20739}" rpy="0 0 0"/>
+        <origin xyz="0.0006 -0.0005 ${reflect*0.20739}" rpy="0 0 0"/>
         <mass value="2.148" />
-        <!-- NOTE: Assuming cylinder with r=0.05, h=0.05 roughly around second motor -->
-        <inertia ixx="0"  ixy="0"  ixz="0" iyy="0" iyz="0" izz="0" />
-<!--         <inertia ixx="0.0026850"  ixy="0"  ixz="0" iyy="0.0017900" iyz="0" izz="0.0017900" /> -->
+        <!-- NOTE: Assuming cylinder centered at CoM with r=0.05, h=0.05 with axis parallel to x coordinate -->
+        <inertia ixx="0.0026850"  ixy="0"  ixz="0" iyy="0.0017900" iyz="0" izz="0.0017900" />
       </inertial>
       <visual>
@@ -63,7 +62,8 @@
    <link name="arm_${side}_2_link">
       <inertial>
-        <origin xyz="0.0183 -0.09275 -0.00478" rpy="0 0 0"/>
+        <origin xyz="0.0183 -0.09275 ${reflect*0.00478}" rpy="0 0 0"/>
         <mass value="1.610" />
-        <inertia ixx="0"  ixy="0"  ixz="0" iyy="0" iyz="0" izz="0" />
+        <!-- NOTE: Assuming cylinder centered at CoM with r=0.05, h=0.05 with axis parallel to y coordinate -->
+        <inertia ixx="0.0013417"  ixy="0"  ixz="0" iyy="0.0020125" iyz="0" izz="0.0013417" />
       </inertial>
       <visual>
@@ -91,7 +91,8 @@
     <link name="arm_${side}_3_link">
       <inertial>
-        <origin xyz="0.00045 ${reflect * -0.01547} ${reflect * -0.07654}" rpy="0 0 0"/>
+        <origin xyz="0.00045 -0.01547 ${reflect * 0.07654}" rpy="0 0 0"/>
         <mass value="1.656" />
-        <inertia ixx="0"  ixy="0"  ixz="0" iyy="0" iyz="0" izz="0" />
+        <!-- NOTE: Assuming cylinder centered at CoM with r=0.05, h=0.05 with axis parallel to x coordinate -->
+        <inertia ixx="0.0020700"  ixy="0"  ixz="0" iyy="0.0013800" iyz="0" izz="0.0013800" />
       </inertial>
       <visual>
@@ -146,7 +147,8 @@
     <link name="arm_${side}_4_link">
       <inertial>
-        <origin xyz="-0.06424 ${-reflect * 0.01712} ${-reflect * 0.00666}" rpy="0 0 0"/>
+        <origin xyz="-0.06424 0.01712 ${-reflect * 0.00666}" rpy="0 0 0"/>
         <mass value="1.013" />
-        <inertia ixx="0"  ixy="0"  ixz="0" iyy="0" iyz="0" izz="0" />
+        <!-- NOTE: Assuming cylinder centered at CoM with r=0.05, h=0.05 with axis parallel to x coordinate -->
+        <inertia ixx="0.0012663"  ixy="0"  ixz="0" iyy="0.00084417" iyz="0" izz="0.00084417" />
       </inertial>
       <visual>
@@ -177,7 +179,8 @@
     <link name="arm_${side}_5_link">
       <inertial>
-        <origin xyz="-0.00045 -0.00009 ${reflect * -0.08726}" rpy="0 0 0"/>
+        <origin xyz="-0.00045 -0.00009 ${reflect * 0.08726}" rpy="0 0 0"/>
         <mass value="1.858" />
-        <inertia ixx="0"  ixy="0"  ixz="0" iyy="0" iyz="0" izz="0" />
+        <!-- NOTE: Assuming cylinder centered at CoM with r=0.05, h=0.1 with axis parallel to z coordinate -->
+        <inertia ixx="0.0027096"  ixy="0"  ixz="0" iyy="0.0027096" iyz="0" izz="0.0023225" />
       </inertial>
       <visual>
@@ -205,7 +208,8 @@
     <link name="arm_${side}_6_link">
       <inertial>
-        <origin xyz="-0.0002 -0.01155 0.00002" rpy="0 0 0"/>
+        <origin xyz="-0.0002 -0.01155 ${reflect * 0.00002}" rpy="0 0 0"/>
         <mass value="0.255" />
-        <inertia ixx="0.0001335"  ixy="0"  ixz="0" iyy="0.0001335" iyz="0" izz="0.000204" />
+        <!-- NOTE: Assuming cylinder centered at CoM with r=0.02, h=0.08 with axis parallel to z coordinate -->
+        <inertia ixx="0.0001615"  ixy="0"  ixz="0" iyy="0.0001615" iyz="0" izz="0.000051" />
       </inertial>
       <visual>
@@ -234,6 +238,7 @@
       <inertial>
         <!--TODO: Verify these inertial parameters-->
-        <origin xyz="0.001880317  -0.005168045 -0.109404509" rpy="0 0 0"/>
+        <origin xyz="0.001880317  -0.005168045 ${reflect * 0.109404509}" rpy="0 0 0"/>
         <mass value="0.152461831" />
+        <!-- NOTE: Assuming point mass -->
         <inertia ixx="0"  ixy="0"  ixz="0" iyy="0" iyz="0" izz="0" />
       </inertial>

File: reem_description/urdf/base/base.urdf.xacro (robot description, xacro)
@@ -71,7 +71,5 @@
         <origin xyz="0 0 0" rpy="0 0 0"/>
         <mass value="0.1" />
-        <inertia  ixx="0" ixy="0" ixz="0"
-                  iyy="0" iyz="0"
-                  izz="0" />
+        <inertia  ixx="0" ixy="0" ixz="0" iyy="0" iyz="0" izz="0" />
       </inertial>
       <visual>
@@ -93,7 +91,5 @@
         <origin xyz="0 0 0" rpy="0 0 0"/>
         <mass value="0.4" />
-        <inertia  ixx="0.00044" ixy="0" ixz="0"
-                  iyy="0.00044" iyz="0"
-                  izz="0.00078" />
+        <inertia  ixx="0.00044" ixy="0" ixz="0" iyy="0.00044" iyz="0" izz="0.00078" />
         </inertial>
       <visual>
@@ -132,18 +128,8 @@
   <property name="base_laser_y" value="0.0" />
   <property name="base_laser_z" value="0.08" />
-  <property name="base_laser_size_x" value="0.11" />
-  <property name="base_laser_size_y" value="0.11" />
-  <property name="base_laser_size_z" value="0.16" />
-  <property name="base_laser_collision_offset_z" value="0.00" />
-  <property name="base_laser_collision_offset_y" value="0.00" />
-  <property name="base_laser_collision_offset_x" value="0.00" />
   <!-- simplified box collision geometry for hokuyo laser -->
   <property name="torso_laser_x" value="0.04" />
   <property name="torso_laser_y" value="0.0" />
   <property name="torso_laser_z" value="0.77" />
-  <!--property name="torso_laser_size_x" value="0.05" />
-  <property name="torso_laser_size_y" value="0.05" />
-  <property name="torso_laser_size_z" value="0.03" /-->
-  <!--property name="torso_laser_collision_offset_z" value="0.750" /-->
   <xacro:macro name="reem_base" params="name">
     <!--************************-->
@@ -178,6 +164,5 @@
         <mass value="0.1" />
         <origin xyz="0 0 0" />
-        <inertia ixx="0.0" ixy="0.0" ixz="0.0"
-                 iyy="0.0" iyz="0.0" izz="0.0" />
+        <inertia ixx="0.0" ixy="0.0" ixz="0.0" iyy="0.0" iyz="0.0" izz="0.0" />
       </inertial>
       <visual>
@@ -329,6 +314,5 @@
         <mass value="1.0" />
         <origin xyz="0 0 -0.5" />
-        <inertia ixx="0.0" ixy="0.0" ixz="0.0"
-                 iyy="0.0" iyz="0.0" izz="0.0" />
+        <inertia ixx="0.0" ixy="0.0" ixz="0.0" iyy="0.0" iyz="0.0" izz="0.0" />
       </inertial>
       <visual>

File: reem_description/urdf/hand/hand.urdf.xacro (robot description, xacro)
@@ -120,6 +120,6 @@
     <link name="${name}_${side}_palm_link">
       <inertial>
-        <!--<origin xyz="0.07547 0.00468 0.00291" rpy="0 0 0" />-->  <!--TODO: Figure out why CoM is not properly displayed in Gazebo!-->
-        <origin xyz="0 0 0" rpy="0 0 0" />
+        <!--<origin xyz="0.07547 ${-reflect * 0.00468} 0.00291" rpy="0 0 0" />-->
+        <origin xyz="0 ${-reflect * 0.07547} 0 " rpy="0 0 0" /> <!--TODO: This does not make sense!, there must be a bug in how Gazebo bungles the CoM of a chain of fixed joints-->
         <mass value="0.91066" />
         <inertia ixx="0"  ixy="0"  ixz="0" iyy="0" iyz="0" izz="0" />

File: reem_description/urdf/head/head.urdf.xacro (robot description, xacro)
@@ -14,6 +14,6 @@
   <include filename="$(find reem_description)/urdf/head/head.gazebo.xacro" />
   <include filename="$(find reem_description)/urdf/head/head.transmission.xacro" />
-  <xacro:property name="head_friction" value="3.0" /> <!--TODO: Tune-->
-  <xacro:property name="head_damping"  value="1.0" /> <!--TODO: Tune-->
+  <xacro:property name="head_friction" value="3.0" />
+  <xacro:property name="head_damping"  value="1.0" />
   <xacro:property name="head_max_vel"  value="1.0" />
   <!--************************-->
@@ -60,6 +60,5 @@
     <link name="${name}_link">
       <inertial>
-<!--         <origin xyz="-0.04431 -0.13008 0.00011" rpy="0 0 0" /> --> <!--TODO: Figure out why CoM is not properly displayed in Gazebo!-->
-        <origin xyz="0 0 0" rpy="0 0 0" />
+        <origin xyz="-0.04431 -0.13008 0.00011" rpy="0 0 0" />
         <mass value="1.20862" />
         <!-- NOTE: Assuming box with d=0.28433, w=0.20302, h=0.26741 -->

File: reem_description/urdf/torso/torso.urdf.xacro (robot description, xacro)
@@ -14,6 +14,4 @@
   <include filename="$(find reem_description)/urdf/torso/torso.gazebo.xacro" />
   <include filename="$(find reem_description)/urdf/torso/torso.transmission.xacro" />
-  <xacro:property name="torso_friction" value="10.0" /> <!--TODO: Tune-->
-  <xacro:property name="torso_damping"  value="10.0" />  <!--TODO: Tune-->
   <xacro:property name="torso_max_vel"  value="1.0" />
   <xacro:macro name="reem_torso" params="name parent">
@@ -46,5 +44,5 @@
       <axis xyz="0 0 1" />
       <limit lower="${-75.0 * deg_to_rad}" upper="${75.0 * deg_to_rad}" effort="0.0" velocity="${torso_max_vel}" />
-      <dynamics damping="${torso_damping}" friction="${torso_friction}"/>
+      <dynamics damping="10.0" friction="5.0"/>
     </joint>
     <!-- extensions -->
@@ -79,5 +77,5 @@
       <axis xyz="0 0 1" />
       <limit lower="${-15.0 * deg_to_rad}" upper="${45.0 * deg_to_rad}" effort="0.0" velocity="${torso_max_vel}" />
-      <dynamics damping="${torso_damping}" friction="${torso_friction}"/>
+      <dynamics damping="10.0" friction="10.0"/>
     </joint>
     <!-- extensions -->

Commit message: Reduce damping for certain joints.

File: reem_description/urdf/arm/arm.urdf.xacro (robot description, xacro)
@@ -17,5 +17,5 @@
   <xacro:property name="arm_friction"    value="5.0" />
   <xacro:property name="wrist_friction"  value="5.0" />
-  <xacro:property name="arm_damping"     value="2.0" />
+  <xacro:property name="arm_damping"     value="0.1" />
   <xacro:property name="wrist_damping"   value="0.1" />
  <xacro:property name="arm_max_vel"      value="1.0" />

File: reem_description/urdf/torso/torso.urdf.xacro (robot description, xacro)
@@ -44,5 +44,5 @@
       <axis xyz="0 0 1" />
       <limit lower="${-75.0 * deg_to_rad}" upper="${75.0 * deg_to_rad}" effort="0.0" velocity="${torso_max_vel}" />
-      <dynamics damping="10.0" friction="5.0"/>
+      <dynamics damping="5.0" friction="5.0"/>
     </joint>
     <!-- extensions -->
@@ -77,5 +77,5 @@
       <axis xyz="0 0 1" />
       <limit lower="${-15.0 * deg_to_rad}" upper="${45.0 * deg_to_rad}" effort="0.0" velocity="${torso_max_vel}" />
-      <dynamics damping="10.0" friction="10.0"/>
+      <dynamics damping="5.0" friction="10.0"/>
     </joint>
     <!-- extensions -->

Commit message: Update arm_3 geometry and remove arm_3_internal.

File: reem_description/urdf/arm/arm.urdf.xacro (robot description, xacro)
@@ -118,28 +118,4 @@
       <dynamics friction="${arm_friction}" damping="${arm_damping}"/>
     </joint>
-    <!-- Dummy visualization-only link -->
-    <link name="arm_${side}_3_internal_link">
-      <visual>
-        <origin xyz="0 0 0" rpy="0 0 0" />
-        <geometry>
-          <cylinder radius="0.045" length="0.01"/>
-        </geometry>
-        <material name="DarkGrey" />
-      </visual>
-      <collision>
-        <origin xyz="0 0 0" rpy="0 0 0" />
-        <geometry>
-          <cylinder radius="0.045" length="0.01"/>
-        </geometry>
-      </collision>
-    </link>
-    <gazebo reference="arm_${side}_3_internal_link">
-      <material>reem/DarkGrey</material>
-    </gazebo>
-    <joint name="arm_${side}_3_internal_joint" type="fixed">
-      <parent link="arm_${side}_3_link" />
-      <child link="arm_${side}_3_internal_link" />
-      <origin xyz="0 0 ${-reflect * 0.025}" rpy="0 0 0" />
-    </joint>
     <!--************************-->
     <!--        ELBOW           -->
