Commit message: Update effort limits (non-realistic values).

File: reem_description/urdf/arm/wrist.urdf.xacro (robot description, xacro)
@@ -51,5 +51,5 @@
       <origin xyz="-0.088 0.02 0" rpy="0 ${-90.0 * reflect * deg_to_rad} 0" />
       <axis xyz="0 0 1" />
-      <limit lower="${-120.0 * deg_to_rad}" upper="${120.0 * deg_to_rad}" effort="6" velocity="${wrist_max_vel}" /> <!--TODO: Check effort value!-->
+      <limit lower="${-120.0 * deg_to_rad}" upper="${120.0 * deg_to_rad}" effort="16" velocity="${wrist_max_vel}" /> <!--TODO: Check effort value!-->
       <dynamics friction="${wrist_friction}" damping="0.5"/>
     </joint>
@@ -81,5 +81,5 @@
       <origin xyz="0 0 ${0.15 * reflect}" rpy="${-90.0 * reflect * deg_to_rad} 0 0" />
       <axis xyz="0 0 1" />
-      <limit lower="${-90.0 * deg_to_rad}" upper="${90.0 * deg_to_rad}" effort="6" velocity="${wrist_max_vel}" />
+      <limit lower="${-90.0 * deg_to_rad}" upper="${90.0 * deg_to_rad}" effort="12" velocity="${wrist_max_vel}" />
       <dynamics friction="${wrist_friction}" damping="0.1"/>
     </joint>
@@ -112,5 +112,5 @@
       <origin xyz="0 0 0" rpy="${90.0 * reflect * deg_to_rad} 0 0" />
       <axis xyz="0 0 1" />
-      <limit lower="${-120.0 * deg_to_rad}" upper="${120.0 * deg_to_rad}" effort="6" velocity="${wrist_max_vel}" />
+      <limit lower="${-120.0 * deg_to_rad}" upper="${120.0 * deg_to_rad}" effort="12" velocity="${wrist_max_vel}" />
       <dynamics friction="${wrist_friction}" damping="0.1"/>
     </joint>

File: reem_description/urdf/torso/torso.urdf.xacro (robot description, xacro)
@@ -42,5 +42,5 @@
       <origin xyz="-0.108 0 0.8725" rpy="0 0 0" />
       <axis xyz="0 0 1" />
-      <limit lower="${-75.0 * deg_to_rad}" upper="${75.0 * deg_to_rad}" effort="11.9" velocity="${torso_max_vel}" />
+      <limit lower="${-75.0 * deg_to_rad}" upper="${75.0 * deg_to_rad}" effort="30" velocity="${torso_max_vel}" />
       <dynamics damping="5.0" friction="1.0"/>
     </joint>
@@ -79,13 +79,13 @@
     <!-- Torso Front Sonar Ring -->
    <!-- torso sonar left -->
-   <xacro:range_reem name="${name}_sonar_14" parent="${name}_2" ros_topic="sonar_torso" update_rate="5" maxRange="0.7" minRange="0.005" fov="0.3491" radiation="ultrasound">
+   <xacro:range_reem name="${name}_sonar_14" parent="${name}_2" ros_topic="sonar_torso" update_rate="5" maxRange="0.7" minRange="0.01" fov="0.3491" radiation="ultrasound">
       <origin xyz="0.185 -0.029 0.075" rpy="0.0 0.0 0.0" />
    </xacro:range_reem>
    <!-- torso sonar right -->
-   <xacro:range_reem name="${name}_sonar_15" parent="${name}_2" ros_topic="sonar_torso" update_rate="5" maxRange="0.7" minRange="0.005" fov="0.3491" radiation="ultrasound">
+   <xacro:range_reem name="${name}_sonar_15" parent="${name}_2" ros_topic="sonar_torso" update_rate="5" maxRange="0.7" minRange="0.01" fov="0.3491" radiation="ultrasound">
       <origin xyz="0.185 -0.029 -0.075" rpy="0.0 0.0 0.0" />
    </xacro:range_reem>
    <!-- torso sonar back -->
-   <xacro:range_reem name="${name}_sonar_13" parent="${name}_2" ros_topic="sonar_torso" update_rate="5" maxRange="0.7" minRange="0.005" fov="0.3491" radiation="ultrasound">
+   <xacro:range_reem name="${name}_sonar_13" parent="${name}_2" ros_topic="sonar_torso" update_rate="5" maxRange="0.7" minRange="0.01" fov="0.3491" radiation="ultrasound">
       <origin xyz="-0.2 -0.149 0.0" rpy="0.0 ${180.0*deg_to_rad} 0.0" />
    </xacro:range_reem>
