Commit message: Tweak joint dynamics (ad hoc).

File: reem_description/urdf/torso/torso.urdf.xacro (robot description, xacro)
@@ -14,7 +14,7 @@
   <include filename="$(find reem_description)/urdf/torso/torso.gazebo.xacro" />
   <include filename="$(find reem_description)/urdf/torso/torso.transmission.xacro" />
-  <xacro:property name="torso_friction" value="20.0" /> <!--TODO: Tune-->
-  <xacro:property name="torso_damping"  value="1.0" />  <!--TODO: Tune-->
-  <xacro:property name="torso_max_vel"  value="0.5" />
+  <xacro:property name="torso_friction" value="10.0" /> <!--TODO: Tune-->
+  <xacro:property name="torso_damping"  value="10.0" />  <!--TODO: Tune-->
+  <xacro:property name="torso_max_vel"  value="1.0" />
   <xacro:macro name="reem_torso" params="name parent">
     <!--************************-->
@@ -59,6 +59,5 @@
         <mass value="13.299" />
         <!-- NOTE: Assuming box with d=0.2, w=0.4, h=0.46 -->
-<!--         <inertia ixx="0.41183"  ixy="0"  ixz="0" iyy="0.22165" iyz="0" izz="0.27884" /> --> <!--TODO: Tune controller!-->
-        <inertia ixx="1"  ixy="0"  ixz="0" iyy="1" iyz="0" izz="1" />
+         <inertia ixx="0.41183"  ixy="0"  ixz="0" iyy="0.22165" iyz="0" izz="0.27884" />
       </inertial>
       <visual>
@@ -77,5 +76,4 @@
       <parent link="${name}_1_link" />
       <child link="${name}_2_link" />
-<!--       <origin xyz="-0 0 0" rpy="${-90.0 * deg_to_rad} 0 0" /> -->
       <origin xyz="-0 0 0.1985" rpy="${-90.0 * deg_to_rad} 0 0" />
       <axis xyz="0 0 1" />

Commit message: Update torso 2 joint position limits.

File: reem_description/urdf/torso/torso.urdf.xacro (robot description, xacro)
@@ -74,5 +74,5 @@
       <origin xyz="-0 0 0.1985" rpy="${-90.0 * deg_to_rad} 0 0" />
       <axis xyz="0 0 1" />
-      <limit lower="${-15.0 * deg_to_rad}" upper="${45.0 * deg_to_rad}" effort="80" velocity="${torso_max_vel}" />
+      <limit lower="${-15.0 * deg_to_rad}" upper="${40.0 * deg_to_rad}" effort="80" velocity="${torso_max_vel}" />
       <dynamics damping="10.0" friction="1.0"/> <!--NOTE: Joint can do 46.2, but set to higher value because of unmodeled springs-->
     </joint>
