Commit message: Bumper visualization geometry made minimal.

File: reem_description/urdf/sensors/bumper.urdf.xacro (robot description, xacro)
@@ -28,9 +28,7 @@
            <origin xyz="0 0 0" rpy="0 0 0" />
            <geometry>
-              <box size="0.05 0.1 0.02"/>
+              <box size="0.001 0.001 0.001"/>
            </geometry>
-           <material name="White">
-                   <color rgba="0 0 0  1.0"/>
-           </material>
+           <material name="White"/>
          </visual>
          <collision>
