Commit message: Add Gazebo material property to laser scanners.

File: reem_description/urdf/sensors/hokuyo_laser_reem.gazebo.xacro (robot description, xacro)
@@ -33,4 +33,5 @@
         </controller:gazebo_ros_laser>
       </sensor:ray>
+      <material>Gazebo/Grey</material>
     </gazebo>
   </xacro:macro>

File: reem_description/urdf/sensors/hokuyo_lx30_laser.gazebo.xacro (robot description, xacro)
@@ -35,4 +35,5 @@
         </controller:gazebo_ros_laser>
       </sensor:ray>
+      <material>Gazebo/Grey</material>
     </gazebo>
   </xacro:macro>

File: reem_description/urdf/sensors/sick_laser_reem.gazebo.xacro (robot description, xacro)
@@ -34,4 +34,5 @@
         </controller:gazebo_ros_laser>
       </sensor:ray>
+      <material>Gazebo/Grey</material>
     </gazebo>
   </xacro:macro>
