Commit message: Resize SICK laser bounding box to a smaller volume.

File: reem_description/urdf/sensors/sick_laser_reem.urdf.xacro (robot description, xacro)
@@ -28,5 +28,5 @@
         <origin xyz="0 0 0" rpy="0 0 0" />
         <geometry>
-          <box size="0.105 0.105 0.152" />
+          <box size="0.105 0.105 0.11" />
         </geometry>
         <material name="DarkGrey" />
@@ -35,5 +35,5 @@
         <origin xyz="0 0 0" rpy="0 0 0" />
         <geometry>
-          <box size="0.105 0.105 0.152" />
+          <box size="0.105 0.105 0.11" />
         </geometry>
       </collision >
