Commit message: Update stereo camera macros.
Patch by Jordi Pages.

File: reem_description/urdf/sensors/stereo_camera.gazebo.xacro (robot description, xacro)
@@ -12,5 +12,5 @@
        xmlns:xacro="http://ros.org/wiki/xacro">
   <!-- this macro is used for creating wide and narrow double stereo camera in simulation -->
-  <xacro:macro name="stereo_camera_gazebo_v0" params="name focal_length hfov image_width image_height">
+  <xacro:macro name="stereo_camera_gazebo_v0" params="name focal_length_left hfov_left focal_length_right hfov_right image_width image_height">
     <gazebo reference="${name}_link">
       <material value="PR2/Blue" />

File: reem_description/urdf/sensors/stereo_camera.urdf.xacro (robot description, xacro)
@@ -21,5 +21,5 @@
   <property name="stereo_rz" value="0.00" />
   <!-- this macro is used for creating wide and narrow double stereo camera links -->
-  <xacro:macro name="stereo_camera_v0" params="name parent focal_length hfov image_format image_width image_height *origin">
+  <xacro:macro name="stereo_camera_v0" params="name parent focal_length_left hfov_left focal_length_right hfov_right image_format image_width image_height *origin">
     <joint name="${name}_frame_joint" type="fixed">
       <insert_block name="origin" />
@@ -59,5 +59,5 @@
     <xacro:stingrayf033c_camera_v0 name="${name}_gazebo_l_stereo_camera" image_format="${image_format}" image_topic_name="${name}/left/image"
                             camera_info_topic_name="${name}/left/camera_info" parent="${name}_link"
-                            hfov="${hfov}" focal_length="${focal_length}"
+                            hfov="${hfov_left}" focal_length="${focal_length_left}"
                             frame_id="${name}_optical_frame" hack_baseline="0"
                             image_width="${image_width}" image_height="${image_height}">
@@ -67,5 +67,5 @@
     <xacro:stingrayf033c_camera_v0 name="${name}_gazebo_r_stereo_camera" image_format="${image_format}" image_topic_name="${name}/right/image"
                             camera_info_topic_name="${name}/right/camera_info" parent="${name}_gazebo_l_stereo_camera_frame"
-                            hfov="${hfov}" focal_length="${focal_length}"
+                            hfov="${hfov_right}" focal_length="${focal_length_right}"
                             frame_id="${name}_optical_frame" hack_baseline="${-stereo_dy}"
                             image_width="${image_width}" image_height="${image_height}">
@@ -73,5 +73,7 @@
     </xacro:stingrayf033c_camera_v0>
     <!-- extensions -->
-    <xacro:stereo_camera_gazebo_v0 name="${name}" focal_length="${focal_length}" hfov="${hfov}"
+    <xacro:stereo_camera_gazebo_v0 name="${name}"
+                                   focal_length_left="${focal_length_left}" hfov_left="${hfov_left}"
+                                   focal_length_right="${focal_length_right}" hfov_right="${hfov_right}"
                                    image_width="${image_width}" image_height="${image_height}"/>
   </xacro:macro>
