Commit message: Update sensor description to work in ROS fuerte.

File: reem_description/urdf/sensors/back_camera.gazebo.xacro (robot description, xacro)
@@ -15,9 +15,9 @@
     <gazebo reference="${name}_link">
       <material value="PR2/Blue" />
-      <turnGravityOff value="true" />
+      <turnGravityOff value="false" />
     </gazebo>
     <gazebo reference="${name}_optical_frame">
       <material value="Gazebo/White" />
-      <turnGravityOff value="true" />
+      <turnGravityOff value="false" />
     </gazebo>
   </xacro:macro>

File: reem_description/urdf/sensors/bumper.gazebo.xacro (robot description, xacro)
@@ -12,17 +12,17 @@
        xmlns:xacro="http://ros.org/wiki/xacro">
   <xacro:macro name="bumper_reem_gazebo" params="name ros_topic update_rate">
-   <gazebo reference="${name}_link">
+     <gazebo reference="${name}_link">
         <selfCollide>false</selfCollide>
-        <sensor:contact name="{name}_contact">
-           <geom>base_footprint_geom_${name}_link</geom>
-           <updateRate>100.0</updateRate>
-             <controller:reem_bumper_gazebo name="reem_gazebo_bumper_controller1" plugin="libreem_bumper_gazebo.so">
-             <alwaysOn>true</alwaysOn>
-             <updateRate>100.0</updateRate>
-             <frameId>${name}_link</frameId>
-             <bumperTopicName>${ros_topic}</bumperTopicName>
-             <interface:bumper name="${name}_iface1" />
-           </controller:reem_bumper_gazebo>
-       </sensor:contact>
+        <sensor:contact name="contact_sensor">
+          <geom>${name}_link_geom</geom>
+          <updateRate>20.0</updateRate>
+          <controller:reem_bumper_gazebo name="gazebo_reem_ros_bumper" plugin="libreem_bumper_gazebo.so">
+              <alwaysOn>true</alwaysOn>
+              <updateRate>20.0</updateRate>
+              <frameName>${name}_link</frameName>
+              <bumperTopicName>${ros_topic}</bumperTopicName>
+          <interface:bumper name="bumper_iface" />
+          </controller:reem_bumper_gazebo>
+      </sensor:contact>
     </gazebo>
   </xacro:macro>

File: reem_description/urdf/sensors/hokuyo_laser_reem.gazebo.xacro (robot description, xacro)
@@ -31,4 +31,5 @@
           <frameName>${name}_link</frameName>
           <interface:laser name="gazebo_ros_${name}_iface" />
+          <hokuyoMinIntensity>101.0</hokuyoMinIntensity>
         </controller:gazebo_ros_laser>
       </sensor:ray>

File: reem_description/urdf/sensors/hokuyo_laser_reem.urdf.xacro (robot description, xacro)
@@ -39,8 +39,4 @@
       </collision>
     </link>
-    <gazebo reference="${name}_link">
-		  <material>Gazebo/Red</material>
-		  <!-- <turnGravityOff>false</turnGravityOff> -->
-    </gazebo>
     <!-- gazebo extensions -->
     <xacro:hokuyo_laser_reem_gazebo name="${name}" ros_topic="${ros_topic}" update_rate="${update_rate}" min_angle="${min_angle}" max_angle="${max_angle}" />

File: reem_description/urdf/sensors/hokuyo_lx30_laser.gazebo.xacro (robot description, xacro)
@@ -33,4 +33,5 @@
           <frameName>${name}_link</frameName>
           <interface:laser name="gazebo_ros_${name}_iface" />
+          <hokuyoMinIntensity>101.0</hokuyoMinIntensity>
         </controller:gazebo_ros_laser>
       </sensor:ray>

File: reem_description/urdf/sensors/range.gazebo.xacro (robot description, xacro)
@@ -14,5 +14,4 @@
     <gazebo reference="${name}_link">
       <sensor:ray name="${name}">
-        <!-- displayRays>fan</displayRays -->
         <rayCount>5</rayCount>
         <rangeCount>5</rangeCount>
@@ -29,10 +28,8 @@
         <controller:gazebo_ros_sonar name="gazebo_ros_${name}_controller" plugin="libgazebo_ros_sonar.so">
           <gaussianNoise>0.005</gaussianNoise>
-          <alwaysOn>true</alwaysOn>
-          <updateRate>${update_rate}</updateRate>
           <topicName>${ros_topic}</topicName>
           <frameId>${name}_link</frameId>
+          <fov>${fov}</fov>
           <radiation>${radiation}</radiation>
-          <fov>${fov}</fov>
         </controller:gazebo_ros_sonar>
       </sensor:ray>

File: reem_description/urdf/sensors/sick_laser_reem.gazebo.xacro (robot description, xacro)
@@ -32,4 +32,5 @@
           <frameName>${name}_link</frameName>
           <interface:laser name="gazebo_ros_${name}_iface" />
+          <hokuyoMinIntensity>101.0</hokuyoMinIntensity>
         </controller:gazebo_ros_laser>
       </sensor:ray>

File: reem_description/urdf/sensors/sick_laser_reem.urdf.xacro (robot description, xacro)
@@ -40,6 +40,4 @@
     </link>
     <gazebo reference="${name}_link">
-		  <material>Gazebo/Red</material>
-		  <!-- <turnGravityOff>false</turnGravityOff> -->
     </gazebo>
     <!-- gazebo extensions -->

File: reem_description/urdf/sensors/stereo_camera.gazebo.xacro (robot description, xacro)
@@ -15,9 +15,9 @@
     <gazebo reference="${name}_link">
       <material value="PR2/Blue" />
-      <turnGravityOff value="true" />
+      <turnGravityOff value="false" />
     </gazebo>
     <gazebo reference="${name}_optical_frame">
       <material value="Gazebo/White" />
-      <turnGravityOff value="true" />
+      <turnGravityOff value="false" />
     </gazebo>
   </xacro:macro>

File: reem_description/urdf/sensors/stereo_camera.urdf.xacro (robot description, xacro)
@@ -30,7 +30,9 @@
     <link name="${name}_link">
       <inertial>
-        <mass value="0.1" />
+        <mass value="0.01" />
         <origin xyz="0 0 0" rpy="0 0 0" />
-        <inertia ixx="0.01"  ixy="0"  ixz="0" iyy="0.01"  iyz="0"  izz="0.01" /> <!-- this inertia is made up for now. -->
+        <inertia ixx="0"  ixy="0"  ixz="0"
+                 iyy="0"  iyz="0"
+                 izz="0" /> <!-- this inertia is made up for now. -->
       </inertial>
       <visual>
@@ -55,8 +57,16 @@
     </joint>
     <!-- optical frame for the stereo camera, with z-forward notation, this is the frame stereo camera images users should refer to -->
-    <link name="${name}_optical_frame" type="camera"/>
+    <link name="${name}_optical_frame" type="camera">
+      <inertial>
+        <mass value="0.01" />
+        <origin xyz="0 0 0" rpy="0 0 0" />
+        <inertia ixx="0"  ixy="0"  ixz="0"
+                 iyy="0"  iyz="0"
+                 izz="0" /> <!-- this inertia is made up for now. -->
+      </inertial>
+    </link>
     <!-- stereo left camera -->
-    <xacro:stingrayf033c_camera_v0 name="${name}_gazebo_l_stereo_camera" image_format="${image_format}" image_topic_name="${name}/left/image"
-                            camera_info_topic_name="${name}/left/camera_info" parent="${name}_link"
+    <xacro:stingrayf033c_camera_v0 name="${name}_gazebo_l_stereo_camera" image_format="${image_format}" image_topic_name="/${name}/left/image"
+                            camera_info_topic_name="/${name}/left/camera_info" parent="${name}_link"
                             hfov="${hfov_left}" focal_length="${focal_length_left}"
                             frame_id="${name}_optical_frame" hack_baseline="0"
@@ -65,6 +75,6 @@
     </xacro:stingrayf033c_camera_v0>
     <!-- stereo right camera -->
-    <xacro:stingrayf033c_camera_v0 name="${name}_gazebo_r_stereo_camera" image_format="${image_format}" image_topic_name="${name}/right/image"
-                            camera_info_topic_name="${name}/right/camera_info" parent="${name}_gazebo_l_stereo_camera_frame"
+    <xacro:stingrayf033c_camera_v0 name="${name}_gazebo_r_stereo_camera" image_format="${image_format}" image_topic_name="/${name}/right/image"
+                            camera_info_topic_name="/${name}/right/camera_info" parent="${name}_gazebo_l_stereo_camera_frame"
                             hfov="${hfov_right}" focal_length="${focal_length_right}"
                             frame_id="${name}_optical_frame" hack_baseline="${-stereo_dy}"

File: reem_description/urdf/sensors/stingrayf033c_camera.gazebo.xacro (robot description, xacro)
@@ -13,32 +13,32 @@
   <xacro:macro name="stingrayf033c_camera_gazebo_v0" params="name image_format image_topic_name camera_info_topic_name hfov focal_length frame_id hack_baseline image_width image_height">
     <gazebo reference="${name}_frame">
-      <sensor:camera name="${name}_sensor">
-        <imageSize>${image_width} ${image_height}</imageSize>
-        <imageFormat>${image_format}</imageFormat>
-        <hfov>${hfov}</hfov>
-        <nearClip>0.1</nearClip>
-        <farClip>100</farClip>
+    <sensor:camera name="${name}_sensor">
+      <imageFormat>R8G8B8</imageFormat>
+      <imageSize>${image_width} ${image_height}</imageSize>
+      <hfov>${hfov}</hfov>
+      <nearClip>0.1</nearClip>
+      <farClip>100</farClip>
+      <updateRate>25.0</updateRate>
+      <controller:gazebo_ros_prosilica name="${name}_controller" plugin="libgazebo_ros_prosilica.so">
+        <alwaysOn>true</alwaysOn>
         <updateRate>25.0</updateRate>
-        <controller:gazebo_ros_camera name="${name}_controller" plugin="libgazebo_ros_camera.so">
-          <alwaysOn>true</alwaysOn>
-          <updateRate>25.0</updateRate>
-          <imageTopicName>${image_topic_name}</imageTopicName>
-          <cameraInfoTopicName>${camera_info_topic_name}</cameraInfoTopicName>
-          <frameName>${frame_id}</frameName>
-          <hackBaseline>${hack_baseline}</hackBaseline>
-          <CxPrime>${(image_width+1)/2}</CxPrime>
-          <Cx>${(image_width+1)/2}</Cx>
-          <Cy>${(image_height+1)/2}</Cy>
-          <focal_length>${focal_length}</focal_length>
-          <distortion_k1>0.00000001</distortion_k1>  <!-- -0.26932955  -->
-          <distortion_k2>0.00000001</distortion_k2>  <!--  0.055528346 -->
-          <distortion_k3>0.00000001</distortion_k3>
-          <distortion_t1>0.00000001</distortion_t1>  <!--  0.00005650  -->
-          <distortion_t2>0.00000001</distortion_t2>  <!--  0.00092793  -->
-          <interface:camera name="${name}_iface" />
-        </controller:gazebo_ros_camera>
-      </sensor:camera>
-      <turnGravityOff>true</turnGravityOff>
-      <material>PR2/Blue</material>
+        <cameraName>${name}</cameraName>
+        <hackBaseline>${hack_baseline}</hackBaseline>
+        <imageTopicName>${image_topic_name}</imageTopicName>
+        <cameraInfoTopicName>${camera_info_topic_name}</cameraInfoTopicName>
+        <!-- <pollServiceName>request_image</pollServiceName> -->
+        <frameName>${frame_id}</frameName>
+        <CxPrime>${(image_width+1)/2}</CxPrime>
+        <Cx>${(image_width+1)/2}</Cx>
+        <Cy>${(image_height+1)/2}</Cy>
+        <focalLength>${focal_length}</focalLength> <!-- image_width / (2*tan(hfov_radian /2)) -->
+        <distortionK1>0.0</distortionK1>
+        <distortionK2>0.0</distortionK2>
+        <distortionK3>0.0</distortionK3>
+        <distortionT1>0.0</distortionT1>
+        <distortionT2>0.0</distortionT2>
+      </controller:gazebo_ros_prosilica>
+    </sensor:camera>
+    <material value="Gazebo/Black" />
     </gazebo>
   </xacro:macro>

File: reem_description/urdf/sensors/stingrayf033c_camera.urdf.xacro (robot description, xacro)
@@ -25,7 +25,7 @@
         <mass value="0.01" />
         <origin xyz="0 0 0" />
-        <inertia ixx="0.001"  ixy="0.0"  ixz="0.0"
-                 iyy="0.001"  iyz="0.0"
-                 izz="0.001" />
+        <inertia ixx="0"  ixy="0.0"  ixz="0.0"
+                 iyy="0"  iyz="0.0"
+                 izz="0" />
       </inertial>
       <visual>
@@ -35,4 +35,5 @@
         </geometry>
       </visual>
+      <!--
       <collision>
         <origin xyz="0 0 0" rpy="0 0 0"/>
@@ -41,4 +42,5 @@
         </geometry>
       </collision>
+      -->
     </link>
     <joint name="${name}_optical_frame_joint" type="fixed">
@@ -47,5 +49,13 @@
       <child link="${name}_optical_frame"/>
     </joint>
-    <link name="${name}_optical_frame"/>
+    <link name="${name}_optical_frame">
+      <inertial>
+        <mass value="0.1" />
+        <origin xyz="0 0 0" />
+        <inertia ixx="0"  ixy="0.0"  ixz="0.0"
+                 iyy="0"  iyz="0.0"
+                 izz="0" />
+      </inertial>
+    </link>
     <!-- extensions -->
     <xacro:stingrayf033c_camera_gazebo_v0 name="${name}" image_format="${image_format}" image_topic_name="${image_topic_name}"
