Commit message: Update ASUS Xtion Pro Live model.
- No longer compensate mesh non-standards compliance in URDF:
  - Scale mesh to meters.
  - Re-orient mesh origin.

- Make visualization texture darker.

- Use box collision geometry instead of a more expensive convex decomposition.
.

File: reem_description/urdf/sensors/xtion_withoutbase.urdf.xacro (robot description, xacro)
@@ -40,23 +40,8 @@
                  izz="0.01" />
       </inertial>
-    </link>
-    <!-- Visual mesh and collision geometry -->
-    <joint name="${name}_visual_joint" type="fixed">
-      <origin xyz="0.0 0.0 0.0" rpy="${M_PI/2} 0.0 ${M_PI/2}" />
-      <parent link="${name}_link"/>
-      <child link="${name}_visual_link"/>
-    </joint>
-    <link name="${name}_visual_link">
-      <inertial>
-        <mass value="0.1" />
-        <origin xyz="0 0 0" rpy="0 0 0"/>
-        <inertia ixx="0.01"  ixy="0.0"  ixz="0.0"
-                 iyy="0.01"  iyz="0.0"
-                 izz="0.01" />
-      </inertial>
       <visual>
         <origin xyz="0 0 0" rpy="0 0 0"/>
         <geometry>
-          <mesh filename="package://reem_description/meshes/sensors/xtion/xtion_pro_live.dae" scale="0.001 0.001 0.001" />
+          <mesh filename="package://reem_description/meshes/sensors/xtion/xtion_pro_live.dae" />
         </geometry>
         <material name="gray">
@@ -65,8 +50,7 @@
       </visual>
       <collision>
-        <origin xyz="0.0 0.0 0" rpy="0 0 0"/>
+        <origin xyz="-0.0075 0.0025 0" rpy="0 0 0"/>
         <geometry>
-          <!--<box size="0.19 0.03 0.04"/> -->
-          <mesh filename="package://reem_description/meshes/sensors/xtion/xtion_pro_live_collision.stl" scale="0.0011 0.0011 0.0011" />
+          <box size="0.04 0.185 0.03"/>
         </geometry>
       </collision>
