Commit message: Change sensor material properties.

File: reem_description/urdf/sensors/openni.gazebo.xacro (robot description, xacro)
@@ -43,5 +43,4 @@
         </controller:gazebo_ros_openni_kinect>
       </sensor:camera>
-      <material value="Gazebo/Red" />
     </gazebo>
   </xacro:macro>
@@ -72,5 +71,4 @@
         </controller:gazebo_ros_openni_kinect>
       </sensor:camera>
-      <material value="Gazebo/Red" />
     </gazebo>
   </xacro:macro>

File: reem_description/urdf/sensors/xtion_pro_live.urdf.xacro (robot description, xacro)
@@ -45,5 +45,5 @@
           <mesh filename="package://reem_description/meshes/sensors/xtion_pro_live/xtion_pro_live.dae" />
         </geometry>
-        <material name="gray">
+        <material name="Grey">
           <color rgba="0.5 0.5 0.5 1"/>
         </material>
