Commit message: Workaround Gazebo 1.0.2 bug with RGBD sensors.
There seems to be interference between the collision geometry and the camera image
and generated pointclouds of the ASUS xtion pro live sensor.

File: reem_description/urdf/sensors/xtion_pro_live.urdf.xacro (robot description, xacro)
@@ -50,5 +50,5 @@
       </visual>
       <collision>
-        <origin xyz="-0.0075 0.0025 0" rpy="0 0 0"/>
+        <origin xyz="-0.02 0.0025 0" rpy="0 0 0"/> <!--TODO: Tune x coordinate. In Gazebo 1.0.2 collision geom conflicts with RGBD sensor, WTF?!-->
         <geometry>
           <box size="0.04 0.185 0.03"/>

Commit message: Silence Gazebo startup warnings and errors.
- Add dummy inertia to links.
- Manually add missing expected collada atttribute to transparency element.

File: reem_description/urdf/sensors/xtion_pro_live.urdf.xacro (robot description, xacro)
@@ -34,9 +34,9 @@
     <link name="${name}_link">
       <inertial>
-        <mass value="0.1" />
+        <mass value="0.01" />
         <origin xyz="0 0 0" rpy="0 0 0"/>
-        <inertia ixx="0.01"  ixy="0.0"  ixz="0.0"
-                 iyy="0.01"  iyz="0.0"
-                 izz="0.01" />
+        <inertia ixx="0.0"  ixy="0.0"  ixz="0.0"
+                 iyy="0.0"  iyz="0.0"
+                 izz="0.0" />
       </inertial>
       <visual>
@@ -67,9 +67,9 @@
       <!-- This link is the reference for the IR sensor in Gazebo, so it has inertia properties -->
       <inertial>
-        <mass value="0.1" />
+        <mass value="0.01" />
         <origin xyz="0 0 0" rpy="0 0 0"/>
-        <inertia ixx="0.01"  ixy="0.0"  ixz="0.0"
-                 iyy="0.01"  iyz="0.0"
-                 izz="0.01" />
+        <inertia ixx="0.0"  ixy="0.0"  ixz="0.0"
+                 iyy="0.0"  iyz="0.0"
+                 izz="0.0" />
       </inertial>
     </link>
@@ -80,5 +80,13 @@
       <child link="${name}_ir_optical_frame"/>
     </joint>
-    <link name="${name}_ir_optical_frame"/>
+    <link name="${name}_ir_optical_frame">
+      <inertial>
+        <mass value="0.01" />
+        <origin xyz="0 0 0" rpy="0 0 0"/>
+        <inertia ixx="0.0"  ixy="0.0"  ixz="0.0"
+                 iyy="0.0"  iyz="0.0"
+                 izz="0.0" />
+      </inertial>
+    </link>
     <!-- OpenNI IR sensor Gazebo extensions -->
     <xacro:openni_ir_gazebo_v0 link_name="${name}_ir_link" frame_name="${name}_ir_optical_frame" camera_name="${name}" />
@@ -93,9 +101,9 @@
       <!-- This link is the reference for the RGB sensor in Gazebo, so it has inertia properties -->
       <inertial>
-        <mass value="0.1" />
+        <mass value="0.01" />
         <origin xyz="0 0 0" rpy="0 0 0"/>
-        <inertia ixx="0.01"  ixy="0.0"  ixz="0.0"
-                 iyy="0.01"  iyz="0.0"
-                 izz="0.01" />
+        <inertia ixx="0.0"  ixy="0.0"  ixz="0.0"
+                 iyy="0.0"  iyz="0.0"
+                 izz="0.0" />
       </inertial>
     </link>
@@ -106,5 +114,13 @@
       <child link="${name}_rgb_optical_frame"/>
     </joint>
-    <link name="${name}_rgb_optical_frame"/>
+    <link name="${name}_rgb_optical_frame">
+       <inertial>
+        <mass value="0.01" />
+        <origin xyz="0 0 0" rpy="0 0 0"/>
+        <inertia ixx="0.0"  ixy="0.0"  ixz="0.0"
+                 iyy="0.0"  iyz="0.0"
+                 izz="0.0" />
+      </inertial>
+    </link>
     <!-- OpenNI RGB sensor Gazebo extensions -->
     <xacro:openni_rgb_gazebo_v0 link_name="${name}_rgb_link" frame_name="${name}_rgb_optical_frame" camera_name="${name}" />

Commit message: Fixed ASUS Xtion collision geometry. Due to a Gazebo bug, all visual/collision geometry must have zero origin. Added a new, simplified STL collision mesh instead.

File: reem_description/urdf/sensors/xtion_pro_live.urdf.xacro (robot description, xacro)
@@ -50,7 +50,7 @@
       </visual>
       <collision>
-        <origin xyz="-0.02 0.0025 0" rpy="0 0 0"/> <!--TODO: Tune x coordinate. In Gazebo 1.0.2 collision geom conflicts with RGBD sensor, WTF?!-->
+        <origin xyz="0 0 0" rpy="0 0 0"/>
         <geometry>
-          <box size="0.04 0.185 0.03"/>
+          <mesh filename="package://reem_description/meshes/sensors/xtion_pro_live/xtion_pro_live_collision.stl" />
         </geometry>
       </collision>

Commit message: Fix RGBD collision geometry origin.

File: reem_description/urdf/sensors/xtion_pro_live.urdf.xacro (robot description, xacro)
@@ -48,5 +48,5 @@
       </visual>
       <collision>
-        <origin xyz="-0.02 0.0025 0" rpy="0 0 0"/> <!--TODO: Tune x coordinate. In Gazebo 1.0.2 collision geom conflicts with RGBD sensor, WTF?!-->
+        <origin xyz="-0.01 0.0025 0" rpy="0 0 0"/>
         <geometry>
           <box size="0.04 0.185 0.03"/>
