Commit message: Revert inclined laser joint type to fixed.

File: reem_description/urdf/sensors/hokuyo_laser_reem.urdf.xacro (robot description, xacro)
@@ -34,5 +34,5 @@
       </collision>
     </link>
-    <joint name="${name}_joint" type="revolute">
+    <!--joint name="${name}_joint" type="revolute">
         <origin xyz="0.04 0 0.745" rpy="-0.03 ${52 * deg_to_rad} -0.05" />
         <axis xyz="0 1 0"/>
@@ -46,6 +46,12 @@
       <joint name="${name}_joint" />
       <mechanicalReduction>1.0</mechanicalReduction>
-    </transmission>
-    <!-- gazebo extensions -->
+    </transmission-->
+    <joint name="${name}_joint" type="fixed">
+      <axis xyz="0 1 0" />
+      <insert_block name="origin" />
+      <parent link="base_link"/>
+      <child link="${name}_link"/>
+    </joint>
+<!-- gazebo extensions -->
     <xacro:hokuyo_reem_laser_gazebo name="${name}" ros_topic="${ros_topic}" update_rate="${update_rate}" min_angle="${min_angle}" max_angle="${max_angle}" />
   </xacro:macro>
