Commit message: Use more descriptive head depth sensor name.
- Remove hardcoded _rgbd suffix, let name parameter set it.

- Name parameter changed to head_mount_xtion, instead of head_mount_rgbd, as
  confusing topic names were appearing, eg. head_mount_rgbd_rgb.

File: reem_description/robots/reem_xtion.urdf.xacro (robot description, xacro)
@@ -56,9 +56,9 @@
   </xacro:back_camera_v0>-->
   <!-- head-mounted ASUS Xtion Pro Live -->
-  <xacro:xtion_withoutbase parent="head_2_link" name="head_mount" > <!-- name is appended to create link and topic names -->
+  <xacro:xtion_withoutbase parent="head_2_link" name="head_mount_xtion" > <!-- name is appended to create link and topic names -->
      <origin xyz="0.056 -0.252 0.0" rpy="${M_PI/2} 0.0 0.34906" /> <!-- 0.252   = height above neck joint
                                                                         0.34906 = pitch angle downwards   -->
-     <origin xyz="${cal_head_mount_rgbd_x} ${cal_head_mount_rgbd_y} ${cal_head_mount_rgbd_z}"
-             rpy="${-M_PI/2+cal_head_mount_rgbd_roll} ${0.0+cal_head_mount_rgbd_pitch} ${-M_PI/2+cal_head_mount_rgbd_yaw}" />
+     <origin xyz="${cal_head_mount_xtion_x} ${cal_head_mount_xtion_y} ${cal_head_mount_xtion_z}"
+             rpy="${-M_PI/2+cal_head_mount_xtion_roll} ${0.0+cal_head_mount_xtion_pitch} ${-M_PI/2+cal_head_mount_xtion_yaw}" />
   </xacro:xtion_withoutbase>
 </robot>

File: reem_description/urdf/sensors/calibration.xacro (robot description, xacro)
@@ -12,11 +12,11 @@
   <!-- Head-mounted ASUS Xtion Pro Live -->
   <!-- These calibration values affect 2 frames:
-         (name)_rgbd_ir_optical_frame
-         (name)_rgbd_rgb_optical_frame              -->
-  <property name="cal_head_mount_rgbd_x" value="0.0" />
-  <property name="cal_head_mount_rgbd_y" value="0.0" />
-  <property name="cal_head_mount_rgbd_z" value="0.0" />
-  <property name="cal_head_mount_rgbd_roll"  value="0.0" />
-  <property name="cal_head_mount_rgbd_pitch" value="0.0" />
-  <property name="cal_head_mount_rgbd_yaw"   value="0.0" />
+         (name)_xtion_ir_optical_frame
+         (name)_xtion_rgb_optical_frame              -->
+  <property name="cal_head_mount_xtion_x"     value="0.0" />
+  <property name="cal_head_mount_xtion_y"     value="0.0" />
+  <property name="cal_head_mount_xtion_z"     value="0.0" />
+  <property name="cal_head_mount_xtion_roll"  value="0.0" />
+  <property name="cal_head_mount_xtion_pitch" value="0.0" />
+  <property name="cal_head_mount_xtion_yaw"   value="0.0" />
 </robot>

File: reem_description/urdf/sensors/xtion_withoutbase.urdf.xacro (robot description, xacro)
@@ -42,10 +42,10 @@
     </link>
     <!-- Visual mesh and collision geometry -->
-    <joint name="${name}_rgbd_visual_joint" type="fixed">
+    <joint name="${name}_visual_joint" type="fixed">
       <origin xyz="0.0 0.0 0.0" rpy="${M_PI/2} 0.0 ${M_PI/2}" />
       <parent link="${name}_link"/>
-      <child link="${name}_rgbd_visual_link"/>
+      <child link="${name}_visual_link"/>
     </joint>
-    <link name="${name}_rgbd_visual_link">
+    <link name="${name}_visual_link">
       <inertial>
         <mass value="0.1" />
@@ -73,12 +73,12 @@
     </link>
     <!-- Xtion IR sensor physical attachment -->
-    <joint name="${name}_rgbd_ir_joint" type="fixed">
+    <joint name="${name}_ir_joint" type="fixed">
       <!-- This relates the IR sensor to the Xtion base link -->
       <!-- 4.8 cm because sensors are offset to right, from center -->
       <origin xyz="0 0.048 0" rpy="0 0 0"/>
       <parent link="${name}_link"/>
-      <child link="${name}_rgbd_ir_link"/>
+      <child link="${name}_ir_link"/>
     </joint>
-    <link name="${name}_rgbd_ir_link">
+    <link name="${name}_ir_link">
       <!-- This link is the reference for the IR sensor in Gazebo, so it has inertia properties -->
       <inertial>
@@ -91,20 +91,20 @@
     </link>
     <!-- Xtion IR sensor frame -->
-    <joint name="${name}_rgbd_ir_optical_frame_joint" type="fixed">
+    <joint name="${name}_ir_optical_frame_joint" type="fixed">
       <insert_block name="calibration_origin" /> <!-- macro argument -->
-      <parent link="${name}_rgbd_ir_link"/>
-      <child link="${name}_rgbd_ir_optical_frame"/>
+      <parent link="${name}_ir_link"/>
+      <child link="${name}_ir_optical_frame"/>
     </joint>
-    <link name="${name}_rgbd_ir_optical_frame"/>
+    <link name="${name}_ir_optical_frame"/>
     <!-- OpenNI IR sensor Gazebo extensions -->
-    <xacro:openni_ir_gazebo_v0 link_name="${name}_rgbd_ir_link" frame_name="${name}_rgbd_ir_optical_frame" camera_name="${name}_rgbd" />
+    <xacro:openni_ir_gazebo_v0 link_name="${name}_ir_link" frame_name="${name}_ir_optical_frame" camera_name="${name}" />
     <!-- Xtion RGB sensor physical attachment -->
-    <joint name="${name}_rgbd_rgb_joint" type="fixed">
+    <joint name="${name}_rgb_joint" type="fixed">
       <!-- The measured distance from RGB lens back to IR lens, approx 2.5cm, but PR2 is using 3.0cm -->
       <origin xyz="0 -0.025 0" rpy="0 0 0"/>
-      <parent link="${name}_rgbd_ir_link"/>
-      <child link="${name}_rgbd_rgb_link"/>
+      <parent link="${name}_ir_link"/>
+      <child link="${name}_rgb_link"/>
     </joint>
-    <link name="${name}_rgbd_rgb_link" >
+    <link name="${name}_rgb_link" >
       <!-- This link is the reference for the RGB sensor in Gazebo, so it has inertia properties -->
       <inertial>
@@ -117,12 +117,12 @@
     </link>
     <!-- Xtion RGB sensor frame -->
-    <joint name="${name}_rgbd_rgb_optical_frame_joint" type="fixed">
+    <joint name="${name}_rgb_optical_frame_joint" type="fixed">
       <insert_block name="calibration_origin" /> <!-- macro argument -->
-      <parent link="${name}_rgbd_rgb_link"/>
-      <child link="${name}_rgbd_rgb_optical_frame"/>
+      <parent link="${name}_rgb_link"/>
+      <child link="${name}_rgb_optical_frame"/>
     </joint>
-    <link name="${name}_rgbd_rgb_optical_frame"/>
+    <link name="${name}_rgb_optical_frame"/>
     <!-- OpenNI RGB sensor Gazebo extensions -->
-    <xacro:openni_rgb_gazebo_v0 link_name="${name}_rgbd_rgb_link" frame_name="${name}_rgbd_rgb_optical_frame" camera_name="${name}_rgbd" />
+    <xacro:openni_rgb_gazebo_v0 link_name="${name}_rgb_link" frame_name="${name}_rgb_optical_frame" camera_name="${name}" />
   </xacro:macro>
 </robot>

Commit message: Remove code duplication.
When launching reem with the head-mounted ASUS Xtion Pro Live, include the file
containing the stock REEM, instead of duplicating its contents.

File: reem_description/robots/reem_xtion.urdf.xacro (robot description, xacro)
@@ -6,7 +6,4 @@
   To view a copy of this license, visit http://creativecommons.org/licenses/by-nc-nd/3.0/ or send a letter to
   Creative Commons, 444 Castro Street, Suite 900, Mountain View, California, 94041, USA.
-  REEM robot, with
-    - stereo cameras
-    - ASUS Xtion Pro Live (head-mounted)
 -->
 <robot  xmlns:xacro="http://www.ros.org/wiki/xacro"
@@ -15,50 +12,17 @@
         xmlns:interface="http://playerstage.sourceforge.net/gazebo/xmlschema/#interface"
         name="reem" >
-  <!-- The following included files set up definitions of parts of the robot body -->
-  <!-- Base -->
-  <include filename="$(find reem_description)/urdf/base/base.urdf.xacro" />
-  <!-- Torso -->
-  <include filename="$(find reem_description)/urdf/torso/torso.urdf.xacro" />
-  <!-- Head -->
-  <include filename="$(find reem_description)/urdf/head/head.urdf.xacro" />
-  <!-- Arm -->
-  <include filename="$(find reem_description)/urdf/arm/arm.urdf.xacro" />
-  <!-- Hand -->
-  <include filename="$(find reem_description)/urdf/hand/hand.urdf.xacro" />
-  <!-- Camera sensors -->
-  <include filename="$(find reem_description)/urdf/sensors/stereo_camera.urdf.xacro" />
-  <!--<include filename="$(find reem_description)/urdf/sensors/back_camera.urdf.xacro" /> -->
-  <!-- RGBD sensors -->
+  <!-- Stock REEM robot -->
+  <include filename="$(find reem_description)/robots/reem.urdf.xacro" />
+  <!-- Head-mounted ASUS Xtion Pro Live -->
   <include filename="$(find reem_description)/urdf/sensors/xtion_withoutbase.urdf.xacro" />
-  <!-- Generic simulator_gazebo plugins -->
-  <include filename="$(find reem_description)/gazebo/gazebo.urdf.xacro" />
-  <!-- Materials for visualization -->
-  <include filename="$(find reem_description)/urdf/materials.urdf.xacro" />
-  <!-- Now we can start using the macros included above to define the actual robot -->
-  <xacro:reem_base  name="base"/>
-  <xacro:reem_cargo  name="base"/>
-  <xacro:reem_torso name="torso" parent="base_link"/>
-  <xacro:reem_head  name="head"  parent="torso_2_link"/>
-  <!-- The reflect parameter takes the value 1 or -1 to respectively distinguish right from left side in expressions -->
-  <xacro:reem_arm name="arm" parent="torso_2_link" side="right" reflect="1.0"  />
-  <xacro:reem_arm name="arm" parent="torso_2_link" side="left"  reflect="-1.0" />
-  <xacro:reem_hand name="hand" parent="arm_right_tool_link" side="right" reflect="1.0"  />
-  <xacro:reem_hand name="hand" parent="arm_left_tool_link"  side="left"  reflect="-1.0" />
-  <!-- stereo camera -->
-  <!-- IMPORTANT: focal_length = image_width/(2tan(hfov/2)) -->
-  <xacro:stereo_camera_v0 parent="head_2_link" name="stereo" focal_length_left="459.838918" hfov_left="71" focal_length_right="459.838918" hfov_right="71" image_format="B8G8R8" image_width="656" image_height="492">
-    <!-- The following transformations expresses the pose of the stereo_link (X pointing forward, Z upwards and Y leftwards, contrary to the stereo_optical_link which has Z pointing forward) wrt  head_2_link. -->
-     <origin xyz="0.08203  -0.09558  0.04132" rpy="1.56293 -0.00855922 -0.0201307" />
-  </xacro:stereo_camera_v0>
-  <!--<xacro:back_camera_v0 parent="torso_2_link" name="back" focal_length="557" hfov="75" image_format="B8G8R8" image_width="640" image_height="480" >  -->
-    <!-- The following transformations expresses the pose of the back_link (X pointing forward, Z upwards and Y leftwards, contrary to the stereo_optical_link which has Z pointing forward) wrt  torso_2_link. -->
-    <!--<origin xyz="-0.140 -0.302 -0.000" rpy="-3.142 1.571 0.211" />
-  </xacro:back_camera_v0>-->
-  <!-- head-mounted ASUS Xtion Pro Live -->
   <xacro:xtion_withoutbase parent="head_2_link" name="head_mount_xtion" > <!-- name is appended to create link and topic names -->
      <origin xyz="0.056 -0.252 0.0" rpy="${M_PI/2} 0.0 0.34906" /> <!-- 0.252   = height above neck joint
                                                                         0.34906 = pitch angle downwards   -->
-     <origin xyz="${cal_head_mount_xtion_x} ${cal_head_mount_xtion_y} ${cal_head_mount_xtion_z}"
-             rpy="${-M_PI/2+cal_head_mount_xtion_roll} ${0.0+cal_head_mount_xtion_pitch} ${-M_PI/2+cal_head_mount_xtion_yaw}" />
+     <origin xyz="${cal_head_mount_xtion_x}
+                  ${cal_head_mount_xtion_y}
+                  ${cal_head_mount_xtion_z}"
+             rpy="${-M_PI/2+cal_head_mount_xtion_roll}
+                  ${0.0+cal_head_mount_xtion_pitch}
+                  ${-M_PI/2+cal_head_mount_xtion_yaw}" />
   </xacro:xtion_withoutbase>
 </robot>
