Commit message: Rename ASUS sensor files and folders consistently.

File: reem_description/robots/reem_xtion_pro_live.urdf.xacro (robot description, xacro)
@@ -15,6 +15,6 @@
   <include filename="$(find reem_description)/robots/reem.urdf.xacro" />
   <!-- Head-mounted ASUS Xtion Pro Live -->
-  <include filename="$(find reem_description)/urdf/sensors/xtion_withoutbase.urdf.xacro" />
-  <xacro:xtion_withoutbase parent="head_2_link" name="head_mount_xtion" > <!-- name is appended to create link and topic names -->
+  <include filename="$(find reem_description)/urdf/sensors/xtion_pro_live.urdf.xacro" />
+  <xacro:xtion_pro_live parent="head_2_link" name="head_mount_xtion" > <!-- name is appended to create link and topic names -->
      <origin xyz="0.056 -0.252 0.0" rpy="${M_PI/2} 0.0 0.34906" /> <!-- 0.252   = height above neck joint
                                                                         0.34906 = pitch angle downwards   -->
@@ -25,4 +25,4 @@
                   ${0.0+cal_head_mount_xtion_pitch}
                   ${-M_PI/2+cal_head_mount_xtion_yaw}" />
-  </xacro:xtion_withoutbase>
+  </xacro:xtion_pro_live>
 </robot>

File: reem_description/urdf/sensors/xtion_pro_live.urdf.xacro (robot description, xacro)
@@ -25,8 +25,8 @@
   <property name="M_PI" value="3.1415926535897931" />
   <!-- Macro -->
-  <xacro:macro name="xtion_withoutbase" params="name parent *origin *calibration_origin">
+  <xacro:macro name="xtion_pro_live" params="name parent *origin *calibration_origin">
     <!-- base link -->
     <joint name="${name}_joint" type="fixed">
-      <insert_block name="origin" /> <!-- macro argument -->
+      <insert_block name="origin" />
       <parent link="${parent}"/>
       <child link="${name}_link"/>
@@ -43,5 +43,5 @@
         <origin xyz="0 0 0" rpy="0 0 0"/>
         <geometry>
-          <mesh filename="package://reem_description/meshes/sensors/xtion/xtion_pro_live.dae" />
+          <mesh filename="package://reem_description/meshes/sensors/xtion_pro_live/xtion_pro_live.dae" />
         </geometry>
         <material name="gray">

Commit message: Modified x-position & pitch angle of ASUS Xtion. The sensor needs to be located more forward, and angled downwards at the table. However this position is not calibrated, and may not be suitable for other vision tasks.

File: reem_description/robots/reem_xtion_pro_live.urdf.xacro (robot description, xacro)
@@ -17,6 +17,6 @@
   <include filename="$(find reem_description)/urdf/sensors/xtion_pro_live.urdf.xacro" />
   <xacro:xtion_pro_live parent="head_2_link" name="head_mount_xtion" > <!-- name is appended to create link and topic names -->
-     <origin xyz="0.056 -0.252 0.0" rpy="${M_PI/2} 0.0 0.34906" /> <!-- 0.252   = height above neck joint
-                                                                        0.34906 = pitch angle downwards   -->
+     <origin xyz="0.100 -0.252 0.0" rpy="${M_PI/2} 0.0 1.0" /> <!-- 0.252   = height above neck joint
+                                                                        1.0 = pitch angle downwards   -->
      <origin xyz="${cal_head_mount_xtion_x}
                   ${cal_head_mount_xtion_y}

Commit message: Added parameter to specify topic prefix for ASUS. A new parameter to specify the namespace prefix for the topics output from the simulated OpenNI sensor. By modifying this namespace, you can then publish real sensor data on these topics, thereby using the real sensor data in simulation.

File: reem_description/robots/reem_xtion_pro_live.urdf.xacro (robot description, xacro)
@@ -16,13 +16,14 @@
   <!-- Head-mounted ASUS Xtion Pro Live -->
   <include filename="$(find reem_description)/urdf/sensors/xtion_pro_live.urdf.xacro" />
-  <xacro:xtion_pro_live parent="head_2_link" name="head_mount_xtion" > <!-- name is appended to create link and topic names -->
-     <origin xyz="0.100 -0.252 0.0" rpy="${M_PI/2} 0.0 1.0" /> <!-- 0.252   = height above neck joint
-                                                                        1.0 = pitch angle downwards   -->
-     <origin xyz="${cal_head_mount_xtion_x}
-                  ${cal_head_mount_xtion_y}
-                  ${cal_head_mount_xtion_z}"
-             rpy="${-M_PI/2+cal_head_mount_xtion_roll}
-                  ${0.0+cal_head_mount_xtion_pitch}
-                  ${-M_PI/2+cal_head_mount_xtion_yaw}" />
+  <xacro:xtion_pro_live parent="head_2_link" name="head_mount_xtion" namespace="head_mount_xtion" > <!-- 'name' is appended to create link/frame/camera names -->
+                                                                                                    <!-- 'namespace' is the prefix for the output topics -->
+     <origin xyz="0.100 -0.252 0.0" rpy="${M_PI/2} 0.0 1.0" /> <!--  0.252 = height above neck joint
+                                                                       1.0 = pitch angle downwards   -->
+     <calibration_origin xyz="${cal_head_mount_xtion_x}
+                              ${cal_head_mount_xtion_y}
+                              ${cal_head_mount_xtion_z}"
+                         rpy="${-M_PI/2+cal_head_mount_xtion_roll}
+                              ${0.0+cal_head_mount_xtion_pitch}
+                              ${-M_PI/2+cal_head_mount_xtion_yaw}" />
   </xacro:xtion_pro_live>
 </robot>

File: reem_description/urdf/sensors/openni.gazebo.xacro (robot description, xacro)
@@ -15,5 +15,5 @@
        xmlns:interface="http://playerstage.sourceforge.net/gazebo/xmlschema/#interface"
        xmlns:xacro="http://ros.org/wiki/xacro">
-  <xacro:macro name="openni_ir_gazebo_v0" params="link_name frame_name camera_name">
+  <xacro:macro name="openni_ir_gazebo_v0" params="link_name frame_name camera_name topic_namespace">
     <gazebo reference="${link_name}">
       <sensor:camera name="${name}_ir_sensor">
@@ -29,9 +29,9 @@
           <updateRate>1.0</updateRate>
           <cameraName>${camera_name}_ir</cameraName>
-          <imageTopicName>/${camera_name}/depth/image_raw</imageTopicName>
-          <cameraInfoTopicName>/${camera_name}/depth/camera_info</cameraInfoTopicName>
-          <depthImageTopicName>/${camera_name}/depth/image_raw</depthImageTopicName>
-          <depthImageInfoTopicName>/${camera_name}/depth/camera_info</depthImageInfoTopicName>
-          <pointCloudTopicName>/${camera_name}/depth/points</pointCloudTopicName>
+          <imageTopicName>/${topic_namespace}/depth/image_raw</imageTopicName>
+          <cameraInfoTopicName>/${topic_namespace}/depth/camera_info</cameraInfoTopicName>
+          <depthImageTopicName>/${topic_namespace}/depth/image_raw</depthImageTopicName>
+          <depthImageInfoTopicName>/${topic_namespace}/depth/camera_info</depthImageInfoTopicName>
+          <pointCloudTopicName>/${topic_namespace}/depth/points</pointCloudTopicName>
           <frameName>${frame_name}</frameName>
           <pointCloudCutoff>0.5</pointCloudCutoff>
@@ -45,5 +45,5 @@
     </gazebo>
   </xacro:macro>
-  <xacro:macro name="openni_rgb_gazebo_v0" params="link_name frame_name camera_name">
+  <xacro:macro name="openni_rgb_gazebo_v0" params="link_name frame_name camera_name topic_namespace">
     <gazebo reference="${link_name}">
       <sensor:camera name="${name}_rgb_sensor">
@@ -59,7 +59,7 @@
           <updateRate>1.0</updateRate>
           <cameraName>${camera_name}_rgb</cameraName>
-          <imageTopicName>/${camera_name}/rgb/image_raw</imageTopicName>
-          <cameraInfoTopicName>/${camera_name}/rgb/camera_info</cameraInfoTopicName>
-          <pointCloudTopicName>/${camera_name}/depth_registered/points</pointCloudTopicName>
+          <imageTopicName>/${topic_namespace}/rgb/image_raw</imageTopicName>
+          <cameraInfoTopicName>/${topic_namespace}/rgb/camera_info</cameraInfoTopicName>
+          <pointCloudTopicName>/${topic_namespace}/depth_registered/points</pointCloudTopicName>
           <frameName>${frame_name}</frameName>
           <pointCloudCutoff>0.5</pointCloudCutoff>

File: reem_description/urdf/sensors/xtion_pro_live.urdf.xacro (robot description, xacro)
@@ -11,9 +11,7 @@
     - TF frames
     - loads Gazebo plugin
-    Note: There is a bug that Gazebo in ROS Fuerte ignores the roll/pitch/yaw in the visual tag,
-          therefore it needs to be in a separate link, with the orientation specified at the joint.
-    ToDo: Fix visual mesh, re-scale it, & the origin is not centered along the frontal axis.
-          Can simplify collision mesh.
-          Rotate origin in mesh, to match the orientation of the base link and bypass the bug.
+    Note: There is a bug in ROS Fuerte Gazebo that mis-handles the origin tag for any visual or collision
+          geometry. The origin must be zero.
+          To specify the geometry, use a mesh with an origin that matches the joint, or use a separate link.
 -->
 <robot xmlns:sensor="http://playerstage.sourceforge.net/gazebo/xmlschema/#sensor"
@@ -25,5 +23,5 @@
   <property name="M_PI" value="3.1415926535897931" />
   <!-- Macro -->
-  <xacro:macro name="xtion_pro_live" params="name parent *origin *calibration_origin">
+  <xacro:macro name="xtion_pro_live" params="name namespace parent *origin *calibration_origin">
     <!-- base link -->
     <joint name="${name}_joint" type="fixed">
@@ -90,5 +88,5 @@
     </link>
     <!-- OpenNI IR sensor Gazebo extensions -->
-    <xacro:openni_ir_gazebo_v0 link_name="${name}_ir_link" frame_name="${name}_ir_optical_frame" camera_name="${name}" />
+    <xacro:openni_ir_gazebo_v0 link_name="${name}_ir_link" frame_name="${name}_ir_optical_frame" camera_name="${name}" topic_namespace="${namespace}" />
     <!-- Xtion RGB sensor physical attachment -->
     <joint name="${name}_rgb_joint" type="fixed">
@@ -124,5 +122,5 @@
     </link>
     <!-- OpenNI RGB sensor Gazebo extensions -->
-    <xacro:openni_rgb_gazebo_v0 link_name="${name}_rgb_link" frame_name="${name}_rgb_optical_frame" camera_name="${name}" />
+    <xacro:openni_rgb_gazebo_v0 link_name="${name}_rgb_link" frame_name="${name}_rgb_optical_frame" camera_name="${name}" topic_namespace="${namespace}" />
   </xacro:macro>
 </robot>

Commit message: Removed bug with macro block.

File: reem_description/robots/reem_xtion_pro_live.urdf.xacro (robot description, xacro)
@@ -16,14 +16,17 @@
   <!-- Head-mounted ASUS Xtion Pro Live -->
   <include filename="$(find reem_description)/urdf/sensors/xtion_pro_live.urdf.xacro" />
-  <xacro:xtion_pro_live parent="head_2_link" name="head_mount_xtion" namespace="head_mount_xtion" > <!-- 'name' is appended to create link/frame/camera names -->
+  <xacro:xtion_pro_live parent="head_2_link" name="head_mount_xtion" namespace="head_mount_xtion" >
+                                                                                                    <!-- 'name' is appended to create link/frame/camera names -->
                                                                                                     <!-- 'namespace' is the prefix for the output topics -->
+     <!-- this block is the "origin" param -->
      <origin xyz="0.100 -0.252 0.0" rpy="${M_PI/2} 0.0 1.0" /> <!--  0.252 = height above neck joint
                                                                        1.0 = pitch angle downwards   -->
-     <calibration_origin xyz="${cal_head_mount_xtion_x}
-                              ${cal_head_mount_xtion_y}
-                              ${cal_head_mount_xtion_z}"
-                         rpy="${-M_PI/2+cal_head_mount_xtion_roll}
-                              ${0.0+cal_head_mount_xtion_pitch}
-                              ${-M_PI/2+cal_head_mount_xtion_yaw}" />
+     <!-- this block is the "calibration_origin" param -->
+     <origin xyz="${cal_head_mount_xtion_x}
+                  ${cal_head_mount_xtion_y}
+                  ${cal_head_mount_xtion_z}"
+             rpy="${-M_PI/2+cal_head_mount_xtion_roll}
+                  ${0.0+cal_head_mount_xtion_pitch}
+                  ${-M_PI/2+cal_head_mount_xtion_yaw}" />
   </xacro:xtion_pro_live>
 </robot>
