Commit message: Sync robot model with internal repo.
Update sensor locations, types, and naming convention.

File: reem_description/robots/reem.urdf.xacro (robot description, xacro)
@@ -25,4 +25,5 @@
   <!-- Camera sensors -->
   <include filename="$(find reem_description)/urdf/sensors/stereo_camera.urdf.xacro" />
+<!--   <include filename="$(find reem_description)/urdf/sensors/back_camera.urdf.xacro" /> -->
   <!-- Generic simulator_gazebo plugins -->
   <include filename="$(find reem_description)/gazebo/gazebo.urdf.xacro" />
@@ -45,3 +46,7 @@
     <origin xyz="0.08203  -0.09558  0.04132" rpy="1.56293 -0.00855922 -0.0201307" />
   </xacro:stereo_camera_v0>
+<!--   <xacro:back_camera_v0 parent="torso_2_link" name="back" focal_length="557" hfov="75" image_format="B8G8R8" image_width="640" image_height="480" >  -->
+    <!-- The following transformations expresses the pose of the back_link (X pointing forward, Z upwards and Y leftwards, contrary to the stereo_optical_link which has Z pointing forward) wrt  torso_2_link. -->
+    <!--<origin xyz="-0.140 -0.302 -0.000" rpy="-3.142 1.571 0.211" />
+  </xacro:back_camera_v0>-->
 </robot>

File: reem_description/urdf/base/base.urdf.xacro (robot description, xacro)
@@ -19,4 +19,5 @@
   <include filename="$(find reem_description)/urdf/sensors/microstrain_3dmgx2_imu.urdf.xacro" />
   <include filename="$(find reem_description)/urdf/sensors/range.urdf.xacro" />
+  <include filename="$(find reem_description)/urdf/sensors/bumper.urdf.xacro" />
   <!--wheel characteristics-->
   <property name="dist_between_wheels" value="0.489" />
@@ -207,60 +208,98 @@
     </xacro:hokuyo_laser_reem>
     <!-- base sonar -->
-    <xacro:range_reem name="${name}_sonar_04" parent="${name}" ros_topic="sonar_base" update_rate="5" maxRange="1.5" minRange="0.005" fov="0.3491">
+    <xacro:range_reem name="${name}_sonar_04" parent="${name}" ros_topic="sonar_base" update_rate="5" maxRange="1.5" minRange="0.005" fov="0.3491" radiation="ultrasound">
       <origin xyz="0.17131 0.0 0.1425" rpy="0.0 0.0 0.0" />
     </xacro:range_reem>
     <!-- base sonar -->
-    <xacro:range_reem name="${name}_sonar_05" parent="${name}" ros_topic="sonar_base" update_rate="5" maxRange="1.5" minRange="0.005" fov="0.3491">
-      <origin xyz="0.16919 0.12345 0.1425" rpy="0.0 0.0 0.349" />
-    </xacro:range_reem>
-   <!-- base sonar -->
-    <xacro:range_reem name="${name}_sonar_15" parent="${name}" ros_topic="sonar_base" update_rate="5" maxRange="1.5" minRange="0.0" fov="0.3491" >
-      <origin xyz="0.16919 -0.12345 0.1425" rpy="0.0 0.0 -0.349" />
-    </xacro:range_reem>
-   <!-- base sonar -->
-    <xacro:range_reem name="${name}_sonar_06" parent="${name}" ros_topic="sonar_base" update_rate="5" maxRange="1.5" minRange="0.0" fov="0.3491" >
-      <origin xyz="0.13676 0.27111 0.13702" rpy="0.0 0.0 0.8377" /> <!--3 y 4  x=0.11676 y=0.25111-->
-    </xacro:range_reem>
-   <!-- base sonar -->
-    <xacro:range_reem name="${name}_sonar_14" parent="${name}" ros_topic="sonar_base" update_rate="5" maxRange="1.5" minRange="0.0" fov="0.3491" >
+    <xacro:range_reem name="${name}_sonar_05" parent="${name}" ros_topic="sonar_base" update_rate="5" maxRange="1.5" minRange="0.005" fov="0.3491" radiation="ultrasound">
+      <origin xyz="0.18919 0.16919 0.1425" rpy="0.0 0.0 0.349" />
+    </xacro:range_reem>
+   <!-- base sonar -->
+    <xacro:range_reem name="${name}_sonar_15" parent="${name}" ros_topic="sonar_base" update_rate="5" maxRange="1.5" minRange="0.005" fov="0.3491" radiation="ultrasound">
+      <origin xyz="0.18919 -0.16919 0.1425" rpy="0.0 0.0 -0.349" />
+    </xacro:range_reem>
+   <!-- base sonar -->
+    <xacro:range_reem name="${name}_sonar_06" parent="${name}" ros_topic="sonar_base" update_rate="5" maxRange="1.5" minRange="0.005" fov="0.3491" radiation="ultrasound">
+      <origin xyz="0.13676 0.27111 0.13702" rpy="0.0 0.0 0.8377" />
+    </xacro:range_reem>
+   <!-- base sonar -->
+    <xacro:range_reem name="${name}_sonar_14" parent="${name}" ros_topic="sonar_base" update_rate="5" maxRange="1.5" minRange="0.005" fov="0.3491" radiation="ultrasound">
       <origin xyz="0.13676 -0.27111 0.13702" rpy="0.0 0.0 -0.8377" />
     </xacro:range_reem>
    <!-- base sonar -->
-    <xacro:range_reem name="${name}_sonar_07" parent="${name}" ros_topic="sonar_base" update_rate="5" maxRange="1.5" minRange="0.0" fov="0.3491" >
-      <origin xyz="0.064 0.33455 0.1475" rpy="0.0 0.0 1.5708" /> <!--5 y 6  y=0.29455 -->
-    </xacro:range_reem>
-   <!-- base sonar -->
-    <xacro:range_reem name="${name}_sonar_13" parent="${name}" ros_topic="sonar_base" update_rate="5" maxRange="1.5" minRange="0.0" fov="0.3491" >
+    <xacro:range_reem name="${name}_sonar_07" parent="${name}" ros_topic="sonar_base" update_rate="5" maxRange="1.5" minRange="0.005" fov="0.3491" radiation="ultrasound">
+      <origin xyz="0.064 0.33455 0.1475" rpy="0.0 0.0 1.5708" />
+    </xacro:range_reem>
+   <!-- base sonar -->
+    <xacro:range_reem name="${name}_sonar_13" parent="${name}" ros_topic="sonar_base" update_rate="5" maxRange="1.5" minRange="0.005" fov="0.3491" radiation="ultrasound">
       <origin xyz="0.064 -0.31455 0.1475" rpy="0.0 0.0 -1.5708" />
     </xacro:range_reem>
    <!-- base sonar -->
-    <xacro:range_reem name="${name}_sonar_08" parent="${name}" ros_topic="sonar_base" update_rate="5" maxRange="1.5" minRange="0.0" fov="0.3491" >
-      <origin xyz="-0.35563 0.28266 0.11219" rpy="0.0 0.0 1.9547" /> <!--7 y 8  y=0.27266 -->
-    </xacro:range_reem>
-   <!-- base sonar -->
-    <xacro:range_reem name="${name}_sonar_12" parent="${name}" ros_topic="sonar_base" update_rate="5" maxRange="1.5" minRange="0.0" fov="0.3491" >
+    <xacro:range_reem name="${name}_sonar_08" parent="${name}" ros_topic="sonar_base" update_rate="5" maxRange="1.5" minRange="0.005" fov="0.3491" radiation="ultrasound">
+      <origin xyz="-0.35563 0.28266 0.11219" rpy="0.0 0.0 1.9547" />
+    </xacro:range_reem>
+   <!-- base sonar -->
+    <xacro:range_reem name="${name}_sonar_12" parent="${name}" ros_topic="sonar_base" update_rate="5" maxRange="1.5" minRange="0.005" fov="0.3491" radiation="ultrasound">
       <origin xyz="-0.35563 -0.28266 0.11219" rpy="0.0 0.0 -1.9547" />
     </xacro:range_reem>
    <!-- base sonar -->
-    <xacro:range_reem name="${name}_sonar_09" parent="${name}" ros_topic="sonar_base" update_rate="5" maxRange="1.5" minRange="0.0" fov="0.3491" >
-      <origin xyz="-0.49412 0.15127 0.15748" rpy="0.0 0.0 2.6354" /> <!--10 y 9  x=0.45412 -->
-    </xacro:range_reem>
-   <!-- base sonar -->
-    <xacro:range_reem name="${name}_sonar_11" parent="${name}" ros_topic="sonar_base" update_rate="5" maxRange="1.5" minRange="0.0" fov="0.3491" >
+    <xacro:range_reem name="${name}_sonar_09" parent="${name}" ros_topic="sonar_base" update_rate="5" maxRange="1.5" minRange="0.005" fov="0.3491" radiation="ultrasound">
+      <origin xyz="-0.49412 0.15127 0.15748" rpy="0.0 0.0 2.6354" />
+    </xacro:range_reem>
+   <!-- base sonar -->
+    <xacro:range_reem name="${name}_sonar_11" parent="${name}" ros_topic="sonar_base" update_rate="5" maxRange="1.5" minRange="0.005" fov="0.3491" radiation="ultrasound">
       <origin xyz="-0.49412 -0.15127 0.15748" rpy="0.0 0.0 -2.6354" />
     </xacro:range_reem>
    <!-- base sonar -->
-    <xacro:range_reem name="${name}_sonar_10" parent="${name}" ros_topic="sonar_base" update_rate="5" maxRange="1.5" minRange="0.0" fov="0.3491" >
-      <origin xyz="-0.52188 0.0 0.12547" rpy="0.0 0.0 -3.1415" />  <!--11  x=-0.50188 -->
-    </xacro:range_reem>
- <!-- Torso Front Sonar Ring -->
+    <xacro:range_reem name="${name}_sonar_10" parent="${name}" ros_topic="sonar_base" update_rate="5" maxRange="1.5" minRange="0.005" fov="0.3491" radiation="ultrasound">
+      <origin xyz="-0.52188 0.0 0.12547" rpy="0.0 0.0 -3.1415" />
+    </xacro:range_reem>
+<!-- Torso Front Sonar Ring -->
    <!-- torso sonar left -->
-   <xacro:range_reem name="${name}_sonar_18" parent="${name}" ros_topic="sonar_torso" update_rate="5" maxRange="1.45" minRange="0.0" fov="0.3491" >
+   <xacro:range_reem name="${name}_sonar_18" parent="${name}" ros_topic="sonar_torso" update_rate="5" maxRange="1.45" minRange="0.005" fov="0.3491" radiation="ultrasound">
       <origin xyz="0.04 0.065 0.95" rpy="0.0 0.0 0.0" />
    </xacro:range_reem>
    <!-- torso sonar right -->
-   <xacro:range_reem name="${name}_sonar_19" parent="${name}" ros_topic="sonar_torso" update_rate="5" maxRange="1.45" minRange="0.0" fov="0.3491" >
+   <xacro:range_reem name="${name}_sonar_19" parent="${name}" ros_topic="sonar_torso" update_rate="5" maxRange="1.45" minRange="0.005" fov="0.3491" radiation="ultrasound">
       <origin xyz="0.04 -0.065 0.95" rpy="0.0 0.0 0.0" />
    </xacro:range_reem>
+   <!-- base ir -->
+    <xacro:range_reem name="${name}_ir_01" parent="${name}" ros_topic="ir_base" update_rate="10" maxRange="1.45" minRange="0.005" fov="0.1" radiation="infrared">
+      <origin xyz="0.15904 -0.12463 0.0859" rpy="0.0 -0.8726 0.0" />
+    </xacro:range_reem>
+    <xacro:range_reem name="${name}_ir_02" parent="${name}" ros_topic="ir_base" update_rate="10" maxRange="1.45" minRange="0.005" fov="0.1" radiation="infrared">
+      <origin xyz="0.17074 0.0 0.08597" rpy="0.0 -0.8726 0.0" />
+    </xacro:range_reem>
+    <xacro:range_reem name="${name}_ir_03" parent="${name}" ros_topic="ir_base" update_rate="10" maxRange="1.45" minRange="0.005" fov="0.1" radiation="infrared">
+      <origin xyz="0.15904 0.12463 0.0859" rpy="0.0 -0.8726 0.0" />
+    </xacro:range_reem>
+    <!-- bumper front right -->
+    <xacro:bumper_reem name="${name}_bumper_01" parent="${name}" ros_topic="bumper_contact" update_rate="25" >
+      <origin xyz="0.15 -0.15 0.15" rpy="0 0 0" />
+    </xacro:bumper_reem>
+    <!-- bumper front left -->
+    <xacro:bumper_reem name="${name}_bumper_02" parent="${name}" ros_topic="bumper_contact" update_rate="25" >
+      <origin xyz="0.15 0.15 0.15" rpy="0 0 0" />
+    </xacro:bumper_reem>
+    <!-- bumper left 1 -->
+    <xacro:bumper_reem name="${name}_bumper_03" parent="${name}" ros_topic="bumper_contact" update_rate="25" >
+      <origin xyz="0.064 0.30 0.1" rpy="0 0 1.57" />
+    </xacro:bumper_reem>
+    <!-- bumper left 2 -->
+    <xacro:bumper_reem name="${name}_bumper_04" parent="${name}" ros_topic="bumper_contact" update_rate="25" >
+      <origin xyz="-0.35 -0.27 0.075" rpy="0 0 1.57" />
+    </xacro:bumper_reem>
+    <!-- bumper back -->
+    <xacro:bumper_reem name="${name}_bumper_05" parent="${name}" ros_topic="bumper_contact" update_rate="25" >
+      <origin xyz="-0.51 0.0 0.075" rpy="0 0 -3.1415" />
+    </xacro:bumper_reem>
+    <!-- bumper right 2 -->
+    <xacro:bumper_reem name="${name}_bumper_06" parent="${name}" ros_topic="bumper_contact" update_rate="25" >
+      <origin xyz="-0.35 0.27 0.075" rpy="0 0 1.57" />
+    </xacro:bumper_reem>
+    <!-- bumper right 1 -->
+    <xacro:bumper_reem name="${name}_bumper_07" parent="${name}" ros_topic="bumper_contact" update_rate="25" >
+      <origin xyz="0.064 -0.30 0.1" rpy="0 0 1.57" />
+    </xacro:bumper_reem>
     <!-- gyroscope microinfinity XA3300
     <xacro:microinfinity_xa3300 name="imu" parent="${name}" imu_topic="imu/data" update_rate="100.0" stdev="0.0005" >

File: reem_description/urdf/head/head.urdf.xacro (robot description, xacro)
@@ -87,6 +87,6 @@
     </joint>
        <!-- Head Sonar -->
-   <xacro:range_reem name="head_sonar_20" parent="${name}" ros_topic="sonar_torso" update_rate="5" maxRange="1.5" minRange="0.0" fov="0.3491" >
-      <origin xyz="0.066 -0.195 0.0" rpy="1.57 0.0 0.0" />
+   <xacro:range_reem name="head_sonar_20" parent="${name}" ros_topic="sonar_torso" update_rate="5" maxRange="1.5" minRange="0.0" fov="0.3491" radiation="ultrasound">
+      <origin xyz="0.086 -0.195 0.0" rpy="1.57 0.0 0.0" />
    </xacro:range_reem>
     <!-- extensions -->

File: reem_description/urdf/sensors/kinect.gazebo.xacro (robot description, xacro)
@@ -40,5 +40,5 @@
 </xacro:macro>-->
  <xacro:macro name="sim_kinect">
-  <gazebo reference="kinect_link">
+  <gazebo reference="openni_camera">
     <sensor:camera name="kinect">
       <imageFormat>R8G8B8</imageFormat>
@@ -56,5 +56,5 @@
         <pointCloudTopicName>/camera/depth/points</pointCloudTopicName>
         <cameraInfoTopicName>/camera/camera_info</cameraInfoTopicName>
-        <frameName>kinect_rgb_optical_frame</frameName>
+        <frameName>openni_rgb_optical_frame</frameName>
         <distortion_k1>0.0</distortion_k1>
         <distortion_k2>0.0</distortion_k2>

File: reem_description/urdf/sensors/kinect.urdf.xacro (robot description, xacro)
@@ -14,11 +14,11 @@
   <include filename="$(find reem_description)/urdf/sensors/kinect.gazebo.xacro" />
   <xacro:macro name="kinect_v0" params="parent name *origin">
-   <joint name="${name}_kinect_joint" type="fixed">
+   <joint name="${name}_joint" type="fixed">
     <origin xyz="${reem_calib_cam_x} ${reem_calib_cam_y} ${reem_calib_cam_z}"
             rpy="${reem_calib_cam_rr} ${reem_calib_cam_rp} ${reem_calib_cam_ry}" />
     <parent link="${reem_camera_parent_name}" />
-    <child link="${name}_link" />
+    <child link="${name}_camera" />
   </joint>
-  <link name="${name}_link">
+  <link name="${name}_camera">
     <inertial>
       <mass value="0.01" />
@@ -41,10 +41,10 @@
     </collision>
   </link>
-  <joint name="kinect_depth_joint" type="fixed">
+  <joint name="${name}_depth_joint" type="fixed">
     <origin xyz="0 0.018 0" rpy="0 0 0" />
-    <parent link="kinect_link" />
-    <child link="kinect_depth_frame" />
+    <parent link="${name}_camera" />
+    <child link="${name}_depth_frame" />
   </joint>
-  <link name="kinect_depth_frame">
+  <link name="${name}_depth_frame">
     <inertial>
       <mass value="0.01" />
@@ -55,10 +55,10 @@
     </inertial>
   </link>
-  <joint name="kinect_depth_optical_joint" type="fixed">
+  <joint name="${name}_depth_optical_joint" type="fixed">
     <origin xyz="0 0 0" rpy="${-M_PI/2} 0 ${-M_PI/2}" />
-    <parent link="kinect_depth_frame" />
-    <child link="kinect_depth_optical_frame" />
+    <parent link="${name}_depth_frame" />
+    <child link="${name}_depth_optical_frame" />
   </joint>
-  <link name="kinect_depth_optical_frame">
+  <link name="${name}_depth_optical_frame">
     <inertial>
       <mass value="0.001" />
@@ -69,10 +69,10 @@
     </inertial>
   </link>
-  <joint name="kinect_rgb_joint" type="fixed">
+  <joint name="${name}_rgb_joint" type="fixed">
     <origin xyz="0 -0.005 0" rpy="0 0 0" />
-    <parent link="kinect_link" />
-    <child link="kinect_rgb_frame" />
+    <parent link="${name}_camera" />
+    <child link="${name}_rgb_frame" />
   </joint>
-  <link name="kinect_rgb_frame">
+  <link name="${name}_rgb_frame">
     <inertial>
       <mass value="0.001" />
@@ -83,10 +83,10 @@
     </inertial>
   </link>
-  <joint name="kinect_rgb_optical_joint" type="fixed">
+  <joint name="${name}_rgb_optical_joint" type="fixed">
     <origin xyz="0 0 0" rpy="${-M_PI/2} 0 ${-M_PI/2}" />
-    <parent link="kinect_rgb_frame" />
-    <child link="kinect_rgb_optical_frame" />
+    <parent link="${name}_rgb_frame" />
+    <child link="${name}_rgb_optical_frame" />
   </joint>
-  <link name="kinect_rgb_optical_frame">
+  <link name="${name}_rgb_optical_frame">
     <inertial>
       <mass value="0.001" />

File: reem_description/urdf/sensors/range.gazebo.xacro (robot description, xacro)
@@ -11,16 +11,15 @@
        xmlns:interface="http://playerstage.sourceforge.net/gazebo/xmlschema/#interface"
        xmlns:xacro="http://ros.org/wiki/xacro">
-  <xacro:macro name="range_reem_gazebo" params="name ros_topic update_rate maxRange minRange fov">
+  <xacro:macro name="range_reem_gazebo" params="name ros_topic update_rate maxRange minRange fov radiation" >
     <gazebo reference="${name}_link">
-      <sensor:ir name="${name}">
-	<rayCount>5</rayCount>
-	<!--verticalRayCount>3</verticalRayCount-->
-	<!--irCount>10</irCount-->
-	<rangeCount>1</rangeCount>
-        <origin>0.0 0.0 0.0</origin>
-        <displayRays>false</displayRays>
-	<minAngle>${-fov/2}</minAngle>
+      <sensor:ray name="${name}">
+        <!-- displayRays>fan</displayRays -->
+        <rayCount>5</rayCount>
+        <rangeCount>5</rangeCount>
+        <verticalRayCount>5</verticalRayCount>
+        <verticalRangeCount>5</verticalRangeCount>
+        <minAngle>-${fov/2}</minAngle>
+        <verticalMinAngle>-${fov/2}</verticalMinAngle>
         <maxAngle>${fov/2}</maxAngle>
-	<verticalMinAngle>${-fov/2}</verticalMinAngle>
         <verticalMaxAngle>${fov/2}</verticalMaxAngle>
         <minRange>${minRange}</minRange>
@@ -28,16 +27,14 @@
         <resRange>0.01</resRange>
         <updateRate>${update_rate}</updateRate>
-        <controller:gazebo_ros_ir name="gazebo_ros_${name}_controller" plugin="libgazebo_ros_ir.so">
-          <gaussianNoise>0.0005</gaussianNoise>
+        <controller:gazebo_ros_sonar name="gazebo_ros_${name}_controller" plugin="libgazebo_ros_sonar.so">
+          <gaussianNoise>0.005</gaussianNoise>
           <alwaysOn>true</alwaysOn>
           <updateRate>${update_rate}</updateRate>
           <topicName>${ros_topic}</topicName>
-          <frameName>${name}_link</frameName>
-  	  <maxRange>${maxRange}</maxRange>
-  	  <minRange>${minRange}</minRange>
-  	  <fov>${fov}</fov>
-          <interface:irarray name="gazebo_ros_${name}_iface" />
-        </controller:gazebo_ros_ir>
-      </sensor:ir>
+          <frameId>${name}_link</frameId>
+          <radiation>${radiation}</radiation>
+          <fov>${fov}</fov>
+        </controller:gazebo_ros_sonar>
+      </sensor:ray>
     </gazebo>
   </xacro:macro>

File: reem_description/urdf/sensors/range.urdf.xacro (robot description, xacro)
@@ -12,5 +12,5 @@
        xmlns:xacro="http://ros.org/wiki/xacro">
   <include filename="$(find reem_description)/urdf/sensors/range.gazebo.xacro" />
-  <xacro:macro name="range_reem" params="name parent *origin ros_topic update_rate maxRange minRange fov">
+  <xacro:macro name="range_reem" params="name parent *origin ros_topic update_rate maxRange minRange fov radiation">
     <joint name="${name}_joint" type="fixed">
       <axis xyz="0 0 0" rpy="0 0 0"/>
@@ -27,5 +27,5 @@
     </link>
     <!-- gazebo extensions -->
-    <xacro:range_reem_gazebo name="${name}" ros_topic="${ros_topic}" update_rate="${update_rate}" maxRange="${maxRange}" minRange="${minRange}" fov="${fov}"/>
+    <xacro:range_reem_gazebo name="${name}" ros_topic="${ros_topic}" update_rate="${update_rate}" maxRange="${maxRange}" minRange="${minRange}" fov="${fov}" radiation="${radiation}"/>
   </xacro:macro>
 </robot>
