Commit message: Add REEM-H3 hand description.
- Not using production visualization/collision geometries, but temporary STLs.

- Inertial parameters other than mass not yet set.

- Joint ranges have to be confirmed.

File: reem_description/robots/reem.urdf.xacro (robot description, xacro)
@@ -35,9 +35,9 @@
   <xacro:reem_torso name="torso" parent="base_link"/>
   <xacro:reem_head  name="head"  parent="torso_2_link"/>
-   This is a common convention, to use a reflect parameter that equals +-1 to distinguish left from right
+  <!-- The reflect parameter takes the value 1 or -1 to respectively distinguish right from left side in expressions -->
   <xacro:reem_arm name="arm" side="right" reflect="1.0" />
   <xacro:reem_arm name="arm" side="left"  reflect="-1.0" />
-  <xacro:reem_hand name="hand" side="right" reflect="1.0" />
-  <xacro:reem_hand name="hand" side="left"  reflect="-1.0" />
+  <xacro:reem_hand name="hand" parent="arm_right_tool_link" side="right" reflect="1.0"  />
+  <xacro:reem_hand name="hand" parent="arm_left_tool_link"  side="left"  reflect="-1.0" />
   <!-- stereo camera -->
   <!-- IMPORTANT: focal_length = image_width/(2tan(hfov/2)) -->

File: reem_description/urdf/hand/hand.gazebo.xacro (robot description, xacro)
@@ -11,7 +11,7 @@
        xmlns:interface="http://playerstage.sourceforge.net/gazebo/xmlschema/#interface"
        xmlns:xacro="http://ros.org/wiki/xacro">
-    <xacro:macro name="rh1_hand_1_gazebo" params="name side">
-    <gazebo reference="hand_${side}_1_link">
-      <material>Gazebo/Grey</material>
+    <xacro:macro name="hand_gazebo" params="name">
+    <gazebo reference="${name}_link">
+      <material>Gazebo/White</material>
       <turnGravityOff>false</turnGravityOff>
     </gazebo>

File: reem_description/urdf/hand/hand.transmission.xacro (robot description, xacro)
@@ -11,8 +11,8 @@
       xmlns:interface="http://playerstage.sourceforge.net/gazebo/xmlschema/#interface"
       xmlns:xacro="http://ros.org/wiki/xacro">
-  <xacro:macro name="reem_hand_1_transmission" params="name side" >
-    <transmission type="SimpleTransmission" name="${name}_${side}_1_trans">
-      <actuator name="${name}_${side}_1_motor" />
-      <joint name="${name}_${side}_1_joint" />
+  <xacro:macro name="hand_simple_transmission" params="name" >
+    <transmission type="SimpleTransmission" name="${name}_trans">
+      <actuator name="${name}_motor" />
+      <joint name="${name}_joint" />
       <mechanicalReduction>1.0</mechanicalReduction>
     </transmission>

File: reem_description/urdf/hand/hand.urdf.xacro (robot description, xacro)
@@ -14,15 +14,26 @@
   <include filename="$(find reem_description)/urdf/hand/hand.gazebo.xacro" />
   <include filename="$(find reem_description)/urdf/hand/hand.transmission.xacro" />
-  <xacro:macro name="reem_hand" params="name side reflect">
-    <link name="hand_${side}_link">
+  <xacro:property name="hand_friction" value="0.1" /> <!--TODO: Tune-->
+  <xacro:property name="hand_damping"  value="0.1" /> <!--TODO: Tune-->
+  <xacro:property name="hand_max_vel" value="1.0" />
+  <xacro:macro name="reem_finger" params="hand_name hand_side hand_reflect finger_name finger_reflect">
+    <joint name="${hand_name}_${hand_side}_${finger_name}_1_joint" type="revolute">
+      <parent link="${hand_name}_${hand_side}_palm_link" />
+      <child link="${hand_name}_${hand_side}_${finger_name}_1_link" />
+      <origin xyz="0.101 ${reflect * 0.0025} ${finger_reflect * 0.0165}" rpy="${(90.0 - reflect * 90.0) * deg_to_rad} 0 ${reflect * 90.0 * deg_to_rad}" />
+      <axis xyz="0 0 1" />
+      <limit lower="${0.0 * deg_to_rad}" upper="${90.0 * deg_to_rad}" effort="0.0" velocity="${hand_max_vel}" />
+      <dynamics friction="${hand_friction}" damping="${hand_damping}"/>
+    </joint>
+    <link name="${hand_name}_${hand_side}_${finger_name}_1_link">
       <inertial>
-        <origin xyz="0.01747 ${reflect * 0.0014} ${reflect * 0.128}" rpy="0 0 0" />
-        <mass value="0.8" />
-        <inertia ixx="0"  ixy="0"  ixz="0" iyy="0" iyz="0" izz="0" />
+        <origin xyz="0 0 0" rpy="0 0 0" /> <!--TODO: Fill up-->
+        <mass value="0.1" />
+        <inertia ixx="0"  ixy="0"  ixz="0" iyy="0" iyz="0" izz="0" /> <!--TODO: Fill up-->
       </inertial>
       <visual>
         <origin xyz="0 0 0" rpy="0 0 0" />
         <geometry>
-          <mesh filename="package://reem_description/meshes/hand/hand_${side}_low.stl" />
+          <mesh filename="package://reem_description/meshes/hand/hand_finger_1.stl" scale="1 1 ${-reflect * finger_reflect}" />
         </geometry>
         <material name="LightGrey" />
@@ -31,16 +42,136 @@
         <origin xyz="0 0 0" rpy="0 0 0" />
         <geometry>
-          <mesh filename="package://reem_description/meshes/hand/hand_${side}_low_convex.stlb" />
+          <mesh filename="package://reem_description/meshes/hand/hand_finger_1_collision.stl" scale="1 1 ${-reflect * finger_reflect}" />
         </geometry>
       </collision>
     </link>
-    <joint name="hand_${side}_joint" type="fixed">
-      <parent link="arm_${side}_7_link" />
-      <child link="hand_${side}_link" />
+    <joint name="${hand_name}_${hand_side}_${finger_name}_2_joint" type="revolute">
+      <parent link="${hand_name}_${hand_side}_${finger_name}_1_link" />
+      <child link="${hand_name}_${hand_side}_${finger_name}_2_link" />
+      <origin xyz="0.00357 -0.04084 0" rpy="0 0 0" />
+      <axis xyz="0 0 1" />
+      <limit lower="${0.0 * deg_to_rad}" upper="${90.0 * deg_to_rad}" effort="0.0" velocity="${hand_max_vel}" />
+      <dynamics friction="${hand_friction}" damping="${hand_damping}"/>
+      <mimic joint="${hand_name}_${hand_side}_${finger_name}_1_joint" multiplier="1" offset="0"/>
+    </joint>
+    <link name="${hand_name}_${hand_side}_${finger_name}_2_link">
+      <inertial>
+        <origin xyz="0 0 0" rpy="0 0 0" /> <!--TODO: Fill up-->
+        <mass value="0.05" />
+        <inertia ixx="0"  ixy="0"  ixz="0" iyy="0" iyz="0" izz="0" /> <!--TODO: Fill up-->
+      </inertial>
+      <visual>
+        <origin xyz="0 0 0" rpy="0 0 0" />
+        <geometry>
+          <mesh filename="package://reem_description/meshes/hand/hand_finger_2.stl" scale="1 1 ${-reflect * finger_reflect }" />
+        </geometry>
+        <material name="LightGrey" />
+      </visual>
+      <collision>
+        <origin xyz="0 0 0" rpy="0 0 0" />
+        <geometry>
+          <mesh filename="package://reem_description/meshes/hand/hand_finger_2_collision.stl" scale="1 1 ${-reflect * finger_reflect}" />
+        </geometry>
+      </collision>
+    </link>
+    <joint name="${hand_name}_${hand_side}_${finger_name}_3_joint" type="revolute">
+      <parent link="${hand_name}_${hand_side}_${finger_name}_2_link" />
+      <child link="${hand_name}_${hand_side}_${finger_name}_3_link" />
+      <origin xyz="0.00572 -0.0269 0" rpy="0 0 0" />
+      <axis xyz="0 0 1" />
+      <limit lower="${0.0 * deg_to_rad}" upper="${90.0 * deg_to_rad}" effort="0.0" velocity="${hand_max_vel}" />
+      <dynamics friction="${hand_friction}" damping="${hand_damping}"/>
+      <mimic joint="${hand_name}_${hand_side}_${finger_name}_2_joint" multiplier="1" offset="0"/>
+    </joint>
+    <link name="${hand_name}_${hand_side}_${finger_name}_3_link">
+      <inertial>
+        <origin xyz="0 0 0" rpy="0 0 0" /> <!--TODO: Fill up-->
+        <mass value="0.05" />
+        <inertia ixx="0"  ixy="0"  ixz="0" iyy="0" iyz="0" izz="0" /> <!--TODO: Fill up-->
+      </inertial>
+      <visual>
+        <origin xyz="0 0 0" rpy="0 0 0" />
+        <geometry>
+          <mesh filename="package://reem_description/meshes/hand/hand_finger_3.stl" scale="1 1 ${-reflect * finger_reflect}" />
+        </geometry>
+        <material name="LightGrey" />
+      </visual>
+      <collision>
+        <origin xyz="0 0 0" rpy="0 0 0" />
+        <geometry>
+          <mesh filename="package://reem_description/meshes/hand/hand_finger_3_collision.stl" scale="1 1 ${-reflect * finger_reflect}" />
+        </geometry>
+      </collision>
+    </link>
+    <xacro:hand_gazebo              name="${hand_name}_${hand_side}_${finger_name}_1"/>
+    <xacro:hand_gazebo              name="${hand_name}_${hand_side}_${finger_name}_2"/>
+    <xacro:hand_gazebo              name="${hand_name}_${hand_side}_${finger_name}_3"/>
+    <xacro:hand_simple_transmission name="${hand_name}_${hand_side}_${finger_name}_1" />
+    <xacro:hand_simple_transmission name="${hand_name}_${hand_side}_${finger_name}_2" />
+    <xacro:hand_simple_transmission name="${hand_name}_${hand_side}_${finger_name}_3" />
+  </xacro:macro>
+  <xacro:macro name="reem_hand" params="name parent side reflect">
+    <!-- Palm -->
+    <joint name="${name}_${side}_palm_joint" type="fixed">
+      <parent link="${parent}" />
+      <child link="${name}_${side}_palm_link" />
       <origin xyz="0 0 0" rpy="0 0 0" />
     </joint>
-    <!-- extensions -->
-    <xacro:reem_hand_1_gazebo name="${name}" side="${side}" />
-<!--     <xacro:reem_hand_1_transmission name="${name}" side="${side}" /> --><!--TODO: Remove?-->
+    <link name="${name}_${side}_palm_link">
+      <inertial>
+        <origin xyz="0.07547 0.00468 0.00291" rpy="0 0 0" />
+        <mass value="0.91066" />
+        <inertia ixx="0"  ixy="0"  ixz="0" iyy="0" iyz="0" izz="0" />
+      </inertial>
+      <visual>
+        <origin xyz="0 0 0" rpy="0 0 0" />
+        <geometry>
+          <mesh filename="package://reem_description/meshes/hand/hand_palm.stl" scale="1 ${-reflect} 1" />
+        </geometry>
+        <material name="LightGrey" />
+      </visual>
+      <collision>
+        <origin xyz="0 0 0" rpy="0 0 0" />
+        <geometry>
+          <mesh filename="package://reem_description/meshes/hand/hand_palm_collision.stl" scale="1 ${-reflect} 1" />
+        </geometry>
+      </collision>
+    </link>
+    <xacro:hand_gazebo name="${name}_${side}_palm"/>
+    <!-- Thumb -->
+    <joint name="${name}_${side}_thumb_joint" type="revolute">
+      <parent link="${name}_${side}_palm_link" />
+      <child link="${name}_${side}_thumb_link" />
+      <origin xyz="0.03649 ${reflect * 0.008}  0.02" rpy="0 ${(90.0 + 13) * deg_to_rad} ${reflect * 13.0 * deg_to_rad}" />
+      <axis xyz="0 0 1" />
+      <limit lower="${0.0 * deg_to_rad}" upper="${90.0 * deg_to_rad}" effort="0.0" velocity="${hand_max_vel}" />
+      <dynamics friction="${hand_friction}" damping="${hand_damping}"/>
+    </joint>
+    <link name="${name}_${side}_thumb_link">
+      <inertial>
+        <origin xyz="0 0 0" rpy="0 0 0" /> <!--TODO: Fill up-->
+        <mass value="0.1" />
+        <inertia ixx="0"  ixy="0"  ixz="0" iyy="0" iyz="0" izz="0" /> <!--TODO: Fill up-->
+      </inertial>
+      <visual>
+        <origin xyz="0 0 0" rpy="0 0 0" />
+        <geometry>
+          <mesh filename="package://reem_description/meshes/hand/hand_thumb.stl" scale="1 ${-reflect} 1" />
+        </geometry>
+        <material name="LightGrey" />
+      </visual>
+      <collision>
+        <origin xyz="0 0 0" rpy="0 0 0" />
+        <geometry>
+          <mesh filename="package://reem_description/meshes/hand/hand_thumb_collision.stl" scale="1 ${-reflect} 1" />
+        </geometry>
+      </collision>
+    </link>
+    <xacro:hand_gazebo name="${name}_${side}_thumb"/>
+    <xacro:hand_simple_transmission name="${name}_${side}_thumb" />
+    <!-- Index finger -->
+    <xacro:reem_finger hand_name="${name}" hand_side="${side}" hand_reflect="${reflect}" finger_name="index" finger_reflect="1"/>
+    <!-- Middle finger -->
+    <xacro:reem_finger hand_name="${name}" hand_side="${side}" hand_reflect="${reflect}" finger_name="middle" finger_reflect="-1"/>
   </xacro:macro>
 </robot>

Commit message: Add tool frame to arms, parent attribute to arm xacro.

File: reem_description/robots/reem.urdf.xacro (robot description, xacro)
@@ -36,6 +36,6 @@
   <xacro:reem_head  name="head"  parent="torso_2_link"/>
   <!-- The reflect parameter takes the value 1 or -1 to respectively distinguish right from left side in expressions -->
-  <xacro:reem_arm name="arm" side="right" reflect="1.0" />
-  <xacro:reem_arm name="arm" side="left"  reflect="-1.0" />
+  <xacro:reem_arm name="arm" parent="torso_2_link" side="right" reflect="1.0"  />
+  <xacro:reem_arm name="arm" parent="torso_2_link" side="left"  reflect="-1.0" />
   <xacro:reem_hand name="hand" parent="arm_right_tool_link" side="right" reflect="1.0"  />
   <xacro:reem_hand name="hand" parent="arm_left_tool_link"  side="left"  reflect="-1.0" />

File: reem_description/urdf/arm/arm.urdf.xacro (robot description, xacro)
@@ -16,5 +16,5 @@
   <xacro:property name="wrist_reduction"    value="336.0" />
   <xacro:property name="arm_friction"    value="1.0" /> <!--TODO: Tune-->
-  <xacro:property name="wrist_friction"  value="0.5" /> <!--TODO: Tune-->
+  <xacro:property name="wrist_friction"  value="1.0" /> <!--TODO: Tune-->
   <xacro:property name="arm_damping"     value="1.0" /> <!--TODO: Tune-->
   <xacro:property name="wrist_damping"   value="1.0" /> <!--TODO: Tune-->
@@ -27,5 +27,5 @@
   <include filename="$(find reem_description)/urdf/arm/arm.gazebo.xacro" />
   <include filename="$(find reem_description)/urdf/arm/arm.transmission.xacro" />
-  <xacro:macro name="reem_arm" params="name side reflect">
+  <xacro:macro name="reem_arm" params="name parent side reflect">
     <!--************************-->
     <!--        SHOULDER        -->
@@ -54,5 +54,5 @@
     </link>
     <joint name="arm_${side}_1_joint" type="revolute">
-      <parent link="torso_2_link" />
+      <parent link="${parent}" />
       <child link="arm_${side}_1_link" />
       <origin xyz="-0.015 -0.273 0" rpy="${(-165.0 * reflect) * deg_to_rad} 0 0" />
@@ -207,5 +207,5 @@
         <origin xyz="-0.0002 -0.01155 0.00002" rpy="0 0 0"/>
         <mass value="0.255" />
-        <inertia ixx="0"  ixy="0"  ixz="0" iyy="0" iyz="0" izz="0" />
+        <inertia ixx="0.0001335"  ixy="0"  ixz="0" iyy="0.0001335" iyz="0" izz="0.000204" />
       </inertial>
       <visual>
@@ -239,14 +239,14 @@
       </inertial>
       <visual>
-        <origin xyz="0 0 ${0.0375 * reflect}" rpy="0 0 0" />
-        <geometry>
-          <cylinder radius="0.0135" length="0.02"/>
-        </geometry>
-        <material name="LightGrey" />
-      </visual>
-      <collision>
-        <origin xyz="0 0 ${0.0375 * reflect}" rpy="0 0 0" />
-        <geometry>
-          <cylinder radius="0.0135" length="0.02"/>
+        <origin xyz="0 0 ${0.046 * reflect}" rpy="0 0 0" />
+        <geometry>
+          <cylinder radius="0.02" length="0.005"/>
+        </geometry>
+        <material name="DarkGrey" />
+      </visual>
+      <collision>
+        <origin xyz="0 0 ${0.046 * 0.75 * reflect}" rpy="0 0 0" />
+        <geometry>
+          <cylinder radius="0.02" length="0.023"/>
         </geometry>
       </collision>
@@ -259,4 +259,28 @@
       <limit lower="${-120.0 * deg_to_rad}" upper="${120.0 * deg_to_rad}" effort="0.0" velocity="${wrist_max_vel}" />
       <dynamics friction="${wrist_friction}" damping="${wrist_damping}"/>
+    </joint>
+    <link name="arm_${side}_tool_link">
+      <inertial>
+        <mass value="0.1" />
+        <inertia ixx="0.0" ixy="0.0" ixz="0.0" iyy="0.0" iyz="0.0" izz="0.0" />
+      </inertial>
+      <visual>
+        <origin xyz="0.001 0 0" rpy="0 ${90.0 * deg_to_rad} 0" />
+        <geometry>
+          <cylinder radius="0.005" length="0.005"/>
+        </geometry>
+        <material name="LightGrey" />
+      </visual>
+      <collision>
+        <origin xyz="0.001 0 0" rpy="0 ${90.0 * deg_to_rad} 0" />
+        <geometry>
+          <cylinder radius="0.005" length="0.005"/>
+        </geometry>
+      </collision>
+    </link>
+    <joint name="arm_${side}_tool_joint" type="fixed">
+      <parent link="arm_${side}_7_link" />
+      <child link="arm_${side}_tool_link" />
+      <origin xyz="0 0 ${reflect * 0.046}" rpy="${90.0 * deg_to_rad} ${-90.0 * reflect * deg_to_rad} 0" />
     </joint>
     <!-- extensions -->
