Commit message: Update sensors to Gazebo 1.5.

File: reem_description/robots/reem.urdf.xacro (robot description, xacro)
@@ -24,6 +24,6 @@
   <include filename="$(find reem_description)/urdf/hand/hand.urdf.xacro" />
   <!-- Camera sensors -->
-<!--   <include filename="$(find reem_description)/urdf/sensors/stereo_camera.urdf.xacro" /> -->
-  <!--<include filename="$(find reem_description)/urdf/sensors/back_camera.urdf.xacro" /> -->
+  <include filename="$(find reem_description)/urdf/sensors/stereo_camera.urdf.xacro" />
+  <include filename="$(find reem_description)/urdf/sensors/back_camera.urdf.xacro" />
   <!-- Generic simulator_gazebo plugins -->
   <include filename="$(find reem_description)/gazebo/gazebo.urdf.xacro" />
@@ -42,11 +42,12 @@
   <!-- stereo camera -->
   <!-- IMPORTANT: focal_length = image_width/(2tan(hfov/2)) -->
-<!--  <xacro:stereo_camera_v0 parent="head_2_link" name="stereo" focal_length_left="459.838918" hfov_left="71" focal_length_right="459.838918" hfov_right="71" image_format="B8G8R8" image_width="656" image_height="492">-->
+  <xacro:stereo_camera_v0 parent="head_2_link" name="stereo" focal_length_left="459.838928" hfov_left="${71.0*deg_to_rad}" focal_length_right="459.838928" hfov_right="${71.0*deg_to_rad}" image_format="B8G8R8" image_width="656" image_height="492">
     <!-- The following transformations expresses the pose of the stereo_link (X pointing forward, Z upwards and Y leftwards, contrary to the stereo_optical_link which has Z pointing forward) wrt  head_2_link. -->
-<!--     <origin xyz="0.08203  -0.09558  0.04132" rpy="1.56293 -0.00855922 -0.0201307" />
-  </xacro:stereo_camera_v0>-->
-<!--   <xacro:back_camera_v0 parent="torso_2_link" name="back" focal_length="557" hfov="75" image_format="B8G8R8" image_width="640" image_height="480" >  -->
-    <!-- The following transformations expresses the pose of the back_link (X pointing forward, Z upwards and Y leftwards, contrary to the stereo_optical_link which has Z pointing forward) wrt  torso_2_link. -->
-    <!--<origin xyz="-0.140 -0.302 -0.000" rpy="-3.142 1.571 0.211" />
-  </xacro:back_camera_v0>-->
+    <origin xyz="0.0558343 -0.106811 0.0254842" rpy="1.61 -0.00976311 -0.0519005" />
+  </xacro:stereo_camera_v0>
+  <xacro:reem_back_camera parent="torso_2_link" name="back_camera" focal_length="376.003507" hfov="${89.999451423*deg_to_rad}" image_format="B8G8R8" image_width="752" image_height="480" >
+    <!-- The following transformations expresses the pose of the back_camera_link (X pointing forward, Z upwards and Y leftwards) wrt torso_2_link. -->
+    <!-- <origin xyz="-0.120 -0.302 -0.000" rpy="-3.142 1.571 0.211" /> -->
+    <origin xyz="-0.127 -0.302 -0.000" rpy="-1.5708  0 -2.70526" />
+  </xacro:reem_back_camera>
 </robot>

File: reem_description/urdf/sensors/back_camera.urdf.xacro (robot description, xacro)
@@ -1,5 +1,5 @@
 <?xml version="1.0"?>
 <!--
-  Copyright (c) 2011, PAL Robotics, S.L.
+  Copyright (c) 2013, PAL Robotics, S.L.
   All rights reserved.
   This work is licensed under the Creative Commons Attribution-NonCommercial-NoDerivs 3.0 Unported License.
@@ -12,14 +12,8 @@
        xmlns:xacro="http://ros.org/wiki/xacro">
   <!-- back camera macro uses stingrayf033c_camera macros -->
-  <include filename="$(find reem_description)/urdf/sensors/stingrayf033c_camera.urdf.xacro" />
-  <include filename="$(find reem_description)/urdf/sensors/back_camera.gazebo.xacro" />
-  <property name="back_dx" value="0.00" />
-  <property name="back_dy" value="-0.073" /> <!-- back baseline according to back_link which has X pointing forward, Y leftwards and Z upwards (required by Gazebo for a camera sensor) -->
-  <property name="back_dz" value="0.00" />
-  <property name="back_rx" value="0.00" />
-  <property name="back_ry" value="0.00" />
-  <property name="back_rz" value="0.00" />
+  <include filename="$(find reem_description)/urdf/sensors/mvbluefox_back_camera.gazebo.xacro" />
+  <include filename="$(find reem_description)/urdf/sensors/mvbluefox_camera.urdf.xacro" />
   <!-- this macro is used for creating wide and narrow double back camera links -->
-  <xacro:macro name="back_camera_v0" params="name parent focal_length hfov image_format image_width image_height *origin">
+  <xacro:macro name="reem_back_camera" params="name parent focal_length hfov image_format image_width image_height *origin">
     <joint name="${name}_frame_joint" type="fixed">
       <insert_block name="origin" />
@@ -30,5 +24,5 @@
     <link name="${name}_link">
       <inertial>
-        <mass value="0.1" />
+        <mass value="0.05" />
         <origin xyz="0 0 0" rpy="0 0 0" />
         <inertia ixx="0.01"  ixy="0"  ixz="0" iyy="0.01"  iyz="0"  izz="0.01" /> <!-- this inertia is made up for now. -->
@@ -39,5 +33,4 @@
           <box size="0.001 0.001 0.001" />
         </geometry>
-        <material name="Blue" />
       </visual>
       <collision>
@@ -55,15 +48,18 @@
     </joint>
     <!-- optical frame for the back camera, with z-forward notation, this is the frame back camera images users should refer to -->
-    <link name="${name}_optical_frame" type="camera"/>
-    <!-- camera -->
-    <xacro:stingrayf033c_camera_v0 name="${name}_gazebo_back_camera" image_format="${image_format}" image_topic_name="${name}/left/image"
-                            camera_info_topic_name="${name}/left/camera_info" parent="${name}_link"
-                            hfov="${hfov}" focal_length="${focal_length}"
-                            frame_id="${name}_optical_frame" hack_baseline="0"
-                            image_width="${image_width}" image_height="${image_height}">
+    <link name="${name}_optical_frame" type="camera">
+      <inertial>
+        <mass value="0.05" />
+        <inertia ixx="0"  ixy="0"  ixz="0" iyy="0"  iyz="0"  izz="0" />
+      </inertial>
+    </link>
+    <!-- back camera -->
+    <xacro:mvbluefox_camera name="${name}_gazebo_back_camera" parent="${name}_link">
       <origin xyz="0 0 0" rpy="0.0 0.0 0.0" />
-    </xacro:stingrayf033c_camera_v0>
-    <!-- extensions -->
-    <xacro:back_camera_gazebo_v0 name="${name}" focal_length="${focal_length}" hfov="${hfov}"
+    </xacro:mvbluefox_camera>
+    <!-- Back camera Gazebo simulation -->
+    <xacro:mvbluefox_back_camera_gazebo name="${name}" image_format="${image_format}"
+                                   hfov="${hfov}" focal_length="${focal_length}"
+                                   frame_id="${name}_optical_frame"
                                    image_width="${image_width}" image_height="${image_height}"/>
   </xacro:macro>

File: reem_description/urdf/sensors/hokuyo_laser_reem.gazebo.xacro (robot description, xacro)
@@ -11,18 +11,26 @@
        xmlns:interface="http://playerstage.sourceforge.net/gazebo/xmlschema/#interface"
        xmlns:xacro="http://ros.org/wiki/xacro">
-  <xacro:macro name="hokuyo_laser_reem_gazebo" params="name ros_topic update_rate min_angle max_angle">
-		<gazebo reference="${name}_link">
-      <sensor:ray name="${name}">
-        <rayCount>181</rayCount>
-        <rangeCount>181</rangeCount>
-        <laserCount>1</laserCount>
-        <displayRays>fan</displayRays>
-      	<minAngle>${min_angle}</minAngle>
-        <maxAngle>${max_angle}</maxAngle>
-        <minRange>0.1</minRange>
-        <maxRange>4</maxRange>
-        <resRange>1</resRange>
-        <updateRate>${update_rate}</updateRate>
-        <controller:gazebo_ros_laser name="gazebo_ros_${name}_controller" plugin="libgazebo_ros_laser.so">
+  <xacro:macro name="hokuyo_reem_laser_gazebo" params="name ros_topic update_rate min_angle max_angle">
+    <gazebo reference="${name}_link">
+      <sensor type="ray" name="${name}">
+        <pose>0 0 0 0 0 0</pose>
+        <update_rate>${update_rate}</update_rate>
+        <visualize>true</visualize>
+        <ray>
+          <scan>
+            <horizontal>
+              <samples>513</samples>
+              <resolution>1</resolution>
+              <min_angle>-1.35</min_angle>
+              <max_angle>1.35</max_angle>
+            </horizontal>
+          </scan>
+          <range>
+            <min>0.08</min>
+            <max>10.0</max>
+            <resolution>0.01</resolution>
+          </range>
+        </ray>
+        <plugin filename="libgazebo_ros_laser.so" name="gazebo_ros_hokuyo_laser">
           <gaussianNoise>0.005</gaussianNoise>
           <alwaysOn>true</alwaysOn>
@@ -30,9 +38,6 @@
           <topicName>${ros_topic}</topicName>
           <frameName>${name}_link</frameName>
-          <interface:laser name="gazebo_ros_${name}_iface" />
-          <hokuyoMinIntensity>101.0</hokuyoMinIntensity>
-        </controller:gazebo_ros_laser>
-      </sensor:ray>
-      <material>Gazebo/Grey</material>
+        </plugin>
+      </sensor>
     </gazebo>
   </xacro:macro>

File: reem_description/urdf/sensors/hokuyo_laser_reem.urdf.xacro (robot description, xacro)
@@ -11,15 +11,10 @@
       xmlns:interface="http://playerstage.sourceforge.net/gazebo/xmlschema/#interface"
       xmlns:xacro="http://ros.org/wiki/xacro">
+  <!--include filename="$(find reem_description)/urdf/sensors/hokuyo_laser_reem.gazebo.xacro" /-->
   <include filename="$(find reem_description)/urdf/sensors/hokuyo_laser_reem.gazebo.xacro" />
-  <xacro:macro name="hokuyo_laser_reem" params="name parent *origin ros_topic update_rate min_angle max_angle">
-   <joint name="${name}_joint" type="fixed">
-      <axis xyz="0 1 0" />
-      <insert_block name="origin" />
-      <parent link="base_link"/>
-      <child link="${name}_link"/>
-    </joint>
-  	<link name="${name}_link" type="laser">
+  <xacro:macro name="hokuyo_reem_laser" params="name parent *origin ros_topic update_rate min_angle max_angle">
+     <link name="${name}_link" type="laser">
       <inertial>
-        <mass value="0.001" />
+        <mass value="1" />
         <origin xyz="0 0 0" rpy="0 0 0" />
         <inertia ixx="0.0001" ixy="0" ixz="0" iyy="0.000001" iyz="0" izz="0.0001" />
@@ -39,6 +34,19 @@
       </collision>
     </link>
+    <joint name="${name}_joint" type="revolute">
+        <origin xyz="0.04 0 0.745" rpy="-0.03 ${52 * deg_to_rad} -0.05" />
+        <axis xyz="0 1 0"/>
+        <parent link="${parent}_link"/>
+        <child link="${name}_link"/>
+        <dynamics friction="1.0" damping="1.0"/>
+        <limit lower="0.0" upper="0.0" effort="260" velocity="6.0" />
+    </joint>
+    <transmission type="pr2_mechanism_model/SimpleTransmission" name="hokuyo_fake_trans">
+      <actuator name="${name}_fake_motor" />
+      <joint name="${name}_joint" />
+      <mechanicalReduction>1.0</mechanicalReduction>
+    </transmission>
     <!-- gazebo extensions -->
-    <xacro:hokuyo_laser_reem_gazebo name="${name}" ros_topic="${ros_topic}" update_rate="${update_rate}" min_angle="${min_angle}" max_angle="${max_angle}" />
+    <xacro:hokuyo_reem_laser_gazebo name="${name}" ros_topic="${ros_topic}" update_rate="${update_rate}" min_angle="${min_angle}" max_angle="${max_angle}" />
   </xacro:macro>
 </robot>

File: reem_description/urdf/sensors/mvbluefox_back_camera.gazebo.xacro (robot description, xacro)
@@ -1,5 +1,5 @@
 <?xml version="1.0"?>
 <!--
-  Copyright (c) 2011, PAL Robotics, S.L.
+  Copyright (c) 2013, PAL Robotics, S.L.
   All rights reserved.
   This work is licensed under the Creative Commons Attribution-NonCommercial-NoDerivs 3.0 Unported License.
@@ -7,14 +7,13 @@
   Creative Commons, 444 Castro Street, Suite 900, Mountain View, California, 94041, USA.
 -->
-<robot xmlns:sensor="http://playerstage.sourceforge.net/gazebo/xmlschema/#sensor"
+<robot name="reem" xmlns:sensor="http://playerstage.sourceforge.net/gazebo/xmlschema/#sensor"
        xmlns:controller="http://playerstage.sourceforge.net/gazebo/xmlschema/#controller"
        xmlns:interface="http://playerstage.sourceforge.net/gazebo/xmlschema/#interface"
        xmlns:xacro="http://ros.org/wiki/xacro">
-  <xacro:macro name="stingrayf033c_camera_gazebo_v0" params="name image_format image_topic_name camera_info_topic_name hfov focal_length frame_id hack_baseline image_width image_height">
-    <gazebo reference="${name}_frame">
-      <sensor type="camera" name="${name}_sensor">
+  <xacro:macro name="mvbluefox_back_camera_gazebo" params="name image_format hfov focal_length frame_id image_width image_height">
+    <gazebo reference="${name}_link">
+      <sensor type="camera" name="gazebo_${name}_camera">
         <update_rate>15.0</update_rate>
-        <camera name="${name}">
-          <pose>${hack_baseline} 0 0 0 0 0</pose>
+        <camera>
           <horizontal_fov>${ hfov }</horizontal_fov>
           <image>
@@ -22,18 +21,18 @@
             <height> ${image_height}</height>
             <format>${image_format}</format>
-         </image>
-         <clip>
-           <near>0.01</near>
-           <far>100</far>
-         </clip>
-       </camera>
-       <plugin name="${name}_controller" filename="libgazebo_ros_camera.so">
+          </image>
+          <clip>
+            <near>0.01</near>
+            <far>100</far>
+          </clip>
+        </camera>
+       <plugin name="monocular_camera_controller" filename="libgazebo_ros_camera.so">
          <alwaysOn>true</alwaysOn>
          <updateRate>15.0</updateRate>
          <cameraName>${name}</cameraName>
-         <imageTopicName>${image_topic_name}</imageTopicName>
-         <cameraInfoTopicName>${camera_info_topic_name}</cameraInfoTopicName>
+         <imageTopicName>image</imageTopicName>
+         <cameraInfoTopicName>camera_info</cameraInfoTopicName>
          <frameName>${frame_id}</frameName>
-         <hackBaseline>${hack_baseline}</hackBaseline>
+         <hackBaseline>0</hackBaseline>
          <CxPrime>${(image_width+1)/2}</CxPrime>
          <Cx>${(image_width+1)/2}</Cx>

File: reem_description/urdf/sensors/openni.gazebo.xacro (robot description, xacro)
@@ -15,24 +15,31 @@
        xmlns:interface="http://playerstage.sourceforge.net/gazebo/xmlschema/#interface"
        xmlns:xacro="http://ros.org/wiki/xacro">
-  <xacro:macro name="openni_ir_gazebo_v0" params="link_name frame_name camera_name">
-<!--    <gazebo reference="${link_name}">
-      <sensor:camera name="${name}_ir_sensor">
-        <imageFormat>L8</imageFormat>
-        <imageSize>640 480</imageSize>
-        <hfov>57</hfov>
-        <nearClip>0.01</nearClip>
-        <farClip>5</farClip>
-        <updateRate>1.0</updateRate>
-        <baseline>0.2</baseline>
-        <controller:gazebo_ros_openni_kinect name="${link_name}_controller" plugin="libgazebo_ros_openni_kinect.so">
+  <xacro:macro name="openni_camera_gazebo_v0" params="name">
+    <gazebo reference="${name}_frame">
+      <sensor type="depth" name="${name}_frame_sensor">
+        <always_on>true</always_on>
+        <update_rate>20.0</update_rate>
+        <camera>
+          <horizontal_fov>${57.0*M_PI/180.0}</horizontal_fov>
+          <image>
+            <format>R8G8B8</format>
+            <width>640</width>
+            <height>480</height>
+          </image>
+          <clip>
+            <near>0.01</near>
+            <far>5</far>
+          </clip>
+        </camera>
+        <plugin name="${name}_frame_controller" filename="libgazebo_ros_openni_kinect.so">
           <alwaysOn>true</alwaysOn>
-          <updateRate>1.0</updateRate>
-          <cameraName>${camera_name}_ir</cameraName>
-          <imageTopicName>/${camera_name}/depth/image_raw</imageTopicName>
-          <cameraInfoTopicName>/${camera_name}/depth/camera_info</cameraInfoTopicName>
-          <depthImageTopicName>/${camera_name}/depth/image_raw</depthImageTopicName>
-          <depthImageInfoTopicName>/${camera_name}/depth/camera_info</depthImageInfoTopicName>
-          <pointCloudTopicName>/${camera_name}/depth/points</pointCloudTopicName>
-          <frameName>${frame_name}</frameName>
+          <updateRate>20.0</updateRate>
+          <cameraName>${name}</cameraName>
+          <imageTopicName>ir/image_raw</imageTopicName>
+          <cameraInfoTopicName>/ir/camera_info</cameraInfoTopicName>
+          <depthImageTopicName>depth/image_raw</depthImageTopicName>
+          <depthImageCameraInfoTopicName>depth/camera_info</depthImageCameraInfoTopicName>
+          <pointCloudTopicName>depth/points</pointCloudTopicName>
+          <frameName>${name}_optical_frame</frameName>
           <pointCloudCutoff>0.5</pointCloudCutoff>
           <distortionK1>0.00000001</distortionK1>
@@ -41,26 +48,29 @@
           <distortionT1>0.00000001</distortionT1>
           <distortionT2>0.00000001</distortionT2>
-        </controller:gazebo_ros_openni_kinect>
-      </sensor:camera>
-    </gazebo>-->
-  </xacro:macro>
-  <xacro:macro name="openni_rgb_gazebo_v0" params="link_name frame_name camera_name">
-    <!--<gazebo reference="${link_name}">
-      <sensor:camera name="${name}_rgb_sensor">
-        <imageFormat>R8G8B8</imageFormat>
-        <imageSize>640 480</imageSize>
-        <hfov>57</hfov>
-        <nearClip>0.01</nearClip>
-        <farClip>5</farClip>
-        <updateRate>1.0</updateRate>
-        <baseline>0.2</baseline>
-        <controller:gazebo_ros_openni_kinect name="${link_name}_controller" plugin="libgazebo_ros_openni_kinect.so">
+        </plugin>
+      </sensor>
+      <sensor type="depth" name="${name}_frame_sensor">
+        <always_on>true</always_on>
+        <update_rate>20.0</update_rate>
+        <camera>
+          <horizontal_fov>${57.0*M_PI/180.0}</horizontal_fov>
+          <image>
+            <format>R8G8B8</format>
+            <width>640</width>
+            <height>480</height>
+          </image>
+          <clip>
+            <near>0.01</near>
+            <far>5</far>
+          </clip>
+        </camera>
+        <plugin name="${name}_frame_controller" filename="libgazebo_ros_openni_kinect.so">
           <alwaysOn>true</alwaysOn>
-          <updateRate>1.0</updateRate>
-          <cameraName>${camera_name}_rgb</cameraName>
-          <imageTopicName>/${camera_name}/rgb/image_raw</imageTopicName>
-          <cameraInfoTopicName>/${camera_name}/rgb/camera_info</cameraInfoTopicName>
-          <pointCloudTopicName>/${camera_name}/depth_registered/points</pointCloudTopicName>
-          <frameName>${frame_name}</frameName>
+          <updateRate>20.0</updateRate>
+          <cameraName>${name}</cameraName>
+          <imageTopicName>rgb/image_raw</imageTopicName>
+          <pointCloudTopicName>rgb/points</pointCloudTopicName>
+          <cameraInfoTopicName>rgb/camera_info</cameraInfoTopicName>
+          <frameName>${name}_optical_frame</frameName>
           <pointCloudCutoff>0.5</pointCloudCutoff>
           <distortionK1>0.00000001</distortionK1>
@@ -69,7 +79,7 @@
           <distortionT1>0.00000001</distortionT1>
           <distortionT2>0.00000001</distortionT2>
-        </controller:gazebo_ros_openni_kinect>
-      </sensor:camera>
-    </gazebo>-->
+        </plugin>
+      </sensor>
+    </gazebo>
   </xacro:macro>
 </robot>

File: reem_description/urdf/sensors/range.gazebo.xacro (robot description, xacro)
@@ -13,25 +13,39 @@
   <xacro:macro name="range_reem_gazebo" params="name ros_topic update_rate maxRange minRange fov radiation" >
     <gazebo reference="${name}_link">
-      <sensor:ray name="${name}">
-        <rayCount>5</rayCount>
-        <rangeCount>5</rangeCount>
-        <verticalRayCount>5</verticalRayCount>
-        <verticalRangeCount>5</verticalRangeCount>
-        <minAngle>-${fov/2}</minAngle>
-        <verticalMinAngle>-${fov/2}</verticalMinAngle>
-        <maxAngle>${fov/2}</maxAngle>
-        <verticalMaxAngle>${fov/2}</verticalMaxAngle>
-        <minRange>${minRange}</minRange>
-        <maxRange>${maxRange}</maxRange>
-        <resRange>0.01</resRange>
-        <updateRate>${update_rate}</updateRate>
-        <controller:gazebo_ros_sonar name="gazebo_ros_${name}_controller" plugin="libgazebo_ros_sonar.so">
+      <sensor type="ray" name="${name}">
+        <pose>0 0 0 0 0 0</pose>
+        <update_rate>${update_rate}</update_rate>
+        <visualize>false</visualize>
+        <ray>
+          <scan>
+            <horizontal>
+              <samples>5</samples>
+              <resolution>1</resolution>
+              <min_angle>-${fov/2}</min_angle>
+              <max_angle>${fov/2}</max_angle>
+            </horizontal>
+            <vertical>
+              <samples>5</samples>
+              <resolution>1</resolution>
+              <min_angle>-${fov/2}</min_angle>
+              <max_angle>${fov/2}</max_angle>
+            </vertical>
+          </scan>
+          <range>
+            <min>${minRange}</min>
+            <max>${maxRange}</max>
+            <resolution>0.01</resolution>
+          </range>
+        </ray>
+        <plugin filename="libgazebo_ros_range.so" name="gazebo_ros_range">
           <gaussianNoise>0.005</gaussianNoise>
+          <alwaysOn>true</alwaysOn>
+          <updateRate>${update_rate}</updateRate>
           <topicName>${ros_topic}</topicName>
-          <frameId>${name}_link</frameId>
+          <frameName>${name}_link</frameName>
           <fov>${fov}</fov>
           <radiation>${radiation}</radiation>
-        </controller:gazebo_ros_sonar>
-      </sensor:ray>
+        </plugin>
+      </sensor>
     </gazebo>
   </xacro:macro>

File: reem_description/urdf/sensors/range.urdf.xacro (robot description, xacro)
@@ -13,11 +13,5 @@
   <include filename="$(find reem_description)/urdf/sensors/range.gazebo.xacro" />
   <xacro:macro name="range_reem" params="name parent *origin ros_topic update_rate maxRange minRange fov radiation">
-    <joint name="${name}_joint" type="fixed">
-      <axis xyz="0 0 0" rpy="0 0 0"/>
-      <insert_block name="origin" />
-      <parent link="${parent}_link"/>
-      <child link="${name}_link"/>
-    </joint>
-    <link name="${name}_link" type="irarray">
+    <link name="${name}_link">
       <inertial>
         <mass value="0.001" />
@@ -26,4 +20,10 @@
       </inertial>
     </link>
+    <joint name="${name}_joint" type="fixed">
+      <insert_block name="origin" />
+      <axis xyz="0 0 1"/>
+      <parent link="${parent}_link"/>
+      <child link="${name}_link"/>
+    </joint>
     <!-- gazebo extensions -->
     <xacro:range_reem_gazebo name="${name}" ros_topic="${ros_topic}" update_rate="${update_rate}" maxRange="${maxRange}" minRange="${minRange}" fov="${fov}" radiation="${radiation}"/>
