Commit message: Update sensors to Gazebo 1.5.

File: reem_description/urdf/sensors/sick_laser_reem.gazebo.xacro (robot description, xacro)
@@ -11,19 +11,26 @@
        xmlns:interface="http://playerstage.sourceforge.net/gazebo/xmlschema/#interface"
        xmlns:xacro="http://ros.org/wiki/xacro">
-  <xacro:macro name="sick_laser_reem_gazebo" params="name ros_topic update_rate min_angle max_angle">
-		<gazebo reference="${name}_link">
-      <sensor:ray name="${name}">
-        <rayCount>240</rayCount>
-        <rangeCount>240</rangeCount>
-	<!--			<rangeCount>181</rangeCount> -->
-        <laserCount>1</laserCount>
-        <displayRays>fan</displayRays>
-      	<minAngle>${min_angle}</minAngle>
-        <maxAngle>${max_angle}</maxAngle>
-        <minRange>0.1</minRange>
-        <maxRange>19</maxRange>
-        <resRange>1</resRange>
-        <updateRate>${update_rate}</updateRate>
-        <controller:gazebo_ros_laser name="gazebo_ros_${name}_controller" plugin="libgazebo_ros_laser.so">
+  <xacro:macro name="sick_reem_laser_gazebo" params="name ros_topic update_rate min_angle max_angle">
+    <gazebo reference="${name}_link">
+      <sensor type="ray" name="${name}">
+        <pose>0 0 0 0 0 0</pose>
+        <update_rate>${update_rate}</update_rate>
+        <visualize>true</visualize>
+        <ray>
+          <scan>
+            <horizontal>
+              <samples>513</samples>
+              <resolution>1</resolution>
+              <min_angle>${min_angle}</min_angle>
+              <max_angle>${max_angle}</max_angle>
+            </horizontal>
+          </scan>
+          <range>
+            <min>0.08</min>
+            <max>10.0</max>
+            <resolution>0.01</resolution>
+          </range>
+        </ray>
+        <plugin filename="libgazebo_ros_laser.so" name="gazebo_ros_sick_laser">
           <gaussianNoise>0.005</gaussianNoise>
           <alwaysOn>true</alwaysOn>
@@ -31,9 +38,6 @@
           <topicName>${ros_topic}</topicName>
           <frameName>${name}_link</frameName>
-          <interface:laser name="gazebo_ros_${name}_iface" />
-          <hokuyoMinIntensity>101.0</hokuyoMinIntensity>
-        </controller:gazebo_ros_laser>
-      </sensor:ray>
-      <material>Gazebo/Grey</material>
+        </plugin>
+      </sensor>
     </gazebo>
   </xacro:macro>

File: reem_description/urdf/sensors/sick_laser_reem.urdf.xacro (robot description, xacro)
@@ -11,15 +11,10 @@
       xmlns:interface="http://playerstage.sourceforge.net/gazebo/xmlschema/#interface"
       xmlns:xacro="http://ros.org/wiki/xacro">
+  <!--include filename="$(find reem_description)/urdf/sensors/hokuyo_laser_reem.gazebo.xacro" /-->
   <include filename="$(find reem_description)/urdf/sensors/sick_laser_reem.gazebo.xacro" />
-  <xacro:macro name="sick_laser_reem" params="name parent *origin ros_topic update_rate min_angle max_angle">
-   <joint name="${name}_joint" type="fixed">
-      <axis xyz="0 1 0" />
-      <insert_block name="origin" />
-      <parent link="base_link"/>
-      <child link="${name}_link"/>
-    </joint>
-  	<link name="${name}_link" type="laser">
+  <xacro:macro name="sick_reem_laser" params="name parent *origin ros_topic update_rate min_angle max_angle">
+     <link name="${name}_link" type="laser">
       <inertial>
-        <mass value="0.001" />
+        <mass value="1" />
         <origin xyz="0 0 0" rpy="0 0 0" />
         <inertia ixx="0.0001" ixy="0" ixz="0" iyy="0.000001" iyz="0" izz="0.0001" />
@@ -28,5 +23,5 @@
         <origin xyz="0 0 0" rpy="0 0 0" />
         <geometry>
-          <box size="0.105 0.105 0.11" />
+          <box size="0.05 0.05 0.05" />
         </geometry>
         <material name="DarkGrey" />
@@ -35,12 +30,16 @@
         <origin xyz="0 0 0" rpy="0 0 0" />
         <geometry>
-          <box size="0.105 0.105 0.11" />
+          <box size=".05 .05 .05" />
         </geometry>
-      </collision >
+      </collision>
     </link>
-    <gazebo reference="${name}_link">
-    </gazebo>
+    <joint name="${name}_joint" type="fixed">
+      <axis xyz="0 1 0" />
+      <insert_block name="origin" />
+      <parent link="base_link"/>
+      <child link="${name}_link"/>
+    </joint>
     <!-- gazebo extensions -->
-    <xacro:sick_laser_reem_gazebo name="${name}" ros_topic="${ros_topic}" update_rate="${update_rate}" min_angle="${min_angle}" max_angle="${max_angle}" />
+    <xacro:sick_reem_laser_gazebo name="${name}" ros_topic="${ros_topic}" update_rate="${update_rate}" min_angle="${min_angle}" max_angle="${max_angle}" />
   </xacro:macro>
 </robot>

File: reem_description/urdf/sensors/stereo_camera.urdf.xacro (robot description, xacro)
@@ -13,5 +13,4 @@
   <!-- stereo camera macro uses stingrayf033c_camera macros -->
   <include filename="$(find reem_description)/urdf/sensors/stingrayf033c_camera.urdf.xacro" />
-  <include filename="$(find reem_description)/urdf/sensors/stereo_camera.gazebo.xacro" />
   <property name="stereo_dx" value="0.00" />
   <property name="stereo_dy" value="-0.073" /> <!-- stereo baseline according to stereo_link which has X pointing forward, Y leftwards and Z upwards (required by Gazebo for a camera sensor) -->
@@ -82,9 +81,4 @@
       <origin xyz="${stereo_dx} ${stereo_dy} ${stereo_dz}" rpy="${stereo_rx} ${stereo_ry} ${stereo_rz}" />
     </xacro:stingrayf033c_camera_v0>
-    <!-- extensions -->
-    <xacro:stereo_camera_gazebo_v0 name="${name}"
-                                   focal_length_left="${focal_length_left}" hfov_left="${hfov_left}"
-                                   focal_length_right="${focal_length_right}" hfov_right="${hfov_right}"
-                                   image_width="${image_width}" image_height="${image_height}"/>
   </xacro:macro>
 </robot>

File: reem_description/urdf/sensors/stingrayf033c_camera.urdf.xacro (robot description, xacro)
@@ -30,8 +30,9 @@
       </inertial>
       <visual>
-        <origin xyz="0 0 0" rpy="0 0 0" />
+        <origin xyz="-0.01 0 0" rpy="0 ${deg_to_rad * 90} 0" />
         <geometry>
-          <box size="0.01 0.01 0.01" />
+          <cylinder radius="0.01" length="0.02" />
         </geometry>
+        <material name="Blue" />
       </visual>
       <!--

File: reem_description/urdf/sensors/xtion_pro_live.urdf.xacro (robot description, xacro)
@@ -23,14 +23,12 @@
   <include filename="$(find reem_description)/urdf/sensors/calibration.xacro" />
   <include filename="$(find reem_description)/urdf/sensors/openni.gazebo.xacro" />
-  <property name="M_PI" value="3.1415926535897931" />
   <!-- Macro -->
   <xacro:macro name="xtion_pro_live" params="name parent *origin *calibration_origin">
-    <!-- base link -->
-    <joint name="${name}_joint" type="fixed">
+    <joint name="${name}_frame_joint" type="fixed">
       <insert_block name="origin" />
       <parent link="${parent}"/>
-      <child link="${name}_link"/>
+      <child link="${name}_frame"/>
     </joint>
-    <link name="${name}_link">
+    <link name="${name}_frame">
       <inertial>
         <mass value="0.01" />
@@ -56,14 +54,10 @@
       </collision>
     </link>
-    <!-- Xtion IR sensor physical attachment -->
-    <joint name="${name}_ir_joint" type="fixed">
-      <!-- This relates the IR sensor to the Xtion base link -->
-      <!-- 4.8 cm because sensors are offset to right, from center -->
-      <origin xyz="0 0.048 0" rpy="0 0 0"/>
-      <parent link="${name}_link"/>
-      <child link="${name}_ir_link"/>
+    <joint name="${name}_optical_joint" type="fixed">
+      <insert_block name="calibration_origin" />
+      <parent link="${name}_frame"/>
+      <child link="${name}_optical_frame"/>
     </joint>
-    <link name="${name}_ir_link">
-      <!-- This link is the reference for the IR sensor in Gazebo, so it has inertia properties -->
+    <link name="${name}_optical_frame">
       <inertial>
         <mass value="0.01" />
@@ -74,55 +68,6 @@
       </inertial>
     </link>
-    <!-- Xtion IR sensor frame -->
-    <joint name="${name}_ir_optical_frame_joint" type="fixed">
-      <insert_block name="calibration_origin" /> <!-- macro argument -->
-      <parent link="${name}_ir_link"/>
-      <child link="${name}_ir_optical_frame"/>
-    </joint>
-    <link name="${name}_ir_optical_frame">
-      <inertial>
-        <mass value="0.01" />
-        <origin xyz="0 0 0" rpy="0 0 0"/>
-        <inertia ixx="0.0"  ixy="0.0"  ixz="0.0"
-                 iyy="0.0"  iyz="0.0"
-                 izz="0.0" />
-      </inertial>
-    </link>
-    <!-- OpenNI IR sensor Gazebo extensions -->
-    <xacro:openni_ir_gazebo_v0 link_name="${name}_ir_link" frame_name="${name}_ir_optical_frame" camera_name="${name}" />
-    <!-- Xtion RGB sensor physical attachment -->
-    <joint name="${name}_rgb_joint" type="fixed">
-      <!-- The measured distance from RGB lens back to IR lens, approx 2.5cm, but PR2 is using 3.0cm -->
-      <origin xyz="0 -0.025 0" rpy="0 0 0"/>
-      <parent link="${name}_ir_link"/>
-      <child link="${name}_rgb_link"/>
-    </joint>
-    <link name="${name}_rgb_link" >
-      <!-- This link is the reference for the RGB sensor in Gazebo, so it has inertia properties -->
-      <inertial>
-        <mass value="0.01" />
-        <origin xyz="0 0 0" rpy="0 0 0"/>
-        <inertia ixx="0.0"  ixy="0.0"  ixz="0.0"
-                 iyy="0.0"  iyz="0.0"
-                 izz="0.0" />
-      </inertial>
-    </link>
-    <!-- Xtion RGB sensor frame -->
-    <joint name="${name}_rgb_optical_frame_joint" type="fixed">
-      <insert_block name="calibration_origin" /> <!-- macro argument -->
-      <parent link="${name}_rgb_link"/>
-      <child link="${name}_rgb_optical_frame"/>
-    </joint>
-    <link name="${name}_rgb_optical_frame">
-       <inertial>
-        <mass value="0.01" />
-        <origin xyz="0 0 0" rpy="0 0 0"/>
-        <inertia ixx="0.0"  ixy="0.0"  ixz="0.0"
-                 iyy="0.0"  iyz="0.0"
-                 izz="0.0" />
-      </inertial>
-    </link>
-    <!-- OpenNI RGB sensor Gazebo extensions -->
-    <xacro:openni_rgb_gazebo_v0 link_name="${name}_rgb_link" frame_name="${name}_rgb_optical_frame" camera_name="${name}" />
+    <!-- extensions -->
+    <xacro:openni_camera_gazebo_v0 name="${name}" />
   </xacro:macro>
 </robot>
