Commit message: Update RGBD sensor location.
Patch by David Butterworth.

File: reem_description/robots/reem_rgbd.urdf.xacro (robot description, xacro)
@@ -17,6 +17,6 @@
   <include filename="$(find reem_description)/urdf/sensors/xtion_pro_live.urdf.xacro" />
   <xacro:xtion_pro_live parent="head_2_link" name="head_mount_xtion" > <!-- name is appended to create link and topic names -->
-     <origin xyz="0.056 -0.252 0.0" rpy="${M_PI/2} 0.0 0.34906" /> <!-- 0.252   = height above neck joint
-                                                                        0.34906 = pitch angle downwards   -->
+     <origin xyz="0.1 -0.252 0.0" rpy="${M_PI/2} 0.0 1.0" /> <!-- 0.252   = height above neck joint
+                                                                  1.0 = pitch angle downwards   -->
      <origin xyz="${cal_head_mount_xtion_x}
                   ${cal_head_mount_xtion_y}
