Commit message: Update urdf to use new hand visualization.

File: reem_description/urdf/hand/hand.gazebo.xacro (robot description, xacro)
@@ -13,5 +13,4 @@
     <xacro:macro name="hand_gazebo" params="name">
     <gazebo reference="${name}_link">
-      <material>Gazebo/White</material>
       <turnGravityOff>false</turnGravityOff>
     </gazebo>

File: reem_description/urdf/hand/hand.urdf.xacro (robot description, xacro)
@@ -35,5 +35,5 @@
         <origin xyz="0 0 0" rpy="0 0 0" />
         <geometry>
-          <mesh filename="package://reem_description/meshes/hand/hand_finger_1.stl" scale="1 1 ${-reflect * finger_reflect}" />
+          <mesh filename="package://reem_description/meshes/hand/hand_finger_1.dae" scale="1 1 ${-reflect * finger_reflect}" />
         </geometry>
         <material name="LightGrey" />
@@ -64,5 +64,5 @@
         <origin xyz="0 0 0" rpy="0 0 0" />
         <geometry>
-          <mesh filename="package://reem_description/meshes/hand/hand_finger_2.stl" scale="1 1 ${-reflect * finger_reflect }" />
+          <mesh filename="package://reem_description/meshes/hand/hand_finger_2.dae" scale="1 1 ${-reflect * finger_reflect }" />
         </geometry>
         <material name="LightGrey" />
@@ -93,5 +93,5 @@
         <origin xyz="0 0 0" rpy="0 0 0" />
         <geometry>
-          <mesh filename="package://reem_description/meshes/hand/hand_finger_3.stl" scale="1 1 ${-reflect * finger_reflect}" />
+          <mesh filename="package://reem_description/meshes/hand/hand_finger_3.dae" scale="1 1 ${-reflect * finger_reflect}" />
         </geometry>
         <material name="LightGrey" />
@@ -128,5 +128,5 @@
         <origin xyz="0 0 0" rpy="0 0 0" />
         <geometry>
-          <mesh filename="package://reem_description/meshes/hand/hand_palm.stl" scale="1 ${-reflect} 1" />
+          <mesh filename="package://reem_description/meshes/hand/hand_palm.dae" scale="1 ${-reflect} 1" />
         </geometry>
         <material name="LightGrey" />
@@ -158,5 +158,5 @@
         <origin xyz="0 0 0" rpy="0 0 0" />
         <geometry>
-          <mesh filename="package://reem_description/meshes/hand/hand_thumb.stl" scale="1 1 ${-reflect}" />
+          <mesh filename="package://reem_description/meshes/hand/hand_thumb.dae" scale="1 1 ${-reflect}" />
         </geometry>
         <material name="LightGrey" />

Commit message: Added the generic grasp hack of fuerte for the RH3 hands using the tag gripper

File: reem_description/urdf/hand/hand.gazebo.xacro (robot description, xacro)
@@ -17,3 +17,18 @@
     </gazebo>
     </xacro:macro>
+    <xacro:macro name="hand_grasping_hack" params="side">
+      <gazebo>
+      <!-- a formal implementation of grasp hack in gazebo with fixed joint reference: /opt/ros/fuerte/stacks/pr2_common/pr2_description/urdf/gripper_v0/gripper.gazebo.xacro -->
+        <gripper name="${side}_grasp_hack">
+          <grasp_check attach_steps="20" detach_steps="40" min_contact_count="2" />
+          <gripper_link>hand_${side}_middle_1_link</gripper_link>
+          <gripper_link>hand_${side}_index_1_link</gripper_link>
+          <gripper_link>hand_${side}_middle_2_link</gripper_link>
+          <gripper_link>hand_${side}_index_2_link</gripper_link>
+          <gripper_link>hand_${side}_middle_3_link</gripper_link>
+          <gripper_link>hand_${side}_index_3_link</gripper_link>
+          <palm_link>hand_${side}_thumb_link</palm_link>
+        </gripper>
+      </gazebo>
+    </xacro:macro>
 </robot>

File: reem_description/urdf/hand/hand.urdf.xacro (robot description, xacro)
@@ -178,4 +178,6 @@
     <!-- Middle finger -->
     <xacro:reem_finger hand_name="${name}" hand_side="${side}" hand_reflect="${reflect}" finger_name="middle" finger_reflect="-1"/>
+    <!-- grasping hack -->
+    <xacro:hand_grasping_hack side="${side}" />
   </xacro:macro>
 </robot>
