Commit message: Hand collision geometry no longer generated.

File: reem_description/urdf/hand/hand.urdf.xacro (robot description, xacro)
@@ -31,5 +31,5 @@
         <origin xyz="0 0 0" rpy="0 0 0" />
         <geometry>
-          <mesh filename="package://reem_description/meshes/hand/convex/hand_${side}_low_convex.stlb" />
+          <mesh filename="package://reem_description/meshes/hand/hand_${side}_low_convex.stlb" />
         </geometry>
       </collision>

Commit message: Set hand joint limits, fix right thumb orientation.

File: reem_description/urdf/hand/hand.urdf.xacro (robot description, xacro)
@@ -51,5 +51,5 @@
       <origin xyz="0.00357 -0.04084 0" rpy="0 0 0" />
       <axis xyz="0 0 1" />
-      <limit lower="${0.0 * deg_to_rad}" upper="${90.0 * deg_to_rad}" effort="0.0" velocity="${hand_max_vel}" />
+      <limit lower="${0.0 * deg_to_rad}" upper="${80.0 * deg_to_rad}" effort="0.0" velocity="${hand_max_vel}" />
       <dynamics friction="${hand_friction}" damping="${hand_damping}"/>
       <mimic joint="${hand_name}_${hand_side}_${finger_name}_1_joint" multiplier="1" offset="0"/>
@@ -80,5 +80,5 @@
       <origin xyz="0.00572 -0.0269 0" rpy="0 0 0" />
       <axis xyz="0 0 1" />
-      <limit lower="${0.0 * deg_to_rad}" upper="${90.0 * deg_to_rad}" effort="0.0" velocity="${hand_max_vel}" />
+      <limit lower="${0.0 * deg_to_rad}" upper="${80.0 * deg_to_rad}" effort="0.0" velocity="${hand_max_vel}" />
       <dynamics friction="${hand_friction}" damping="${hand_damping}"/>
       <mimic joint="${hand_name}_${hand_side}_${finger_name}_2_joint" multiplier="1" offset="0"/>
@@ -120,5 +120,6 @@
     <link name="${name}_${side}_palm_link">
       <inertial>
-        <origin xyz="0.07547 0.00468 0.00291" rpy="0 0 0" />
+        <!--<origin xyz="0.07547 0.00468 0.00291" rpy="0 0 0" />-->  <!--TODO: Figure out why CoM is not properly displayed in Gazebo!-->
+        <origin xyz="0 0 0" rpy="0 0 0" />
         <mass value="0.91066" />
         <inertia ixx="0"  ixy="0"  ixz="0" iyy="0" iyz="0" izz="0" />
@@ -143,7 +144,7 @@
       <parent link="${name}_${side}_palm_link" />
       <child link="${name}_${side}_thumb_link" />
-      <origin xyz="0.03649 ${reflect * 0.008}  0.02" rpy="0 ${(90.0 + 13) * deg_to_rad} ${reflect * 13.0 * deg_to_rad}" />
+      <origin xyz="0.03649 ${reflect * 0.008}  0.02" rpy="${(90.0 + reflect * 90.0) * deg_to_rad} ${(90.0 + 13) * deg_to_rad} ${reflect * 13.0 * deg_to_rad}" />
       <axis xyz="0 0 1" />
-      <limit lower="${0.0 * deg_to_rad}" upper="${90.0 * deg_to_rad}" effort="0.0" velocity="${hand_max_vel}" />
+      <limit lower="${0.0 * deg_to_rad}" upper="${92.0 * deg_to_rad}" effort="0.0" velocity="${hand_max_vel}" />
       <dynamics friction="${hand_friction}" damping="${hand_damping}"/>
     </joint>
@@ -157,5 +158,5 @@
         <origin xyz="0 0 0" rpy="0 0 0" />
         <geometry>
-          <mesh filename="package://reem_description/meshes/hand/hand_thumb.stl" scale="1 ${-reflect} 1" />
+          <mesh filename="package://reem_description/meshes/hand/hand_thumb.stl" scale="1 1 ${-reflect}" />
         </geometry>
         <material name="LightGrey" />
@@ -164,5 +165,5 @@
         <origin xyz="0 0 0" rpy="0 0 0" />
         <geometry>
-          <mesh filename="package://reem_description/meshes/hand/hand_thumb_collision.stl" scale="1 ${-reflect} 1" />
+          <mesh filename="package://reem_description/meshes/hand/hand_thumb_collision.stl" scale="1 1 ${-reflect}" />
         </geometry>
       </collision>

Commit message: Removed 2 mimic joints & restored joint limits. The mimic joint functionality does not work in Gazebo, they act like a non-actuated joint with some friction behaviour. Mimic joints only work with the Fake Joint State Publisher GUI. The related joint limits for digits 2 & 3 were restored, so they can be controlled.

File: reem_description/urdf/hand/hand.urdf.xacro (robot description, xacro)
@@ -51,8 +51,6 @@
       <origin xyz="0.00357 -0.04084 0" rpy="0 0 0" />
       <axis xyz="0 0 1" />
-<!--       <limit lower="${0.0 * deg_to_rad}" upper="${80.0 * deg_to_rad}" effort="1.0" velocity="${hand_max_vel}" /> --> <!--TODO: Restore!-->
-      <limit lower="${0.0 * deg_to_rad}" upper="${1.0 * deg_to_rad}" effort="1.0" velocity="${hand_max_vel}" />
+      <limit lower="${0.0 * deg_to_rad}" upper="${80.0 * deg_to_rad}" effort="1.0" velocity="${hand_max_vel}" />
       <dynamics friction="${hand_friction}" damping="${hand_damping}"/>
-      <mimic joint="${hand_name}_${hand_side}_${finger_name}_1_joint" multiplier="1" offset="0"/>
     </joint>
     <link name="${hand_name}_${hand_side}_${finger_name}_2_link">
@@ -81,8 +79,7 @@
       <origin xyz="0.00572 -0.0269 0" rpy="0 0 0" />
       <axis xyz="0 0 1" />
-      <!--<limit lower="${0.0 * deg_to_rad}" upper="${80.0 * deg_to_rad}" effort="1.0" velocity="${hand_max_vel}" />--> <!--TODO: Restore!-->
+      <limit lower="${0.0 * deg_to_rad}" upper="${80.0 * deg_to_rad}" effort="1.0" velocity="${hand_max_vel}" />
       <limit lower="${0.0 * deg_to_rad}" upper="${1.0 * deg_to_rad}" effort="1.0" velocity="${hand_max_vel}" />
       <dynamics friction="${hand_friction}" damping="${hand_damping}"/>
-      <mimic joint="${hand_name}_${hand_side}_${finger_name}_2_joint" multiplier="1" offset="0"/>
     </joint>
     <link name="${hand_name}_${hand_side}_${finger_name}_3_link">

Commit message: Added 10mm offset to thumbs. The offset is a separate number, so it is easily recognizable. The macro change has been tested with both left & right sides.

File: reem_description/urdf/hand/hand.urdf.xacro (robot description, xacro)
@@ -143,5 +143,6 @@
       <parent link="${name}_${side}_palm_link" />
       <child link="${name}_${side}_thumb_link" />
-      <origin xyz="0.03649 ${reflect * 0.008}  0.02" rpy="${(90.0 + reflect * 90.0) * deg_to_rad} ${(90.0 + 13) * deg_to_rad} ${reflect * 13.0 * deg_to_rad}" />
+      <!-- added 10mm offset along y-axis -->
+      <origin xyz="0.03649 ${reflect*0.008 + reflect*0.010}  0.02" rpy="${(90.0 + reflect * 90.0) * deg_to_rad} ${(90.0 + 13) * deg_to_rad} ${reflect * 13.0 * deg_to_rad}" />
       <axis xyz="0 0 1" />
 <!--       <limit lower="${0.0 * deg_to_rad}" upper="${92.0 * deg_to_rad}" effort="2.0" velocity="${hand_max_vel}" /> -->

Commit message: Added optional visual for thumb extension. This temporary addition matches the real hand, so the thumb does not appear to be hanging in mid-air.

File: reem_description/urdf/hand/hand.urdf.xacro (robot description, xacro)
@@ -170,4 +170,26 @@
       </collision>
     </link>
+   <!-- Temporary visual for 10mm thumb offset -->
+   <!-- (there is no collision geometry, but you must still disable collision checking for this link) -->
+    <joint name="${name}_${side}_thumb_extension_joint" type="fixed">
+      <parent link="${name}_${side}_thumb_link" />
+      <child link="${name}_${side}_thumb_extension_link" />
+      <origin xyz="-0.014 -0.002 ${reflect*0.008}" rpy="0 0 0" /> <!-- centered in middle of the gap, 8mm back, 2mm down -->
+      <axis xyz="0 0 1" />
+    </joint>
+    <link name="${name}_${side}_thumb_extension_link">
+      <inertial>
+        <origin xyz="0 0 0" rpy="0 0 0" />
+        <mass value="0.01" />
+        <inertia ixx="0"  ixy="0"  ixz="0" iyy="0" iyz="0" izz="0" />
+      </inertial>
+      <visual>
+        <origin xyz="0 0 0" rpy="0 0 0" />
+        <geometry>
+          <box size="0.012 0.015 0.015"/> <!-- visual is 12mm long and 16mm square -->
+        </geometry>
+        <material name="White" />
+      </visual>
+    </link>
     <xacro:hand_gazebo name="${name}_${side}_thumb"/>
     <xacro:hand_simple_transmission name="${name}_${side}_thumb" reduction="168" />

Commit message: Added hand_{side}_grasping_frame links to hand. The grasp planner will approach the center of an object along the x-axis of this frame.

File: reem_description/urdf/hand/hand.urdf.xacro (robot description, xacro)
@@ -200,4 +200,20 @@
     <!-- grasping hack -->
     <xacro:hand_grasping_hack side="${side}" />
+    <!-- Grasping frame -->
+    <!-- grasp planner will approach along x-axis -->
+    <joint name="${name}_${side}_grasping_frame_joint" type="fixed">
+      <parent link="${name}_${side}_palm_link" />
+      <child link="${name}_${side}_grasping_frame" />
+      <origin xyz="0.0 ${reflect * 0.054} 0.018" rpy="0 0 0" />
+    </joint>
+    <link name="${name}_${side}_grasping_frame">
+      <inertial>
+        <origin xyz="0 0 0" rpy="0 0 0" />
+        <mass value="0.01" />  <!-- matrix below must not be zero, or Gazebo won't load -->
+        <inertia ixx="0.1"  ixy="0.0"  ixz="0.0"
+                 iyy="0.1"  iyz="0.0"
+                 izz="0.1" />
+      </inertial>
+    </link>
   </xacro:macro>
 </robot>

Commit message: Fixed finger joint limit.

File: reem_description/urdf/hand/hand.urdf.xacro (robot description, xacro)
@@ -80,5 +80,4 @@
       <axis xyz="0 0 1" />
       <limit lower="${0.0 * deg_to_rad}" upper="${80.0 * deg_to_rad}" effort="1.0" velocity="${hand_max_vel}" />
-      <limit lower="${0.0 * deg_to_rad}" upper="${1.0 * deg_to_rad}" effort="1.0" velocity="${hand_max_vel}" />
       <dynamics friction="${hand_friction}" damping="${hand_damping}"/>
     </joint>
@@ -146,5 +145,4 @@
       <origin xyz="0.03649 ${reflect*0.008 + reflect*0.010}  0.02" rpy="${(90.0 + reflect * 90.0) * deg_to_rad} ${(90.0 + 13) * deg_to_rad} ${reflect * 13.0 * deg_to_rad}" />
       <axis xyz="0 0 1" />
-<!--       <limit lower="${0.0 * deg_to_rad}" upper="${92.0 * deg_to_rad}" effort="2.0" velocity="${hand_max_vel}" /> -->
       <limit lower="${0.0 * deg_to_rad}" upper="${90.0 * deg_to_rad}" effort="2.0" velocity="${hand_max_vel}" /> <!--TODO: Restore!-->
       <dynamics friction="${hand_friction}" damping="${hand_damping}"/>

Commit message: Apply thumb offset.wq

File: reem_description/urdf/hand/hand.urdf.xacro (robot description, xacro)
@@ -156,5 +156,5 @@
       </inertial>
       <visual>
-        <origin xyz="0 0 0" rpy="0 0 0" />
+        <origin xyz="-0.015 0 0" rpy="0 0 0" /> <!--NOTE: Apply offset-->
         <geometry>
           <mesh filename="package://reem_description/meshes/hand/hand_thumb.dae" scale="1 1 ${-reflect}" />
@@ -163,5 +163,5 @@
       </visual>
       <collision>
-        <origin xyz="0 0 0" rpy="0 0 0" />
+        <origin xyz="-0.015 0 0" rpy="0 0 0" /> <!--NOTE: Apply offset-->
         <geometry>
           <mesh filename="package://reem_description/meshes/hand/hand_thumb_collision.stl" scale="1 1 ${-reflect}" />

Commit message: Re-enable last two finder joints.

File: reem_description/urdf/hand/hand.urdf.xacro (robot description, xacro)
@@ -51,8 +51,6 @@
       <origin xyz="0.00357 -0.04084 0" rpy="0 0 0" />
       <axis xyz="0 0 1" />
-<!--       <limit lower="${0.0 * deg_to_rad}" upper="${80.0 * deg_to_rad}" effort="1.0" velocity="${hand_max_vel}" /> --> <!--TODO: Restore!-->
-      <limit lower="${0.0 * deg_to_rad}" upper="${1.0 * deg_to_rad}" effort="1.0" velocity="${hand_max_vel}" />
+      <limit lower="${0.0 * deg_to_rad}" upper="${80.0 * deg_to_rad}" effort="1.0" velocity="${hand_max_vel}" />
       <dynamics friction="${hand_friction}" damping="${hand_damping}"/>
-      <mimic joint="${hand_name}_${hand_side}_${finger_name}_1_joint" multiplier="1" offset="0"/>
     </joint>
     <link name="${hand_name}_${hand_side}_${finger_name}_2_link">
@@ -81,8 +79,6 @@
       <origin xyz="0.00572 -0.0269 0" rpy="0 0 0" />
       <axis xyz="0 0 1" />
-      <!--<limit lower="${0.0 * deg_to_rad}" upper="${80.0 * deg_to_rad}" effort="1.0" velocity="${hand_max_vel}" />--> <!--TODO: Restore!-->
-      <limit lower="${0.0 * deg_to_rad}" upper="${1.0 * deg_to_rad}" effort="1.0" velocity="${hand_max_vel}" />
+      <limit lower="${0.0 * deg_to_rad}" upper="${80.0 * deg_to_rad}" effort="1.0" velocity="${hand_max_vel}" />
       <dynamics friction="${hand_friction}" damping="${hand_damping}"/>
-      <mimic joint="${hand_name}_${hand_side}_${finger_name}_2_joint" multiplier="1" offset="0"/>
     </joint>
     <link name="${hand_name}_${hand_side}_${finger_name}_3_link">
@@ -145,6 +141,5 @@
       <origin xyz="0.03649 ${reflect * 0.008}  0.02" rpy="${(90.0 + reflect * 90.0) * deg_to_rad} ${(90.0 + 13) * deg_to_rad} ${reflect * 13.0 * deg_to_rad}" />
       <axis xyz="0 0 1" />
-<!--       <limit lower="${0.0 * deg_to_rad}" upper="${92.0 * deg_to_rad}" effort="2.0" velocity="${hand_max_vel}" /> -->
-      <limit lower="${0.0 * deg_to_rad}" upper="${90.0 * deg_to_rad}" effort="2.0" velocity="${hand_max_vel}" /> <!--TODO: Restore!-->
+      <limit lower="${0.0 * deg_to_rad}" upper="${90.0 * deg_to_rad}" effort="2.0" velocity="${hand_max_vel}" />
       <dynamics friction="${hand_friction}" damping="${hand_damping}"/>
     </joint>

Commit message: Add grasping frame.
Patch by David Butterworth.

File: reem_description/urdf/hand/hand.urdf.xacro (robot description, xacro)
@@ -164,4 +164,20 @@
       </collision>
     </link>
+    <!-- Grasping frame -->
+    <!-- grasp planner will approach along x-axis -->
+    <joint name="${name}_${side}_grasping_frame_joint" type="fixed">
+      <parent link="${name}_${side}_palm_link" />
+      <child link="${name}_${side}_grasping_frame" />
+      <origin xyz="0.0 ${reflect * 0.054} 0.018" rpy="0 0 0" />
+    </joint>
+    <link name="${name}_${side}_grasping_frame">
+      <inertial>
+        <origin xyz="0 0 0" rpy="0 0 0" />
+        <mass value="0.01" /> <!-- matrix below must not be zero, or Gazebo won't load -->
+        <inertia ixx="0.1" ixy="0.0" ixz="0.0"
+                 iyy="0.1" iyz="0.0"
+                 izz="0.1" />
+      </inertial>
+    </link>
     <xacro:hand_simple_transmission name="${name}_${side}_thumb" reduction="168" />
     <!-- Index finger -->

Commit message: Thumb position fix.

File: reem_description/urdf/hand/hand.urdf.xacro (robot description, xacro)
@@ -139,5 +139,5 @@
       <parent link="${name}_${side}_palm_link" />
       <child link="${name}_${side}_thumb_link" />
-      <origin xyz="0.03649 ${reflect * 0.008}  0.02" rpy="${(90.0 + reflect * 90.0) * deg_to_rad} ${(90.0 + 13) * deg_to_rad} ${reflect * 13.0 * deg_to_rad}" />
+      <origin xyz="0.03749 ${reflect * 0.008}  0.02" rpy="${(90.0 + reflect * 90.0) * deg_to_rad} ${(90.0 + 13) * deg_to_rad} ${reflect * 13.0 * deg_to_rad}" />
       <axis xyz="0 0 1" />
       <limit lower="${0.0 * deg_to_rad}" upper="${90.0 * deg_to_rad}" effort="2.0" velocity="${hand_max_vel}" />
