Commit message: Initial results with Gazebo 1.4.
- Upper body actuators working as expected.

- No sensors nor mobile base yet integrated.

File: reem_description/gazebo/gazebo.urdf.xacro (robot description, xacro)
@@ -11,23 +11,8 @@
        xmlns:interface="http://playerstage.sourceforge.net/gazebo/xmlschema/#interface">
   <gazebo>
-    <controller:gazebo_ros_controller_manager name="gazebo_ros_controller_manager" plugin="libgazebo_ros_controller_manager.so">
+    <plugin filename="libgazebo_ros_controller_manager.so" name="gazebo_ros_controller_manager">
       <alwaysOn>true</alwaysOn>
       <updateRate>1000.0</updateRate>
-      <interface:audio name="gazebo_ros_controller_manager_dummy_iface" />
-    </controller:gazebo_ros_controller_manager>
-    <!-- TODO: Implement for our robots or remove! -->
-    <controller:gazebo_ros_power_monitor name="gazebo_ros_power_monitor_controller" plugin="libgazebo_ros_power_monitor.so">
-      <alwaysOn>true</alwaysOn>
-      <updateRate>1.0</updateRate>
-      <timeout>5</timeout>
-      <interface:audio name="power_monitor_dummy_interface" />
-      <powerStateTopic>power_state</powerStateTopic>
-      <powerStateRate>10.0</powerStateRate>
-      <fullChargeCapacity>87.78</fullChargeCapacity>
-      <dischargeRate>-474</dischargeRate>
-      <chargeRate>525</chargeRate>
-      <dischargeVoltage>15.52</dischargeVoltage>
-      <chargeVoltage>16.41</chargeVoltage>
-    </controller:gazebo_ros_power_monitor>
+    </plugin>
   </gazebo>
   <!-- define global properties -->

File: reem_description/robots/reem.urdf.xacro (robot description, xacro)
@@ -24,5 +24,5 @@
   <include filename="$(find reem_description)/urdf/hand/hand.urdf.xacro" />
   <!-- Camera sensors -->
-  <include filename="$(find reem_description)/urdf/sensors/stereo_camera.urdf.xacro" />
+<!--   <include filename="$(find reem_description)/urdf/sensors/stereo_camera.urdf.xacro" /> -->
   <!--<include filename="$(find reem_description)/urdf/sensors/back_camera.urdf.xacro" /> -->
   <!-- Generic simulator_gazebo plugins -->
@@ -42,8 +42,8 @@
   <!-- stereo camera -->
   <!-- IMPORTANT: focal_length = image_width/(2tan(hfov/2)) -->
-  <xacro:stereo_camera_v0 parent="head_2_link" name="stereo" focal_length_left="459.838918" hfov_left="71" focal_length_right="459.838918" hfov_right="71" image_format="B8G8R8" image_width="656" image_height="492">
+<!--  <xacro:stereo_camera_v0 parent="head_2_link" name="stereo" focal_length_left="459.838918" hfov_left="71" focal_length_right="459.838918" hfov_right="71" image_format="B8G8R8" image_width="656" image_height="492">-->
     <!-- The following transformations expresses the pose of the stereo_link (X pointing forward, Z upwards and Y leftwards, contrary to the stereo_optical_link which has Z pointing forward) wrt  head_2_link. -->
-     <origin xyz="0.08203  -0.09558  0.04132" rpy="1.56293 -0.00855922 -0.0201307" />
-  </xacro:stereo_camera_v0>
+<!--     <origin xyz="0.08203  -0.09558  0.04132" rpy="1.56293 -0.00855922 -0.0201307" />
+  </xacro:stereo_camera_v0>-->
 <!--   <xacro:back_camera_v0 parent="torso_2_link" name="back" focal_length="557" hfov="75" image_format="B8G8R8" image_width="640" image_height="480" >  -->
     <!-- The following transformations expresses the pose of the back_link (X pointing forward, Z upwards and Y leftwards, contrary to the stereo_optical_link which has Z pointing forward) wrt  torso_2_link. -->

File: reem_description/urdf/arm/arm.urdf.xacro (robot description, xacro)
@@ -22,5 +22,4 @@
   <include filename="$(find reem_description)/urdf/deg_to_rad.xacro" />
   <include filename="$(find reem_description)/urdf/arm/wrist.urdf.xacro" />
-  <include filename="$(find reem_description)/urdf/arm/arm.gazebo.xacro" />
   <include filename="$(find reem_description)/urdf/arm/arm.transmission.xacro" />
   <xacro:macro name="reem_arm" params="name parent side reflect">
@@ -183,8 +182,4 @@
     </joint>
     <!-- extensions -->
-    <xacro:reem_arm_gazebo side="${side}" number="1" />
-    <xacro:reem_arm_gazebo side="${side}" number="2" />
-    <xacro:reem_arm_gazebo side="${side}" number="3" />
-    <xacro:reem_arm_gazebo side="${side}" number="4" />
     <xacro:reem_arm_simple_transmission name="${name}" side="${side}" number="1" reduction="${arm_reduction_high}" />
     <xacro:reem_arm_simple_transmission name="${name}" side="${side}" number="2" reduction="${arm_reduction_high}" />

File: reem_description/urdf/arm/wrist.urdf.xacro (robot description, xacro)
@@ -19,5 +19,4 @@
   <!--File includes-->
   <include filename="$(find reem_description)/urdf/deg_to_rad.xacro" />
-  <include filename="$(find reem_description)/urdf/arm/wrist.gazebo.xacro" />
   <include filename="$(find reem_description)/urdf/arm/wrist.transmission.xacro" />
   <xacro:macro name="reem_wrist" params="name parent side reflect">
@@ -117,7 +116,4 @@
     </joint>
     <!-- extensions -->
-    <xacro:reem_wrist_gazebo name="${name}" side="${side}" number="5" />
-    <xacro:reem_wrist_gazebo name="${name}" side="${side}" number="6" />
-    <xacro:reem_wrist_gazebo name="${name}" side="${side}" number="7" />
     <xacro:reem_wrist_simple_transmission name="${name}" side="${side}" number="5" reduction="${wrist_reduction}" />
     <xacro:reem_wrist_simple_transmission name="${name}" side="${side}" number="6" reduction="${wrist_reduction}" />

File: reem_description/urdf/base/base.gazebo.xacro (robot description, xacro)
@@ -11,28 +11,7 @@
         xmlns:controller="http://playerstage.sourceforge.net/gazebo/xmlschema/#controller"
         xmlns:interface="http://playerstage.sourceforge.net/gazebo/xmlschema/#interface">
-  <xacro:macro name="reem_wheel_gazebo" params="side">
-    <gazebo reference="wheel_${side}_link">
-      <material>reem/DarkGrey</material>
-      <turnGravityOff>false</turnGravityOff>
-    </gazebo>
-  </xacro:macro>
-  <xacro:macro name="reem_caster_gazebo" params="side">
-    <gazebo reference="caster_${side}_1_link">
-      <material>reem/LightGrey</material>
-      <turnGravityOff>false</turnGravityOff>
-    </gazebo>
-    <gazebo reference="caster_${side}_2_link">
-      <material>reem/DarkGrey</material>
-      <turnGravityOff>false</turnGravityOff>
-    </gazebo>
-  </xacro:macro>
-  <xacro:macro name="reem_base_gazebo">
-    <gazebo reference="base_link">
-      <turnGravityOff>false</turnGravityOff>
-    </gazebo>
-  </xacro:macro>
- <xacro:macro name="reem_base_controllers">
+  <xacro:macro name="reem_base_controllers">
         <!-- CONTROLLERS -->
-        <gazebo>
+<!--        <gazebo>
             <canonicalBody>base_footprint</canonicalBody>
             <controller:diffdrive_plugin name="reem_differential_drive_controller" plugin="libreem_diffdrive_plugin.so">
@@ -49,5 +28,5 @@
                 <topicName>/cmd_vel</topicName>
             </controller:diffdrive_plugin>
-        </gazebo>
+        </gazebo>-->
   </xacro:macro>
 </robot>

File: reem_description/urdf/base/base.urdf.xacro (robot description, xacro)
@@ -14,10 +14,10 @@
   <include filename="$(find reem_description)/urdf/base/base.gazebo.xacro" />
   <include filename="$(find reem_description)/urdf/base/base.transmission.xacro" />
-  <include filename="$(find reem_description)/urdf/sensors/sick_laser_reem.urdf.xacro" />
-  <include filename="$(find reem_description)/urdf/sensors/hokuyo_laser_reem.urdf.xacro" />
+<!--   <include filename="$(find reem_description)/urdf/sensors/sick_laser_reem.urdf.xacro" /> -->
+<!--   <include filename="$(find reem_description)/urdf/sensors/hokuyo_laser_reem.urdf.xacro" /> -->
   <!--<include filename="$(find reem_description)/urdf/sensors/microinfinity_xa3300.urdf.xacro" /> -->
-  <include filename="$(find reem_description)/urdf/sensors/microstrain_3dmgx2_imu.urdf.xacro" />
-  <include filename="$(find reem_description)/urdf/sensors/range.urdf.xacro" />
-  <include filename="$(find reem_description)/urdf/sensors/bumper.urdf.xacro" />
+<!--   <include filename="$(find reem_description)/urdf/sensors/microstrain_3dmgx2_imu.urdf.xacro" /> -->
+<!--   <include filename="$(find reem_description)/urdf/sensors/range.urdf.xacro" /> -->
+<!--   <include filename="$(find reem_description)/urdf/sensors/bumper.urdf.xacro" /> -->
   <!--wheel characteristics-->
   <property name="dist_between_wheels" value="0.492" />
@@ -63,5 +63,4 @@
     </joint>
     <!-- extensions -->
-    <xacro:reem_wheel_gazebo side="${side}" />
     <xacro:reem_wheel_transmission side="${side}" />
   </xacro:macro>
@@ -128,5 +127,4 @@
     </joint>
     <!-- extensions -->
-    <xacro:reem_caster_gazebo side="${side}"/>
     <xacro:reem_caster_simple_transmission name="caster" side="${side}" number="1" reduction="1" />
     <xacro:reem_caster_simple_transmission name="caster" side="${side}" number="2" reduction="1" />
@@ -326,5 +324,4 @@
     <xacro:reem_caster side="left"  reflect="-1.0" />
     <!-- extensions -->
-    <xacro:reem_base_gazebo />
     <xacro:reem_base_controllers />
   </xacro:macro>

File: reem_description/urdf/hand/hand.gazebo.xacro (robot description, xacro)
@@ -11,13 +11,6 @@
        xmlns:interface="http://playerstage.sourceforge.net/gazebo/xmlschema/#interface"
        xmlns:xacro="http://ros.org/wiki/xacro">
-    <xacro:macro name="hand_gazebo" params="name">
-    <gazebo reference="${name}_link">
-      <turnGravityOff>false</turnGravityOff>
-      <dampingFactor>0.025</dampingFactor>
-    </gazebo>
-    </xacro:macro>
     <xacro:macro name="hand_grasping_hack" params="side">
       <gazebo>
-      <!-- a formal implementation of grasp hack in gazebo with fixed joint reference: /opt/ros/fuerte/stacks/pr2_common/pr2_description/urdf/gripper_v0/gripper.gazebo.xacro -->
         <gripper name="${side}_grasp_hack">
           <grasp_check attach_steps="20" detach_steps="40" min_contact_count="2" />

File: reem_description/urdf/hand/hand.urdf.xacro (robot description, xacro)
@@ -106,7 +106,4 @@
       </collision>
     </link>
-    <xacro:hand_gazebo              name="${hand_name}_${hand_side}_${finger_name}_1"/>
-    <xacro:hand_gazebo              name="${hand_name}_${hand_side}_${finger_name}_2"/>
-    <xacro:hand_gazebo              name="${hand_name}_${hand_side}_${finger_name}_3"/>
     <xacro:hand_simple_transmission name="${hand_name}_${hand_side}_${finger_name}_1" reduction="200"/>
     <xacro:hand_simple_transmission name="${hand_name}_${hand_side}_${finger_name}_2" reduction="200"/>
@@ -172,5 +169,4 @@
       </collision>
     </link>
-    <xacro:hand_gazebo name="${name}_${side}_thumb"/>
     <xacro:hand_simple_transmission name="${name}_${side}_thumb" reduction="168" />
     <!-- Index finger -->

File: reem_description/urdf/head/head.transmission.xacro (robot description, xacro)
@@ -11,16 +11,9 @@
        xmlns:interface="http://playerstage.sourceforge.net/gazebo/xmlschema/#interface"
        xmlns:xacro="http://ros.org/wiki/xacro">
-  <xacro:macro name="reem_head_1_transmission" params="name">
+  <xacro:macro name="head_transmission" params="name reduction">
     <transmission type="pr2_mechanism_model/SimpleTransmission" name="${name}_trans">
       <actuator name="${name}_motor" />
       <joint name="${name}_joint" />
-      <mechanicalReduction>144.0</mechanicalReduction>
-    </transmission>
-  </xacro:macro>
-  <xacro:macro name="reem_head_2_transmission" params="name">
-    <transmission type="pr2_mechanism_model/SimpleTransmission" name="${name}_trans">
-      <actuator name="${name}_motor" />
-      <joint name="${name}_joint" />
-      <mechanicalReduction>320.32</mechanicalReduction>
+      <mechanicalReduction>${reduction}</mechanicalReduction>
     </transmission>
   </xacro:macro>

File: reem_description/urdf/head/head.urdf.xacro (robot description, xacro)
@@ -12,5 +12,4 @@
        xmlns:xacro="http://ros.org/wiki/xacro">
   <include filename="$(find reem_description)/urdf/deg_to_rad.xacro" />
-  <include filename="$(find reem_description)/urdf/head/head.gazebo.xacro" />
   <include filename="$(find reem_description)/urdf/head/head.transmission.xacro" />
   <xacro:property name="head_friction" value="1.0" />
@@ -52,6 +51,5 @@
     </joint>
     <!-- extensions -->
-    <xacro:reem_head_1_gazebo name="${name}" />
-    <xacro:reem_head_1_transmission name="${name}" />
+    <xacro:head_transmission name="${name}" reduction="144" />
   </xacro:macro>
   <!--************************-->
@@ -95,6 +93,5 @@
     </xacro:range_reem>
     <!-- extensions -->
-    <xacro:reem_head_2_gazebo name="${name}" />
-    <xacro:reem_head_2_transmission name="${name}" />
+    <xacro:head_transmission name="${name}" reduction="320.32" />
   </xacro:macro>
   <xacro:macro name="reem_head" params="name parent">

File: reem_description/urdf/sensors/openni.gazebo.xacro (robot description, xacro)
@@ -16,5 +16,5 @@
        xmlns:xacro="http://ros.org/wiki/xacro">
   <xacro:macro name="openni_ir_gazebo_v0" params="link_name frame_name camera_name">
-    <gazebo reference="${link_name}">
+<!--    <gazebo reference="${link_name}">
       <sensor:camera name="${name}_ir_sensor">
         <imageFormat>L8</imageFormat>
@@ -43,8 +43,8 @@
         </controller:gazebo_ros_openni_kinect>
       </sensor:camera>
-    </gazebo>
+    </gazebo>-->
   </xacro:macro>
   <xacro:macro name="openni_rgb_gazebo_v0" params="link_name frame_name camera_name">
-    <gazebo reference="${link_name}">
+    <!--<gazebo reference="${link_name}">
       <sensor:camera name="${name}_rgb_sensor">
         <imageFormat>R8G8B8</imageFormat>
@@ -71,5 +71,5 @@
         </controller:gazebo_ros_openni_kinect>
       </sensor:camera>
-    </gazebo>
+    </gazebo>-->
   </xacro:macro>
 </robot>

File: reem_description/urdf/torso/torso.urdf.xacro (robot description, xacro)
@@ -12,5 +12,4 @@
        xmlns:interface="http://playerstage.sourceforge.net/gazebo/xmlschema/#interface">
   <include filename="$(find reem_description)/urdf/deg_to_rad.xacro" />
-  <include filename="$(find reem_description)/urdf/torso/torso.gazebo.xacro" />
   <include filename="$(find reem_description)/urdf/torso/torso.transmission.xacro" />
   <xacro:property name="torso_max_vel"  value="1.0" />
@@ -47,5 +46,4 @@
     </joint>
     <!-- extensions -->
-    <xacro:reem_torso_1_gazebo />
     <xacro:reem_torso_1_transmission name="${name}" />
     <!--************************-->
@@ -93,5 +91,4 @@
    </xacro:range_reem>
     <!-- extensions -->
-    <xacro:reem_torso_2_gazebo />
     <xacro:reem_torso_2_transmission name="${name}" />
   </xacro:macro>
