Commit message: Update sensor setup, slightly smaller cargo volume.

File: reem_description/urdf/base/base.urdf.xacro (robot description, xacro)
@@ -199,5 +199,5 @@
     </joint>
    <!-- base laser -->
-    <xacro:sick_laser_reem name="${name}_laser" parent="${name}" ros_topic="/LMS1xx/LAS_00" update_rate="50" min_angle="-135" max_angle="135" >
+    <xacro:sick_laser_reem name="${name}_laser" parent="${name}" ros_topic="/LMS1xx/LAS_00" update_rate="25" min_angle="-135" max_angle="135" >
       <origin xyz="${base_laser_x} ${base_laser_y} ${base_laser_z}" rpy="${180.0 * deg_to_rad} 0 0" />
     </xacro:sick_laser_reem>
@@ -206,64 +206,60 @@
       <origin xyz="${torso_laser_x} ${torso_laser_y} ${torso_laser_z}" rpy="-0.07 ${65 * deg_to_rad} 0 " />
     </xacro:hokuyo_laser_reem>
-    <!-- base ir -->
-    <xacro:range_reem name="${name}_ir_00" parent="${name}" ros_topic="SonarBaseRing" update_rate="5" maxRange="0.83" minRange="0.005" fov="0.3491">
+    <!-- base sonar -->
+    <xacro:range_reem name="${name}_sonar_04" parent="${name}" ros_topic="sonar_base" update_rate="5" maxRange="1.5" minRange="0.005" fov="0.3491">
       <origin xyz="0.17131 0.0 0.1425" rpy="0.0 0.0 0.0" />
     </xacro:range_reem>
-    <!-- base ir -->
-    <xacro:range_reem name="${name}_ir_01" parent="${name}" ros_topic="SonarBaseRing" update_rate="5" maxRange="0.83" minRange="0.005" fov="0.3491">
+    <!-- base sonar -->
+    <xacro:range_reem name="${name}_sonar_05" parent="${name}" ros_topic="sonar_base" update_rate="5" maxRange="1.5" minRange="0.005" fov="0.3491">
       <origin xyz="0.16919 0.12345 0.1425" rpy="0.0 0.0 0.349" />
     </xacro:range_reem>
-   <!-- base sonar 2 -->
-    <xacro:range_reem name="${name}_ir_02" parent="${name}" ros_topic="SonarBaseRing" update_rate="5" maxRange="0.83" minRange="0.0" fov="0.3491" >
+   <!-- base sonar -->
+    <xacro:range_reem name="${name}_sonar_15" parent="${name}" ros_topic="sonar_base" update_rate="5" maxRange="1.5" minRange="0.0" fov="0.3491" >
       <origin xyz="0.16919 -0.12345 0.1425" rpy="0.0 0.0 -0.349" />
     </xacro:range_reem>
-   <!-- base sonar 3 -->
-    <xacro:range_reem name="${name}_ir_03" parent="${name}" ros_topic="SonarBaseRing" update_rate="5" maxRange="0.80" minRange="0.0" fov="0.3491" >
+   <!-- base sonar -->
+    <xacro:range_reem name="${name}_sonar_06" parent="${name}" ros_topic="sonar_base" update_rate="5" maxRange="1.5" minRange="0.0" fov="0.3491" >
       <origin xyz="0.13676 0.27111 0.13702" rpy="0.0 0.0 0.8377" /> <!--3 y 4  x=0.11676 y=0.25111-->
     </xacro:range_reem>
-   <!-- base sonar 4 -->
-    <xacro:range_reem name="${name}_ir_04" parent="${name}" ros_topic="SonarBaseRing" update_rate="5" maxRange="0.80" minRange="0.0" fov="0.3491" >
+   <!-- base sonar -->
+    <xacro:range_reem name="${name}_sonar_14" parent="${name}" ros_topic="sonar_base" update_rate="5" maxRange="1.5" minRange="0.0" fov="0.3491" >
       <origin xyz="0.13676 -0.27111 0.13702" rpy="0.0 0.0 -0.8377" />
     </xacro:range_reem>
-   <!-- base sonar 5 -->
-    <xacro:range_reem name="${name}_ir_05" parent="${name}" ros_topic="SonarBaseRing" update_rate="5" maxRange="0.85" minRange="0.0" fov="0.3491" >
-      <origin xyz="0.064 0.31455 0.1475" rpy="0.0 0.0 1.5708" /> <!--5 y 6  y=0.29455 -->
-    </xacro:range_reem>
-   <!-- base sonar 6 -->
-    <xacro:range_reem name="${name}_ir_06" parent="${name}" ros_topic="SonarBaseRing" update_rate="5" maxRange="0.85" minRange="0.0" fov="0.3491" >
+   <!-- base sonar -->
+    <xacro:range_reem name="${name}_sonar_07" parent="${name}" ros_topic="sonar_base" update_rate="5" maxRange="1.5" minRange="0.0" fov="0.3491" >
+      <origin xyz="0.064 0.33455 0.1475" rpy="0.0 0.0 1.5708" /> <!--5 y 6  y=0.29455 -->
+    </xacro:range_reem>
+   <!-- base sonar -->
+    <xacro:range_reem name="${name}_sonar_13" parent="${name}" ros_topic="sonar_base" update_rate="5" maxRange="1.5" minRange="0.0" fov="0.3491" >
       <origin xyz="0.064 -0.31455 0.1475" rpy="0.0 0.0 -1.5708" />
     </xacro:range_reem>
-   <!-- base sonar 7 -->
-    <xacro:range_reem name="${name}_ir_07" parent="${name}" ros_topic="SonarBaseRing" update_rate="5" maxRange="0.62" minRange="0.0" fov="0.3491" >
+   <!-- base sonar -->
+    <xacro:range_reem name="${name}_sonar_08" parent="${name}" ros_topic="sonar_base" update_rate="5" maxRange="1.5" minRange="0.0" fov="0.3491" >
       <origin xyz="-0.35563 0.28266 0.11219" rpy="0.0 0.0 1.9547" /> <!--7 y 8  y=0.27266 -->
     </xacro:range_reem>
-   <!-- base sonar 8 -->
-    <xacro:range_reem name="${name}_ir_08" parent="${name}" ros_topic="SonarBaseRing" update_rate="5" maxRange="0.62" minRange="0.0" fov="0.3491" >
+   <!-- base sonar -->
+    <xacro:range_reem name="${name}_sonar_12" parent="${name}" ros_topic="sonar_base" update_rate="5" maxRange="1.5" minRange="0.0" fov="0.3491" >
       <origin xyz="-0.35563 -0.28266 0.11219" rpy="0.0 0.0 -1.9547" />
     </xacro:range_reem>
-   <!-- base sonar 9 -->
-    <xacro:range_reem name="${name}_ir_09" parent="${name}" ros_topic="SonarBaseRing" update_rate="5" maxRange="0.87" minRange="0.0" fov="0.3491" >
+   <!-- base sonar -->
+    <xacro:range_reem name="${name}_sonar_09" parent="${name}" ros_topic="sonar_base" update_rate="5" maxRange="1.5" minRange="0.0" fov="0.3491" >
       <origin xyz="-0.49412 0.15127 0.15748" rpy="0.0 0.0 2.6354" /> <!--10 y 9  x=0.45412 -->
     </xacro:range_reem>
-   <!-- base sonar 10 -->
-    <xacro:range_reem name="${name}_ir_10" parent="${name}" ros_topic="SonarBaseRing" update_rate="5" maxRange="0.87" minRange="0.0" fov="0.3491" >
+   <!-- base sonar -->
+    <xacro:range_reem name="${name}_sonar_11" parent="${name}" ros_topic="sonar_base" update_rate="5" maxRange="1.5" minRange="0.0" fov="0.3491" >
       <origin xyz="-0.49412 -0.15127 0.15748" rpy="0.0 0.0 -2.6354" />
     </xacro:range_reem>
-   <!-- base sonar 11 -->
-    <xacro:range_reem name="${name}_ir_11" parent="${name}" ros_topic="SonarBaseRing" update_rate="5" maxRange="0.68" minRange="0.0" fov="0.3491" >
+   <!-- base sonar -->
+    <xacro:range_reem name="${name}_sonar_10" parent="${name}" ros_topic="sonar_base" update_rate="5" maxRange="1.5" minRange="0.0" fov="0.3491" >
       <origin xyz="-0.52188 0.0 0.12547" rpy="0.0 0.0 -3.1415" />  <!--11  x=-0.50188 -->
     </xacro:range_reem>
  <!-- Torso Front Sonar Ring -->
-   <!-- torso sonar 0 -->
-   <xacro:range_reem name="${name}_ir_t_0" parent="${name}" ros_topic="SonarUpperBody" update_rate="10" maxRange="0.45" minRange="0.0" fov="0.3491" >
+   <!-- torso sonar left -->
+   <xacro:range_reem name="${name}_sonar_18" parent="${name}" ros_topic="sonar_torso" update_rate="5" maxRange="1.45" minRange="0.0" fov="0.3491" >
       <origin xyz="0.04 0.065 0.95" rpy="0.0 0.0 0.0" />
    </xacro:range_reem>
-   <!-- torso sonar 1 -->
-   <xacro:range_reem name="${name}_ir_t_1" parent="${name}" ros_topic="SonarUpperBody" update_rate="10" maxRange="0.45" minRange="0.0" fov="0.3491" >
+   <!-- torso sonar right -->
+   <xacro:range_reem name="${name}_sonar_19" parent="${name}" ros_topic="sonar_torso" update_rate="5" maxRange="1.45" minRange="0.0" fov="0.3491" >
       <origin xyz="0.04 -0.065 0.95" rpy="0.0 0.0 0.0" />
-   </xacro:range_reem>
- <!-- Head Sonar -->
-   <xacro:range_reem name="${name}_ir_h_0" parent="${name}" ros_topic="SonarUpperBody" update_rate="10" maxRange="0.5" minRange="0.0" fov="0.3491" >
-      <origin xyz="0.035 0.0 1.55" rpy="0.0 0.0 0.0" />
    </xacro:range_reem>
     <!-- gyroscope microinfinity XA3300
@@ -306,5 +302,5 @@
         <origin xyz="0 0 0.0" rpy="0 0 0" />
         <geometry>
-          <box size="0.45 0.45 0.25" /> <!-- Generous hand luggage size allowed in an airplane is 0.55x0.45x0.25. This slightly smaller. -->
+          <box size="0.40 0.45 0.25" /> <!-- Generous hand luggage size allowed in an airplane is 0.55x0.45x0.25. This slightly smaller. -->
         </geometry>
       </collision>

File: reem_description/urdf/head/head.urdf.xacro (robot description, xacro)
@@ -86,4 +86,8 @@
       <dynamics damping="${head_damping}" friction="${head_friction}"/> <!--TODO: Tune-->
     </joint>
+       <!-- Head Sonar -->
+   <xacro:range_reem name="head_sonar_20" parent="${name}" ros_topic="sonar_torso" update_rate="5" maxRange="1.5" minRange="0.0" fov="0.3491" >
+      <origin xyz="0.066 -0.195 0.0" rpy="1.57 0.0 0.0" />
+   </xacro:range_reem>
     <!-- extensions -->
     <xacro:reem_head_2_gazebo name="${name}" />

Commit message: Update base inertial params. Improve bumper layout.

File: reem_description/urdf/base/base.urdf.xacro (robot description, xacro)
@@ -36,6 +36,6 @@
       <inertial>
         <origin xyz="0 0 0" rpy="0 0 0" />
-        <mass value="1.0" />
-        <inertia ixx="1"  ixy="0"  ixz="0" iyy="1" iyz="0" izz="1" />
+        <mass value="3.5" />
+        <inertia ixx="0.00156"  ixy="0"  ixz="0" iyy="0.00156" iyz="0" izz="0.0273" />
       </inertial>
       <visual>
@@ -92,8 +92,8 @@
       <inertial>
         <origin xyz="0 0 0" rpy="0 0 0"/>
-        <mass value="0.1" />
-        <inertia  ixx="0.012411765597" ixy="-0.000711733678" ixz="0.00050272983"
-                  iyy="0.015218160428" iyz="-0.000004273467"
-                  izz="0.011763977943" />
+        <mass value="0.4" />
+        <inertia  ixx="0.00044" ixy="0" ixz="0"
+                  iyy="0.00044" iyz="0"
+                  izz="0.00078" />
         </inertial>
       <visual>
@@ -176,8 +176,8 @@
     <link name="${name}_footprint">
       <inertial>
-        <mass value="1.0" />
+        <mass value="0.1" />
         <origin xyz="0 0 0" />
-        <inertia ixx="0.01" ixy="0.0" ixz="0.0"
-                 iyy="0.01" iyz="0.0" izz="0.01" />
+        <inertia ixx="0.0" ixy="0.0" ixz="0.0"
+                 iyy="0.0" iyz="0.0" izz="0.0" />
       </inertial>
       <visual>
@@ -277,29 +277,29 @@
     <!-- bumper front right -->
     <xacro:bumper_reem name="${name}_bumper_01" parent="${name}" ros_topic="bumper_contact" update_rate="25" >
-      <origin xyz="0.195 -0.15 0.15" rpy="0 0 ${-15.0 * deg_to_rad}" />
+      <origin xyz="0.205 -0.15 0.15" rpy="0 0 ${-15.0 * deg_to_rad}" />
     </xacro:bumper_reem>
     <!-- bumper front left -->
     <xacro:bumper_reem name="${name}_bumper_02" parent="${name}" ros_topic="bumper_contact" update_rate="25" >
-      <origin xyz="0.195 0.15 0.15" rpy="0 0 ${15.0 * deg_to_rad}" />
+      <origin xyz="0.205 0.15 0.15" rpy="0 0 ${15.0 * deg_to_rad}" />
     </xacro:bumper_reem>
     <!-- bumper left 1 -->
     <xacro:bumper_reem name="${name}_bumper_03" parent="${name}" ros_topic="bumper_contact" update_rate="25" >
-      <origin xyz="0.064 0.30 0.1" rpy="0 0 1.57" />
+      <origin xyz="-0.04 0.31 0.1" rpy="0 0 ${90.0 * deg_to_rad}" />
     </xacro:bumper_reem>
     <!-- bumper left 2 -->
     <xacro:bumper_reem name="${name}_bumper_04" parent="${name}" ros_topic="bumper_contact" update_rate="25" >
-      <origin xyz="-0.35 -0.27 0.075" rpy="0 0 1.57" />
+      <origin xyz="-0.3 0.29 0.1" rpy="0 0 ${100.0 * deg_to_rad}" />
     </xacro:bumper_reem>
     <!-- bumper back -->
     <xacro:bumper_reem name="${name}_bumper_05" parent="${name}" ros_topic="bumper_contact" update_rate="25" >
-      <origin xyz="-0.51 0.0 0.075" rpy="0 0 -3.1415" />
+      <origin xyz="-0.525 0.0 0.1" rpy="0 0 ${180.0 * deg_to_rad}" />
     </xacro:bumper_reem>
     <!-- bumper right 2 -->
     <xacro:bumper_reem name="${name}_bumper_06" parent="${name}" ros_topic="bumper_contact" update_rate="25" >
-      <origin xyz="-0.35 0.27 0.075" rpy="0 0 1.57" />
+      <origin xyz="-0.3 -0.29 0.1" rpy="0 0 ${-100.0 * deg_to_rad}" />
     </xacro:bumper_reem>
     <!-- bumper right 1 -->
     <xacro:bumper_reem name="${name}_bumper_07" parent="${name}" ros_topic="bumper_contact" update_rate="25" >
-      <origin xyz="0.064 -0.30 0.1" rpy="0 0 1.57" />
+      <origin xyz="-0.04 -0.31 0.1" rpy="0 0 ${-90.0 * deg_to_rad}" />
     </xacro:bumper_reem>
     <!-- gyroscope microinfinity XA3300
@@ -328,7 +328,7 @@
       <inertial>
         <mass value="1.0" />
-        <origin xyz="0 0 0" />
-        <inertia ixx="0.01" ixy="0.0" ixz="0.0"
-                 iyy="0.01" iyz="0.0" izz="0.01" />
+        <origin xyz="0 0 -0.5" />
+        <inertia ixx="0.0" ixy="0.0" ixz="0.0"
+                 iyy="0.0" iyz="0.0" izz="0.0" />
       </inertial>
       <visual>

File: reem_description/urdf/sensors/bumper.urdf.xacro (robot description, xacro)
@@ -22,20 +22,19 @@
          <inertial>
            <mass value="1.0" />
-           <origin xyz="0.0 0.0 0.0" />
            <inertia ixx="0.01" ixy="0.0" ixz="0.0" iyy="0.01" iyz="0.0" izz="0.01" />
          </inertial>
          <visual>
-           <origin xyz="0 0 0" rpy="0 0 0" />
+           <origin xyz="-0.02 0 0" rpy="0 0 0" />
            <geometry>
               <box size="0.001 0.001 0.001"/>
            </geometry>
-           <material name="White"/>
+           <material name="DarkGrey"/>
          </visual>
          <collision>
            <origin xyz="0 0 0" rpy="0 0 0" />
            <geometry>
-              <box size="0.05 0.1 0.05"/>
+              <box size="0.01 0.25 0.05"/>
            </geometry>
-	   <material name="LightGrey" />
+           <material name="DarkGrey" />
          </collision>
        </link>

Commit message: Move base_footprint visualization to a place where it is not visible.

File: reem_description/urdf/base/base.urdf.xacro (robot description, xacro)
@@ -182,5 +182,5 @@
       </inertial>
       <visual>
-        <origin xyz="0 0 0" rpy="0 0 0" />
+        <origin xyz="0 0 0.2" rpy="0 0 0" />
         <geometry>
           <box size="0.01 0.01 0.01" />

Commit message: Resize cargo collision geometry.

File: reem_description/urdf/base/base.urdf.xacro (robot description, xacro)
@@ -340,7 +340,7 @@
       </visual>
       <collision>
-        <origin xyz="0 0 0.0" rpy="0 0 0" />
-        <geometry>
-          <box size="0.40 0.45 0.25" /> <!-- Generous hand luggage size allowed in an airplane is 0.55x0.45x0.25. This slightly smaller. -->
+        <origin xyz="0.05 0 0.02" rpy="0 0 0" />
+        <geometry>
+          <box size="0.30 0.40 0.25" /> <!-- Generous hand luggage size allowed in an airplane is 0.55x0.45x0.25. This slightly smaller. -->
         </geometry>
       </collision>

Commit message: Update laser orientation.
Patch by Jose R. Capriles.

File: reem_description/urdf/base/base.urdf.xacro (robot description, xacro)
@@ -217,5 +217,5 @@
    <!-- base laser -->
     <xacro:sick_laser_reem name="${name}_laser" parent="${name}" ros_topic="/LMS1xx/LAS_00" update_rate="25" min_angle="-84" max_angle="84" >
-      <origin xyz="${base_laser_x} ${base_laser_y} ${base_laser_z}" rpy="0 0 0" />
+      <origin xyz="${base_laser_x} ${base_laser_y} ${base_laser_z}" rpy="${180.0 * deg_to_rad} 0 0" />
     </xacro:sick_laser_reem>
     <!-- torso laser -->
