Commit message: Updated urdf scripts with new sensors.

File: reem_description/urdf/base/base.gazebo.xacro (robot description, xacro)
@@ -33,29 +33,41 @@
     </gazebo>
   </xacro:macro>
-  <xacro:macro name="reem_base_controllers">
-		<gazebo>
-		  <controller:differential_position2d name="controller1">
-		    <update>100</update>
-		    <leftJoint>wheel_right_joint</leftJoint>
-		    <rightJoint>wheel_left_joint</rightJoint>
-		    <wheelSeparation>${dist_between_wheels}</wheelSeparation>
-		    <wheelDiameter>${2 * wheel_radius}</wheelDiameter>
-		    <!-- <torque>5</torque> -->
-		    <!--TODO: Remove?-->
-		    <torque>15</torque>
-		    <interface:position name="position_iface_0"/>
-		  </controller:differential_position2d>
-		  <controller:gazebo_ros_p3d name="p3d_base_controller" plugin="libgazebo_ros_p3d.so">
-		    <alwaysOn>true</alwaysOn>
-		    <updateRate>100.0</updateRate>
-		    <bodyName>base_link</bodyName>
-		    <topicName>base_pose_ground_truth</topicName>
-		    <gaussianNoise>0.01</gaussianNoise>
-		    <frameName>odom</frameName>
-		    <xyzOffsets>0 0 0</xyzOffsets>
-		    <rpyOffsets>0 0 0</rpyOffsets>
-		    <interface:position name="p3d_base_position"/>
-		  </controller:gazebo_ros_p3d>
-		</gazebo>
+ <xacro:macro name="reem_base_controllers">
+        <!-- CONTROLLERS -->
+        <gazebo>
+            <controller:reem_diffdrive_plugin name="reem_diffdrive_plugin" plugin="libreemDiffdrivePlugin.so">
+                <alwaysOn>true</alwaysOn>
+                <update>100</update>
+                <updateRate>100.0</updateRate>
+                <leftJoint>wheel_right_joint</leftJoint>
+                <rightJoint>wheel_left_joint</rightJoint>
+                <wheelSeparation>${dist_between_wheels}</wheelSeparation>
+                <wheelDiameter>${2 * wheel_radius}</wheelDiameter>
+                <torque>15</torque>
+                <interface:position name="position_iface_0"/>
+                <robotNamespace>/</robotNamespace>
+                <topicName>cmd_vel</topicName>
+            </controller:reem_diffdrive_plugin>
+            <controller:gazebo_ros_p3d name="p3d_base_controller" plugin="libgazebo_ros_p3d.so">
+                <alwaysOn>true</alwaysOn>
+                <updateRate>100.0</updateRate>
+                <bodyName>base_link</bodyName>
+                <topicName>base_pose_ground_truth</topicName>
+                <gaussianNoise>0.01</gaussianNoise>
+                <frameName>map</frameName>
+                <xyzOffsets>0 0 0</xyzOffsets>
+                <rpyOffsets>0 0 0</rpyOffsets>
+                <interface:position name="p3d_base_position"/>
+            </controller:gazebo_ros_p3d>
+            <canonicalBody>base_footprint</canonicalBody>
+            <!-- this publishes empty joint_states due to no transmission, but
+             triggering robot_state_publisher to publish tf between fixed joints in erratic,
+             (e.g. base_laser_link for the base_scan frame) -->
+       <!--     <controller:gazebo_ros_controller_manager name="gazebo_ros_controller_manager" plugin="libgazebo_ros_controller_manager.so">
+                <alwaysOn>true</alwaysOn>
+                <updateRate>100.0</updateRate>
+                <interface:audio name="gazebo_ros_controller_manager_dummy_iface" />
+            </controller:gazebo_ros_controller_manager> -->
+        </gazebo>
   </xacro:macro>
 </robot>

File: reem_description/urdf/base/base.transmission.xacro (robot description, xacro)
@@ -14,5 +14,5 @@
   <!-- wheels transmission -->
   <xacro:macro name="reem_wheel_transmission" params="side">
-    <transmission type="SimpleTransmission" name="wheel_${side}_trans">
+    <transmission type="pr2_mechanism_model/SimpleTransmission" name="wheel_${side}_trans">
       <actuator name="wheel_${side}_motor" />
       <joint name="wheel_${side}_joint" />
@@ -22,5 +22,5 @@
   <!-- caster transmissions -->
   <xacro:macro name="reem_caster_simple_transmission" params="name side number reduction" >
-    <transmission type="SimpleTransmission" name="${name}_${side}_${number}_trans">
+    <transmission type="pr2_mechanism_model/SimpleTransmission" name="${name}_${side}_${number}_trans">
       <actuator name="${name}_${side}_${number}_motor" />
       <joint name="${name}_${side}_${number}_joint" />

File: reem_description/urdf/base/base.urdf.xacro (robot description, xacro)
@@ -18,4 +18,5 @@
   <!--<include filename="$(find reem_description)/urdf/sensors/microinfinity_xa3300.urdf.xacro" /> -->
   <include filename="$(find reem_description)/urdf/sensors/microstrain_3dmgx2_imu.urdf.xacro" />
+  <include filename="$(find reem_description)/urdf/sensors/range.urdf.xacro" />
   <!--wheel characteristics-->
   <property name="dist_between_wheels" value="0.489" />
@@ -69,10 +70,12 @@
         <origin xyz="0 0 0" rpy="0 0 0"/>
         <mass value="0.1" />
-        <inertia ixx="0"  ixy="0"  ixz="0" iyy="0" iyz="0" izz="0" />
-      </inertial>
-      <visual>
-        <origin xyz="0 0 0" rpy="0 0 0" />
-        <geometry>
-          <cylinder radius="0.01" length="0.04"/>
+        <inertia  ixx="0.012411765597" ixy="-0.000711733678" ixz="0.00050272983"
+                  iyy="0.015218160428" iyz="-0.000004273467"
+                  izz="0.011763977943" />
+      </inertial>
+      <visual>
+        <origin xyz="0 0 0" rpy="0 0 0" />
+        <geometry>
+          <cylinder radius="${caster_radius}" length="${caster_width}"/>
         </geometry>
         <material name="DarkGrey" />
@@ -81,5 +84,5 @@
         <origin xyz="0 0 0" rpy="0 0 0" />
         <geometry>
-          <cylinder radius="0.01" length="0.04"/>
+          <cylinder radius="${caster_radius}" length="${caster_width}"/>
         </geometry>
       </collision>
@@ -135,5 +138,5 @@
   <property name="base_laser_collision_offset_x" value="0.00" />
   <!-- simplified box collision geometry for hokuyo laser -->
-   <property name="torso_laser_x" value="0.04" />
+  <property name="torso_laser_x" value="0.04" />
   <property name="torso_laser_y" value="0.0" />
   <property name="torso_laser_z" value="0.77" />
@@ -203,4 +206,65 @@
       <origin xyz="${torso_laser_x} ${torso_laser_y} ${torso_laser_z}" rpy="-0.07 ${65 * deg_to_rad} 0 " />
     </xacro:hokuyo_laser_reem>
+    <!-- base ir -->
+    <xacro:range_reem name="${name}_ir_00" parent="${name}" ros_topic="SonarBaseRing" update_rate="5" maxRange="0.83" minRange="0.005" fov="0.3491">
+      <origin xyz="0.17131 0.0 0.1425" rpy="0.0 0.0 0.0" />
+    </xacro:range_reem>
+    <!-- base ir -->
+    <xacro:range_reem name="${name}_ir_01" parent="${name}" ros_topic="SonarBaseRing" update_rate="5" maxRange="0.83" minRange="0.005" fov="0.3491">
+      <origin xyz="0.16919 0.12345 0.1425" rpy="0.0 0.0 0.349" />
+    </xacro:range_reem>
+   <!-- base sonar 2 -->
+    <xacro:range_reem name="${name}_ir_02" parent="${name}" ros_topic="SonarBaseRing" update_rate="5" maxRange="0.83" minRange="0.0" fov="0.3491" >
+      <origin xyz="0.16919 -0.12345 0.1425" rpy="0.0 0.0 -0.349" />
+    </xacro:range_reem>
+   <!-- base sonar 3 -->
+    <xacro:range_reem name="${name}_ir_03" parent="${name}" ros_topic="SonarBaseRing" update_rate="5" maxRange="0.80" minRange="0.0" fov="0.3491" >
+      <origin xyz="0.13676 0.27111 0.13702" rpy="0.0 0.0 0.8377" /> <!--3 y 4  x=0.11676 y=0.25111-->
+    </xacro:range_reem>
+   <!-- base sonar 4 -->
+    <xacro:range_reem name="${name}_ir_04" parent="${name}" ros_topic="SonarBaseRing" update_rate="5" maxRange="0.80" minRange="0.0" fov="0.3491" >
+      <origin xyz="0.13676 -0.27111 0.13702" rpy="0.0 0.0 -0.8377" />
+    </xacro:range_reem>
+   <!-- base sonar 5 -->
+    <xacro:range_reem name="${name}_ir_05" parent="${name}" ros_topic="SonarBaseRing" update_rate="5" maxRange="0.85" minRange="0.0" fov="0.3491" >
+      <origin xyz="0.064 0.31455 0.1475" rpy="0.0 0.0 1.5708" /> <!--5 y 6  y=0.29455 -->
+    </xacro:range_reem>
+   <!-- base sonar 6 -->
+    <xacro:range_reem name="${name}_ir_06" parent="${name}" ros_topic="SonarBaseRing" update_rate="5" maxRange="0.85" minRange="0.0" fov="0.3491" >
+      <origin xyz="0.064 -0.31455 0.1475" rpy="0.0 0.0 -1.5708" />
+    </xacro:range_reem>
+   <!-- base sonar 7 -->
+    <xacro:range_reem name="${name}_ir_07" parent="${name}" ros_topic="SonarBaseRing" update_rate="5" maxRange="0.62" minRange="0.0" fov="0.3491" >
+      <origin xyz="-0.35563 0.28266 0.11219" rpy="0.0 0.0 1.9547" /> <!--7 y 8  y=0.27266 -->
+    </xacro:range_reem>
+   <!-- base sonar 8 -->
+    <xacro:range_reem name="${name}_ir_08" parent="${name}" ros_topic="SonarBaseRing" update_rate="5" maxRange="0.62" minRange="0.0" fov="0.3491" >
+      <origin xyz="-0.35563 -0.28266 0.11219" rpy="0.0 0.0 -1.9547" />
+    </xacro:range_reem>
+   <!-- base sonar 9 -->
+    <xacro:range_reem name="${name}_ir_09" parent="${name}" ros_topic="SonarBaseRing" update_rate="5" maxRange="0.87" minRange="0.0" fov="0.3491" >
+      <origin xyz="-0.49412 0.15127 0.15748" rpy="0.0 0.0 2.6354" /> <!--10 y 9  x=0.45412 -->
+    </xacro:range_reem>
+   <!-- base sonar 10 -->
+    <xacro:range_reem name="${name}_ir_10" parent="${name}" ros_topic="SonarBaseRing" update_rate="5" maxRange="0.87" minRange="0.0" fov="0.3491" >
+      <origin xyz="-0.49412 -0.15127 0.15748" rpy="0.0 0.0 -2.6354" />
+    </xacro:range_reem>
+   <!-- base sonar 11 -->
+    <xacro:range_reem name="${name}_ir_11" parent="${name}" ros_topic="SonarBaseRing" update_rate="5" maxRange="0.68" minRange="0.0" fov="0.3491" >
+      <origin xyz="-0.52188 0.0 0.12547" rpy="0.0 0.0 -3.1415" />  <!--11  x=-0.50188 -->
+    </xacro:range_reem>
+ <!-- Torso Front Sonar Ring -->
+   <!-- torso sonar 0 -->
+   <xacro:range_reem name="${name}_ir_t_0" parent="${name}" ros_topic="SonarUpperBody" update_rate="10" maxRange="0.45" minRange="0.0" fov="0.3491" >
+      <origin xyz="0.04 0.065 0.95" rpy="0.0 0.0 0.0" />
+   </xacro:range_reem>
+   <!-- torso sonar 1 -->
+   <xacro:range_reem name="${name}_ir_t_1" parent="${name}" ros_topic="SonarUpperBody" update_rate="10" maxRange="0.45" minRange="0.0" fov="0.3491" >
+      <origin xyz="0.04 -0.065 0.95" rpy="0.0 0.0 0.0" />
+   </xacro:range_reem>
+ <!-- Head Sonar -->
+   <xacro:range_reem name="${name}_ir_h_0" parent="${name}" ros_topic="SonarUpperBody" update_rate="10" maxRange="0.5" minRange="0.0" fov="0.3491" >
+      <origin xyz="0.035 0.0 1.55" rpy="0.0 0.0 0.0" />
+   </xacro:range_reem>
     <!-- gyroscope microinfinity XA3300
     <xacro:microinfinity_xa3300 name="imu" parent="${name}" imu_topic="imu/data" update_rate="100.0" stdev="0.0005" >

Commit message: Update base to high resolution simulation model.
- Collada visualization geometries with color, normal and specularity maps.

- Low-poly stl collision geometries.

- Update dimensions.

- Rearrange front bumper locations.

- Change caster geometry.

File: reem_description/urdf/base/base.gazebo.xacro (robot description, xacro)
@@ -29,5 +29,4 @@
   <xacro:macro name="reem_base_gazebo">
     <gazebo reference="base_link">
-      <material>reem/LightGrey</material>
       <turnGravityOff>false</turnGravityOff>
     </gazebo>

File: reem_description/urdf/base/base.urdf.xacro (robot description, xacro)
@@ -1,5 +1,5 @@
 <?xml version="1.0"?>
 <!--
-  Copyright (c) 2011, PAL Robotics, S.L.
+  Copyright (c) 2011-2012, PAL Robotics, S.L.
   All rights reserved.
   This work is licensed under the Creative Commons Attribution-NonCommercial-NoDerivs 3.0 Unported License.
@@ -7,8 +7,8 @@
   Creative Commons, 444 Castro Street, Suite 900, Mountain View, California, 94041, USA.
 -->
-<robot  xmlns:xacro="http://ros.org/wiki/xacro"
-        xmlns:sensor="http://playerstage.sourceforge.net/gazebo/xmlschema/#sensor"
-        xmlns:controller="http://playerstage.sourceforge.net/gazebo/xmlschema/#controller"
-        xmlns:interface="http://playerstage.sourceforge.net/gazebo/xmlschema/#interface">
+<robot xmlns:xacro="http://ros.org/wiki/xacro"
+       xmlns:sensor="http://playerstage.sourceforge.net/gazebo/xmlschema/#sensor"
+       xmlns:controller="http://playerstage.sourceforge.net/gazebo/xmlschema/#controller"
+       xmlns:interface="http://playerstage.sourceforge.net/gazebo/xmlschema/#interface">
   <include filename="$(find reem_description)/urdf/deg_to_rad.xacro" />
   <include filename="$(find reem_description)/urdf/base/base.gazebo.xacro" />
@@ -21,12 +21,12 @@
   <include filename="$(find reem_description)/urdf/sensors/bumper.urdf.xacro" />
   <!--wheel characteristics-->
-  <property name="dist_between_wheels" value="0.489" />
-  <property name="wheel_radius" value="0.1075" />
-  <property name="wheel_width" value="0.082" />
+  <property name="dist_between_wheels" value="0.492" />
+  <property name="wheel_radius" value="0.125" />
+  <property name="wheel_width" value="0.087" />
  <!--caster characteristics-->
-  <property name="dist_between_casters" value="0.350" />
-  <property name="caster_radius"        value="0.050" />
-  <property name="caster_width"         value="0.032" />
-  <property name="caster_trailing_dist" value="0.033" />
+  <property name="dist_between_casters" value="0.300" />
+  <property name="caster_radius"        value="0.0625" />
+  <property name="caster_width"         value="0.037" />
+  <property name="caster_trailing_dist" value="0.038" />
   <xacro:macro name="reem_wheel" params="side reflect" parent="base_link">
     <!--************************-->
@@ -71,19 +71,19 @@
         <origin xyz="0 0 0" rpy="0 0 0"/>
         <mass value="0.1" />
-        <inertia  ixx="0.012411765597" ixy="-0.000711733678" ixz="0.00050272983"
-                  iyy="0.015218160428" iyz="-0.000004273467"
-                  izz="0.011763977943" />
-      </inertial>
-      <visual>
-        <origin xyz="0 0 0" rpy="0 0 0" />
-        <geometry>
-          <cylinder radius="${caster_radius}" length="${caster_width}"/>
+        <inertia  ixx="0" ixy="0" ixz="0"
+                  iyy="0" iyz="0"
+                  izz="0" />
+      </inertial>
+      <visual>
+        <origin xyz="${0.5 * caster_radius - caster_trailing_dist} 0 ${0.5 * caster_radius}" rpy="0 0 0" />
+        <geometry>
+          <box size="${caster_radius} ${1.2 * caster_width} ${caster_radius}"/>
         </geometry>
         <material name="DarkGrey" />
       </visual>
       <collision>
-        <origin xyz="0 0 0" rpy="0 0 0" />
-        <geometry>
-          <cylinder radius="${caster_radius}" length="${caster_width}"/>
+        <origin xyz="${0.5 * caster_radius - caster_trailing_dist} 0 ${0.5 * caster_radius}" rpy="0 0 0" />
+        <geometry>
+          <box size="${caster_radius} ${1.2 * caster_width} ${caster_radius}"/>
         </geometry>
       </collision>
@@ -152,12 +152,13 @@
     <link name="${name}_link">
       <inertial>
-        <origin xyz="-0.14527 -0.00003 0.24721" rpy="0 0 0" /> <!-- assuming d=0.6, w=0.5, h=0.4 -->
-        <mass value="63.58850" />
-        <inertia ixx="3.42"  ixy="0"  ixz="0" iyy="4.33" iyz="0" izz="5.08" /> <!-- assuming d=0.6, w=0.5, h=0.4 -->
-      </inertial>
-      <visual>
-        <origin xyz="0 0 0" rpy="0 0 0" />
-        <geometry>
-          <mesh filename="package://reem_description/meshes/base/base_low.stl" />
+        <origin xyz="-0.15006 -0.00031 0.24965" rpy="0 0 0" />
+        <mass value="64.063" />
+        <!-- NOTE: Assuming box with d=0.6, w=0.5, h=0.4 -->
+        <inertia ixx="3.42"  ixy="0"  ixz="0" iyy="4.33" iyz="0" izz="5.08" />
+      </inertial>
+      <visual>
+        <origin xyz="0 0 0" rpy="0 0 0" />
+        <geometry>
+          <mesh filename="package://reem_description/meshes/base/base.dae" />
         </geometry>
         <material name="LightGrey" />
@@ -166,5 +167,5 @@
         <origin xyz="0 0 0" rpy="0 0 0" />
         <geometry>
-          <mesh filename="package://reem_description/meshes/base/convex/base_low_convex.stlb" />
+          <mesh filename="package://reem_description/meshes/base/base_collision.stl" />
         </geometry>
         <material name="LightGrey" />
@@ -276,9 +277,9 @@
     <!-- bumper front right -->
     <xacro:bumper_reem name="${name}_bumper_01" parent="${name}" ros_topic="bumper_contact" update_rate="25" >
-      <origin xyz="0.15 -0.15 0.15" rpy="0 0 0" />
+      <origin xyz="0.195 -0.15 0.15" rpy="0 0 ${-15.0 * deg_to_rad}" />
     </xacro:bumper_reem>
     <!-- bumper front left -->
     <xacro:bumper_reem name="${name}_bumper_02" parent="${name}" ros_topic="bumper_contact" update_rate="25" >
-      <origin xyz="0.15 0.15 0.15" rpy="0 0 0" />
+      <origin xyz="0.195 0.15 0.15" rpy="0 0 ${15.0 * deg_to_rad}" />
     </xacro:bumper_reem>
     <!-- bumper left 1 -->
