Commit message: Update diffdrive plugin and range sensor configuration.

File: reem_description/urdf/base/base.gazebo.xacro (robot description, xacro)
@@ -12,21 +12,11 @@
         xmlns:interface="http://playerstage.sourceforge.net/gazebo/xmlschema/#interface">
   <xacro:macro name="reem_base_controllers">
-        <!-- CONTROLLERS -->
-<!--        <gazebo>
-            <canonicalBody>base_footprint</canonicalBody>
-            <controller:diffdrive_plugin name="reem_differential_drive_controller" plugin="libreem_diffdrive_plugin.so">
-                <alwaysOn>true</alwaysOn>
-                <update>100</update>
-                <updateRate>100.0</updateRate>
-                <leftJoint>wheel_right_joint</leftJoint>
-                <rightJoint>wheel_left_joint</rightJoint>
-                <wheelSeparation>${dist_between_wheels}</wheelSeparation>
-                <wheelDiameter>${2 * wheel_radius}</wheelDiameter>
-                <torque>15</torque>
-                <interface:position name="position_iface_0"/>
-                <robotNamespace>/</robotNamespace>
-                <topicName>/cmd_vel</topicName>
-            </controller:diffdrive_plugin>
-        </gazebo>-->
+    <gazebo>
+      <plugin filename="libgazebo_pal_ros_diffdrive.so" name="pal_gazebo_diff_drive">
+        <left_joint>wheel_left_joint</left_joint>
+        <right_joint>wheel_right_joint</right_joint>
+        <torque>15</torque>
+      </plugin>
+    </gazebo>
   </xacro:macro>
 </robot>

File: reem_description/urdf/base/base.urdf.xacro (robot description, xacro)
@@ -14,10 +14,10 @@
   <include filename="$(find reem_description)/urdf/base/base.gazebo.xacro" />
   <include filename="$(find reem_description)/urdf/base/base.transmission.xacro" />
-<!--   <include filename="$(find reem_description)/urdf/sensors/sick_laser_reem.urdf.xacro" /> -->
-<!--   <include filename="$(find reem_description)/urdf/sensors/hokuyo_laser_reem.urdf.xacro" /> -->
-  <!--<include filename="$(find reem_description)/urdf/sensors/microinfinity_xa3300.urdf.xacro" /> -->
-<!--   <include filename="$(find reem_description)/urdf/sensors/microstrain_3dmgx2_imu.urdf.xacro" /> -->
-<!--   <include filename="$(find reem_description)/urdf/sensors/range.urdf.xacro" /> -->
-<!--   <include filename="$(find reem_description)/urdf/sensors/bumper.urdf.xacro" /> -->
+  <include filename="$(find reem_description)/urdf/sensors/sick_laser_reem.urdf.xacro" />
+  <include filename="$(find reem_description)/urdf/sensors/range.urdf.xacro" />
+  <include filename="$(find reem_description)/urdf/sensors/hokuyo_laser_reem.urdf.xacro" />
+  <!-- <include filename="$(find reem_description)/urdf/sensors/microinfinity_xa3300.urdf.xacro" /> -->
+  <!-- <include filename="$(find reem_description)/urdf/sensors/microstrain_3dmgx2_imu.urdf.xacro" /> -->
+  <!-- <include filename="$(find reem_description)/urdf/sensors/bumper.urdf.xacro" /> -->
   <!--wheel characteristics-->
   <property name="dist_between_wheels" value="0.492" />
@@ -216,97 +216,97 @@
     </joint>
    <!-- base laser -->
-    <xacro:sick_laser_reem name="${name}_laser" parent="${name}" ros_topic="/LMS1xx/LAS_00" update_rate="25" min_angle="-84" max_angle="84" >
-      <origin xyz="${base_laser_x} ${base_laser_y} ${base_laser_z}" rpy="${180.0 * deg_to_rad} 0 0" />
-    </xacro:sick_laser_reem>
-    <!-- torso laser -->
-    <xacro:hokuyo_laser_reem name="${name}_torso_laser" parent="${name}" ros_topic="/hokuyo/LAS_01" update_rate="10" min_angle="-86" max_angle="86" >
-      <origin xyz="${torso_laser_x} ${torso_laser_y} ${torso_laser_z}" rpy="-0.03 ${52 * deg_to_rad} -0.05 " />
-    </xacro:hokuyo_laser_reem>
+    <xacro:sick_reem_laser name="${name}_laser" parent="${name}" ros_topic="/LMS1xx/LAS_00" update_rate="20" min_angle="-1.45" max_angle="1.45" >
+      <origin xyz="${base_laser_x} ${base_laser_y} ${base_laser_z}" rpy="0 0 0" />
+    </xacro:sick_reem_laser>
+   <!-- torso laser -->
+    <xacro:hokuyo_reem_laser name="${name}_torso_laser" parent="${name}" ros_topic="/hokuyo/LAS_01" update_rate="10" min_angle="-1.5" max_angle="1.5" >
+      <origin xyz="${torso_laser_x} ${torso_laser_y} ${torso_laser_z}" rpy="-0.03 ${52 * deg_to_rad} -0.05" />
+    </xacro:hokuyo_reem_laser>
     <!-- base sonar -->
-    <xacro:range_reem name="${name}_sonar_02" parent="${name}" ros_topic="sonar_base" update_rate="5" maxRange="0.75" minRange="0.005" fov="0.7" radiation="ultrasound">
+    <xacro:range_reem name="${name}_sonar_02" parent="${name}" ros_topic="sonar_base" update_rate="5" maxRange="0.75" minRange="0.01" fov="0.5" radiation="ultrasound">
       <origin xyz="0.17131 0.0 0.280" rpy="0.0 0.0 0.0" />
     </xacro:range_reem>
     <!-- base sonar -->
-    <xacro:range_reem name="${name}_sonar_03" parent="${name}" ros_topic="sonar_base" update_rate="5" maxRange="0.75" minRange="0.005" fov="0.7" radiation="ultrasound">
+    <xacro:range_reem name="${name}_sonar_03" parent="${name}" ros_topic="sonar_base" update_rate="5" maxRange="0.75" minRange="0.01" fov="0.5" radiation="ultrasound">
       <origin xyz="0.16919 0.14919 0.280" rpy="0.0 0.0 0.349" />
     </xacro:range_reem>
    <!-- base sonar -->
-    <xacro:range_reem name="${name}_sonar_01" parent="${name}" ros_topic="sonar_base" update_rate="5" maxRange="0.75" minRange="0.005" fov="0.7" radiation="ultrasound">
+    <xacro:range_reem name="${name}_sonar_01" parent="${name}" ros_topic="sonar_base" update_rate="5" maxRange="0.75" minRange="0.01" fov="0.5" radiation="ultrasound">
       <origin xyz="0.16919 -0.14919 0.280" rpy="0.0 0.0 -0.349" />
     </xacro:range_reem>
    <!-- base sonar -->
-    <xacro:range_reem name="${name}_sonar_04" parent="${name}" ros_topic="sonar_base" update_rate="5" maxRange="0.75" minRange="0.005" fov="0.7" radiation="ultrasound">
+    <xacro:range_reem name="${name}_sonar_04" parent="${name}" ros_topic="sonar_base" update_rate="5" maxRange="0.75" minRange="0.01" fov="0.5" radiation="ultrasound">
       <origin xyz="0.13676 0.27111 0.280" rpy="0.0 0.0 0.8377" />
     </xacro:range_reem>
    <!-- base sonar -->
-    <xacro:range_reem name="${name}_sonar_12" parent="${name}" ros_topic="sonar_base" update_rate="5" maxRange="0.75" minRange="0.005" fov="0.7" radiation="ultrasound">
+    <xacro:range_reem name="${name}_sonar_12" parent="${name}" ros_topic="sonar_base" update_rate="5" maxRange="0.75" minRange="0.01" fov="0.5" radiation="ultrasound">
       <origin xyz="0.13676 -0.27111 0.280" rpy="0.0 0.0 -0.8377" />
     </xacro:range_reem>
    <!-- base sonar -->
-    <xacro:range_reem name="${name}_sonar_05" parent="${name}" ros_topic="sonar_base" update_rate="5" maxRange="0.5" minRange="0.005" fov="0.7" radiation="ultrasound">
+    <xacro:range_reem name="${name}_sonar_05" parent="${name}" ros_topic="sonar_base" update_rate="5" maxRange="0.5" minRange="0.01" fov="0.5" radiation="ultrasound">
       <origin xyz="-0.14 0.33455 0.27" rpy="0.0 0.0 1.5708" />
     </xacro:range_reem>
    <!-- base sonar -->
-    <xacro:range_reem name="${name}_sonar_11" parent="${name}" ros_topic="sonar_base" update_rate="5" maxRange="0.5" minRange="0.005" fov="0.7" radiation="ultrasound">
+    <xacro:range_reem name="${name}_sonar_11" parent="${name}" ros_topic="sonar_base" update_rate="5" maxRange="0.5" minRange="0.01" fov="0.5" radiation="ultrasound">
       <origin xyz="-0.14 -0.33455 0.27" rpy="0.0 0.0 -1.5708" />
     </xacro:range_reem>
    <!-- base sonar -->
-    <xacro:range_reem name="${name}_sonar_06" parent="${name}" ros_topic="sonar_base" update_rate="5" maxRange="0.5" minRange="0.005" fov="0.7" radiation="ultrasound">
+    <xacro:range_reem name="${name}_sonar_06" parent="${name}" ros_topic="sonar_base" update_rate="5" maxRange="0.5" minRange="0.005" fov="0.5" radiation="ultrasound">
       <origin xyz="-0.35563 0.28266 0.25" rpy="0.0 0.0 1.9547" />
     </xacro:range_reem>
    <!-- base sonar -->
-    <xacro:range_reem name="${name}_sonar_10" parent="${name}" ros_topic="sonar_base" update_rate="5" maxRange="0.5" minRange="0.005" fov="0.7" radiation="ultrasound">
+    <xacro:range_reem name="${name}_sonar_10" parent="${name}" ros_topic="sonar_base" update_rate="5" maxRange="0.5" minRange="0.005" fov="0.5" radiation="ultrasound">
       <origin xyz="-0.35563 -0.28266 0.25" rpy="0.0 0.0 -1.9547" />
     </xacro:range_reem>
    <!-- base sonar -->
-    <xacro:range_reem name="${name}_sonar_07" parent="${name}" ros_topic="sonar_base" update_rate="5" maxRange="0.7" minRange="0.005" fov="0.7" radiation="ultrasound">
+    <xacro:range_reem name="${name}_sonar_07" parent="${name}" ros_topic="sonar_base" update_rate="5" maxRange="0.7" minRange="0.01" fov="0.5" radiation="ultrasound">
       <origin xyz="-0.48412 0.15127 0.29" rpy="0.0 0.0 2.6354" />
     </xacro:range_reem>
    <!-- base sonar -->
-    <xacro:range_reem name="${name}_sonar_09" parent="${name}" ros_topic="sonar_base" update_rate="5" maxRange="0.7" minRange="0.005" fov="0.7" radiation="ultrasound">
+    <xacro:range_reem name="${name}_sonar_09" parent="${name}" ros_topic="sonar_base" update_rate="5" maxRange="0.7" minRange="0.01" fov="0.5" radiation="ultrasound">
       <origin xyz="-0.48412 -0.15127 0.29" rpy="0.0 0.0 -2.6354" />
     </xacro:range_reem>
    <!-- base sonar -->
-    <xacro:range_reem name="${name}_sonar_08" parent="${name}" ros_topic="sonar_base" update_rate="5" maxRange="0.7" minRange="0.005" fov="0.7" radiation="ultrasound">
+    <xacro:range_reem name="${name}_sonar_08" parent="${name}" ros_topic="sonar_base" update_rate="5" maxRange="0.7" minRange="0.01" fov="0.5" radiation="ultrasound">
       <origin xyz="-0.51188 0.0 0.26" rpy="0.0 0.0 -3.1415" />
     </xacro:range_reem>
    <!-- base ir -->
-    <xacro:range_reem name="${name}_ir_01" parent="${name}" ros_topic="ir_base" update_rate="10" maxRange="1.45" minRange="0.005" fov="0.1" radiation="infrared">
+    <xacro:range_reem name="${name}_ir_01" parent="${name}" ros_topic="ir_base" update_rate="10" maxRange="1.45" minRange="0.01" fov="0.1" radiation="infrared">
       <origin xyz="0.1804 -0.12463 0.22" rpy="0.0 -0.8726 0.0" />
     </xacro:range_reem>
-    <xacro:range_reem name="${name}_ir_02" parent="${name}" ros_topic="ir_base" update_rate="10" maxRange="1.45" minRange="0.005" fov="0.1" radiation="infrared">
+    <xacro:range_reem name="${name}_ir_02" parent="${name}" ros_topic="ir_base" update_rate="10" maxRange="1.45" minRange="0.01" fov="0.1" radiation="infrared">
       <origin xyz="0.18574 0.0 0.22" rpy="0.0 -0.8726 0.0" />
     </xacro:range_reem>
-    <xacro:range_reem name="${name}_ir_03" parent="${name}" ros_topic="ir_base" update_rate="10" maxRange="1.45" minRange="0.005" fov="0.1" radiation="infrared">
+    <xacro:range_reem name="${name}_ir_03" parent="${name}" ros_topic="ir_base" update_rate="10" maxRange="1.45" minRange="0.01" fov="0.1" radiation="infrared">
       <origin xyz="0.1804 0.12463 0.22" rpy="0.0 -0.8726 0.0" />
     </xacro:range_reem>
     <!-- bumper front right -->
-    <!--xacro:bumper_reem name="${name}_bumper_01" parent="${name}" ros_topic="bumper_base" update_rate="25" >
+    <xacro:bumper_reem name="${name}_bumper_01" parent="${name}" ros_topic="bumper_base" update_rate="25" >
       <origin xyz="0.325 -0.15 0.15" rpy="0 0 ${-15.0 * deg_to_rad}" />
-    </xacro:bumper_reem-->
+    </xacro:bumper_reem>
     <!-- bumper front left -->
-    <!--xacro:bumper_reem name="${name}_bumper_02" parent="${name}" ros_topic="bumper_contact" update_rate="25" >
+    <xacro:bumper_reem name="${name}_bumper_02" parent="${name}" ros_topic="bumper_contact" update_rate="25" >
       <origin xyz="0.325 0.15 0.15" rpy="0 0 ${15.0 * deg_to_rad}" />
-    </xacro:bumper_reem-->
+    </xacro:bumper_reem>
     <!-- bumper left 1 -->
-    <!--xacro:bumper_reem name="${name}_bumper_03" parent="${name}" ros_topic="bumper_contact" update_rate="25" >
+    <xacro:bumper_reem name="${name}_bumper_03" parent="${name}" ros_topic="bumper_contact" update_rate="25" >
       <origin xyz="-0.04 0.33 0.1" rpy="0 0 ${90.0 * deg_to_rad}" />
-    </xacro:bumper_reem-->
+    </xacro:bumper_reem>
     <!-- bumper left 2 -->
-    <!--xacro:bumper_reem name="${name}_bumper_04" parent="${name}" ros_topic="bumper_contact" update_rate="25" >
+    <xacro:bumper_reem name="${name}_bumper_04" parent="${name}" ros_topic="bumper_contact" update_rate="25" >
       <origin xyz="-0.3 0.31 0.1" rpy="0 0 ${100.0 * deg_to_rad}" />
-    </xacro:bumper_reem-->
+    </xacro:bumper_reem>
     <!-- bumper back -->
-    <!--xacro:bumper_reem name="${name}_bumper_05" parent="${name}" ros_topic="bumper_contact" update_rate="25" >
+    <xacro:bumper_reem name="${name}_bumper_05" parent="${name}" ros_topic="bumper_contact" update_rate="25" >
       <origin xyz="-0.545 0.0 0.1" rpy="0 0 ${180.0 * deg_to_rad}" />
-    </xacro:bumper_reem-->
+    </xacro:bumper_reem>
     <!-- bumper right 2 -->
-    <!--xacro:bumper_reem name="${name}_bumper_06" parent="${name}" ros_topic="bumper_base" update_rate="25" >
+    <xacro:bumper_reem name="${name}_bumper_06" parent="${name}" ros_topic="bumper_base" update_rate="25" >
       <origin xyz="-0.3 -0.31 0.1" rpy="0 0 ${-100.0 * deg_to_rad}" />
-    </xacro:bumper_reem-->
+    </xacro:bumper_reem>
     <!-- bumper right 1 -->
-    <!--xacro:bumper_reem name="${name}_bumper_07" parent="${name}" ros_topic="bumper_contact" update_rate="25" >
+    <xacro:bumper_reem name="${name}_bumper_07" parent="${name}" ros_topic="bumper_contact" update_rate="25" >
       <origin xyz="-0.04 -0.33 0.1" rpy="0 0 ${-90.0 * deg_to_rad}" />
-    </xacro:bumper_reem-->
+    </xacro:bumper_reem>
     <!-- gyroscope microinfinity XA3300
     <xacro:microinfinity_xa3300 name="imu" parent="${name}" imu_topic="imu/data" update_rate="100.0" stdev="0.0005" >

Commit message: Added wheel joint effort and velocity. Removed old diff drive plugin from base urdf.

File: reem_description/urdf/base/base.gazebo.xacro (robot description, xacro)
@@ -12,11 +12,4 @@
         xmlns:interface="http://playerstage.sourceforge.net/gazebo/xmlschema/#interface">
   <xacro:macro name="reem_base_controllers">
-    <gazebo>
-      <plugin filename="libgazebo_pal_ros_diffdrive.so" name="pal_gazebo_diff_drive">
-        <left_joint>wheel_left_joint</left_joint>
-        <right_joint>wheel_right_joint</right_joint>
-        <torque>15</torque>
-      </plugin>
-    </gazebo>
   </xacro:macro>
 </robot>

File: reem_description/urdf/base/base.urdf.xacro (robot description, xacro)
@@ -24,4 +24,6 @@
   <property name="wheel_radius" value="0.125" />
   <property name="wheel_width" value="0.082" />
+  <property name="wheel_torque" value="5.0" />
+  <property name="wheel_velocity" value="1.5" /> <!-- m/s -->
  <!--caster characteristics-->
   <property name="dist_between_casters" value="0.300" />
@@ -61,4 +63,5 @@
       <origin xyz="0 ${-dist_between_wheels / 2 * reflect} ${wheel_radius}" rpy="${-90.0 * deg_to_rad} 0 0" />
       <axis xyz="0 0 1" />
+      <limit effort="${wheel_torque}" velocity="${wheel_velocity / wheel_radius}"/>
     </joint>
     <!-- extensions -->
